File: 2b/hardware/logicboard/p2b-001.sch (EAGLE design)
At the start: 72 parts, among them IC1 74LS06N, IC2 4066N, J1 MKR, J10 1-Wire, J2 GPIO, J3 Vcc, J4** RLY2, J5 SPI, J6 LED, J7 DIN5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

Commit message: Clean up of schematic.
Other:
- moved on the sheet: IC1B, IC1C
Changed lines of the file:
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@@
 <part name="SUPPLY26" library="supply2" deviceset="GND" device=""/>
 <part name="SUPPLY11" library="supply2" deviceset="GND" device=""/>
-<part name="SUPPLY28" library="supply2" deviceset="GND" device=""/>
 <part name="JP4" library="pinhead" library_urn="urn:adsk.eagle:library:325" deviceset="PINHD-1X2" device="" package3d_urn="urn:adsk.eagle:package:22435/2" value="RLYJMP"/>
 <part name="SUPPLY29" library="supply2" deviceset="GND" device=""/>
@@
 <part name="SUPPLY16" library="supply2" deviceset="GND" device=""/>
 <part name="SUPPLY17" library="supply2" deviceset="GND" device=""/>
-<part name="SUPPLY18" library="supply2" library_urn="urn:adsk.eagle:library:372" deviceset="VCC" device=""/>
 <part name="SUPPLY19" library="supply2" library_urn="urn:adsk.eagle:library:372" deviceset="VCC" device=""/>
 <part name="P+1" library="supply1" library_urn="urn:adsk.eagle:library:371" deviceset="VCC/2" device=""/>
@@
 <part name="J10" library="SparkFun-Connectors" library_urn="urn:adsk.eagle:library:513" deviceset="CONN_03" device="JST-PTH-VERT" package3d_urn="urn:adsk.eagle:package:38080/1" value="1-Wire"/>
 <part name="J20" library="SparkFun-Connectors" library_urn="urn:adsk.eagle:library:513" deviceset="CONN_04" device="1.27MM" package3d_urn="urn:adsk.eagle:package:38086/1"/>
+<part name="X1" library="wirepad" library_urn="urn:adsk.eagle:library:412" deviceset="PAD-N" device=""/>
+<part name="X2" library="wirepad" library_urn="urn:adsk.eagle:library:412" deviceset="PAD-N" device=""/>
 </parts>
 <sheets>
@@
 <attribute name="VALUE" x="139.7" y="83.82" size="1.778" layer="96" align="bottom-center"/>
 </instance>
-<instance part="IC1" gate="B" x="134.62" y="38.1" smashed="yes">
-<attribute name="NAME" x="139.7" y="40.64" size="1.778" layer="95" align="bottom-center"/>
-<attribute name="VALUE" x="139.7" y="33.02" size="1.778" layer="96" align="bottom-center"/>
-</instance>
-<instance part="IC1" gate="C" x="134.62" y="25.4" smashed="yes">
-<attribute name="NAME" x="139.7" y="27.94" size="1.778" layer="95" align="bottom-center"/>
-<attribute name="VALUE" x="139.7" y="20.32" size="1.778" layer="96" align="bottom-center"/>
+<instance part="IC1" gate="B" x="127" y="38.1" smashed="yes">
+<attribute name="NAME" x="132.08" y="40.64" size="1.778" layer="95" align="bottom-center"/>
+<attribute name="VALUE" x="132.08" y="33.02" size="1.778" layer="96" align="bottom-center"/>
+</instance>
+<instance part="IC1" gate="C" x="127" y="25.4" smashed="yes">
+<attribute name="NAME" x="132.08" y="27.94" size="1.778" layer="95" align="bottom-center"/>
+<attribute name="VALUE" x="132.08" y="20.32" size="1.778" layer="96" align="bottom-center"/>
 </instance>
 <instance part="IC1" gate="D" x="157.48" y="88.9" smashed="yes">
@@
 </instance>
 <instance part="SUPPLY11" gate="GND" x="241.3" y="198.12" smashed="yes"/>
-<instance part="SUPPLY28" gate="GND" x="203.2" y="198.12" smashed="yes"/>
 <instance part="JP4" gate="G$1" x="96.52" y="208.28" smashed="yes" rot="MR0">
 <attribute name="NAME" x="91.44" y="208.28" size="1.778" layer="95" rot="R90" align="bottom-center"/>
@@
 <instance part="SUPPLY16" gate="GND" x="259.08" y="48.26" smashed="yes"/>
 <instance part="SUPPLY17" gate="GND" x="292.1" y="48.26" smashed="yes"/>
-<instance part="SUPPLY18" gate="G$1" x="203.2" y="243.84" smashed="yes">
-<attribute name="VALUE" x="203.2" y="248.92" size="1.778" layer="96" align="bottom-center"/>
-</instance>
 <instance part="SUPPLY19" gate="G$1" x="167.64" y="170.18" smashed="yes">
 <attribute name="VALUE" x="167.64" y="175.26" size="1.778" layer="96" align="bottom-center"/>
@@
 <instance part="DISP1" gate="G$1" x="360.68" y="83.82" smashed="yes">
 <attribute name="NAME" x="363.22" y="93.98" size="1.778" layer="95"/>
-<attribute name="VALUE" x="363.22" y="71.12" size="1.778" layer="96"/>
+<attribute name="VALUE" x="355.6" y="71.12" size="1.778" layer="96"/>
 </instance>
 <instance part="R101" gate="G$1" x="269.24" y="83.82" smashed="yes" rot="R90">
@@
 <attribute name="NAME" x="40.64" y="38.608" size="1.778" layer="95" font="vector"/>
 </instance>
+<instance part="X1" gate="G$1" x="50.8" y="30.48" smashed="yes"/>
+<instance part="X2" gate="G$1" x="50.8" y="27.94" smashed="yes"/>
 </instances>
 <busses>
@@
 <pinref part="SUPPLY11" gate="GND" pin="GND"/>
 <wire x1="241.3" y1="203.2" x2="241.3" y2="200.66" width="0.1524" layer="91"/>
-</segment>
-<segment>
-<wire x1="200.66" y1="203.2" x2="203.2" y2="203.2" width="0.1524" layer="91"/>
-<pinref part="SUPPLY28" gate="GND" pin="GND"/>
-<wire x1="203.2" y1="203.2" x2="203.2" y2="200.66" width="0.1524" layer="91"/>
 </segment>
 <segment>
@@
 </segment>
 <segment>
-<wire x1="200.66" y1="213.36" x2="203.2" y2="213.36" width="0.1524" layer="91"/>
-<pinref part="SUPPLY18" gate="G$1" pin="VCC"/>
-<wire x1="203.2" y1="213.36" x2="203.2" y2="241.3" width="0.1524" layer="91"/>
-</segment>
-<segment>
 <pinref part="J1" gate="G$1" pin="5"/>
 <wire x1="73.66" y1="68.58" x2="76.2" y2="68.58" width="0.1524" layer="91"/>
@@
 <wire x1="53.34" y1="241.3" x2="53.34" y2="233.68" width="0.1524" layer="91"/>
 <junction x="53.34" y="233.68"/>
+<label x="66.04" y="233.68" size="1.778" layer="95"/>
 </segment>
 <segment>
@@
 </segment>
 <segment>
-<wire x1="200.66" y1="208.28" x2="203.2" y2="208.28" width="0.1524" layer="91"/>
-<label x="203.2" y="208.28" size="0.8128" layer="95" xref="yes"/>
-</segment>
-<segment>
 <pinref part="RN3" gate="1" pin="4"/>
 <wire x1="167.64" y1="142.24" x2="170.18" y2="142.24" width="0.1524" layer="91"/>
@@
 </segment>
 <segment>
-<wire x1="119.38" y1="38.1" x2="121.92" y2="38.1" width="0.1524" layer="91"/>
-<label x="119.38" y="38.1" size="0.8128" layer="95" rot="MR0" xref="yes"/>
+<wire x1="111.76" y1="38.1" x2="114.3" y2="38.1" width="0.1524" layer="91"/>
+<label x="111.76" y="38.1" size="0.8128" layer="95" rot="MR0" xref="yes"/>
 <pinref part="IC1" gate="B" pin="I"/>
-<wire x1="124.46" y1="38.1" x2="121.92" y2="38.1" width="0.1524" layer="91"/>
+<wire x1="116.84" y1="38.1" x2="114.3" y2="38.1" width="0.1524" layer="91"/>
 <pinref part="IC1" gate="C" pin="I"/>
-<wire x1="121.92" y1="25.4" x2="124.46" y2="25.4" width="0.1524" layer="91"/>
-<wire x1="121.92" y1="38.1" x2="121.92" y2="25.4" width="0.1524" layer="91"/>
-<junction x="121.92" y="38.1"/>
+<wire x1="114.3" y1="25.4" x2="116.84" y2="25.4" width="0.1524" layer="91"/>
+<wire x1="114.3" y1="38.1" x2="114.3" y2="25.4" width="0.1524" layer="91"/>
+<junction x="114.3" y="38.1"/>
 </segment>
 <segment>
@@
 <label x="116.84" y="236.22" size="0.8128" layer="95" xref="yes"/>
 <wire x1="88.9" y1="236.22" x2="116.84" y2="236.22" width="0.1524" layer="91"/>
+<label x="93.98" y="236.22" size="1.778" layer="95"/>
 </segment>
 </net>
@@
 <pinref part="JP1" gate="A" pin="5"/>
 <wire x1="81.28" y1="231.14" x2="63.5" y2="231.14" width="0.1524" layer="91"/>
+<label x="66.04" y="231.14" size="1.778" layer="95"/>
 </segment>
 <segment>
@@
 <wire x1="114.3" y1="231.14" x2="114.3" y2="233.68" width="0.1524" layer="91"/>
 <junction x="114.3" y="231.14"/>
+<label x="93.98" y="233.68" size="1.778" layer="95"/>
+<label x="93.98" y="231.14" size="1.778" layer="95"/>
 </segment>
 </net>
@@
 <junction x="124.46" y="200.66"/>
 <wire x1="132.08" y1="200.66" x2="132.08" y2="213.36" width="0.1524" layer="91"/>
-<label x="132.08" y="220.98" size="0.8128" layer="95" rot="R90" xref="yes"/>
+<label x="132.08" y="228.6" size="0.8128" layer="95" rot="R90" xref="yes"/>
 <pinref part="B" gate="1" pin="P"/>
-<wire x1="132.08" y1="213.36" x2="132.08" y2="220.98" width="0.1524" layer="91"/>
+<wire x1="132.08" y1="213.36" x2="132.08" y2="228.6" width="0.1524" layer="91"/>
 <wire x1="106.68" y1="215.9" x2="106.68" y2="208.28" width="0.1524" layer="91"/>
 <junction x="106.68" y="208.28"/>
@@
 <wire x1="137.16" y1="213.36" x2="132.08" y2="213.36" width="0.1524" layer="91"/>
 <junction x="132.08" y="213.36"/>
+<label x="104.14" y="200.66" size="1.778" layer="95"/>
 </segment>
 <segment>
@@
 <pinref part="K1" gate="2" pin="S"/>
 <wire x1="127" y1="210.82" x2="129.54" y2="210.82" width="0.1524" layer="91"/>
-<label x="129.54" y="220.98" size="0.8128" layer="95" rot="R90" xref="yes"/>
-<wire x1="129.54" y1="210.82" x2="129.54" y2="220.98" width="0.1524" layer="91"/>
+<label x="129.54" y="228.6" size="0.8128" layer="95" rot="R90" xref="yes"/>
+<wire x1="129.54" y1="210.82" x2="129.54" y2="228.6" width="0.1524" layer="91"/>
 </segment>
 <segment>
@@
 <pinref part="JP5" gate="A" pin="3"/>
 <wire x1="33.02" y1="236.22" x2="45.72" y2="236.22" width="0.1524" layer="91"/>
+<label x="66.04" y="236.22" size="1.778" layer="95"/>
 </segment>
 </net>
@@
 <pinref part="IC1" gate="B" pin="O"/>
 <pinref part="IC1" gate="E" pin="I"/>
-<wire x1="144.78" y1="38.1" x2="147.32" y2="38.1" width="0.1524" layer="91"/>
-<label x="144.78" y="40.64" size="0.8128" layer="95"/>
+<wire x1="137.16" y1="38.1" x2="147.32" y2="38.1" width="0.1524" layer="91"/>
+<label x="137.16" y="38.1" size="1.778" layer="95"/>
 </segment>
 <segment>
@@
 <pinref part="IC1" gate="C" pin="O"/>
 <pinref part="IC1" gate="F" pin="I"/>
-<wire x1="144.78" y1="25.4" x2="147.32" y2="25.4" width="0.1524" layer="91"/>
-<label x="144.78" y="27.94" size="0.8128" layer="95"/>
-</segment>
-<segment>
+<wire x1="137.16" y1="25.4" x2="147.32" y2="25.4" width="0.1524" layer="91"/>
+<label x="137.16" y="25.4" size="1.778" layer="95"/>
+</segment>
+<segment>
