File: 2b/hardware/logicboard/p2b-001.brd (EAGLE design)
At the start: 91 x 90 mm, 73 parts, among them IC1 74LS06N, IC2 4066N, J1 MKR, J10 1-Wire, J2 GPIO, J20 GPIO, J3 Vcc, J4** RLY2, J5 SPI, J6 LED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

Commit message: Changed pads to Inf-ohm chip resistor.
Parts:
- removed A, B: (no value), wirepad:SMD1,27-2,54
- added RZ0: Inf, rcl:M2012
- moved JP4 0.25 mm to (18.8, 32.5)
Connections:
- net VOUTRAW: now also RZ0.2; no longer B.1
- net VOUTRAW2: now also RZ0.1; no longer A.1
Routing:
- net VOUTRAW: track 89.2 -> 89.7 mm
- net VOUTRAW2: track 46.9 -> 47.5 mm
Changed lines of the file:
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@@
 <attribute name="VALUE" x="61" y="69.5" size="0.8128" layer="27" ratio="10" rot="R180" align="bottom-center"/>
 </element>
-<element name="JP4" library="pinhead" library_urn="urn:adsk.eagle:library:325" package="1X02" package3d_urn="urn:adsk.eagle:package:22435/2" value="RLYJMP" x="19" y="32.5" smashed="yes" rot="R90">
-<attribute name="NAME" x="19" y="29" size="1" layer="25" ratio="10" align="center"/>
-<attribute name="POPULARITY" value="98" x="19" y="32.5" size="1.778" layer="27" rot="R90" display="off"/>
-<attribute name="VALUE" x="17" y="32.5" size="0.8128" layer="27" rot="R90" align="bottom-center"/>
+<element name="JP4" library="pinhead" library_urn="urn:adsk.eagle:library:325" package="1X02" package3d_urn="urn:adsk.eagle:package:22435/2" value="RLYJMP" x="18.75" y="32.5" smashed="yes" rot="R90">
+<attribute name="NAME" x="18.75" y="29" size="1" layer="25" ratio="10" align="center"/>
+<attribute name="POPULARITY" value="98" x="18.75" y="32.5" size="1.778" layer="27" rot="R90" display="off"/>
+<attribute name="VALUE" x="16.75" y="32.5" size="0.8128" layer="27" rot="R90" align="bottom-center"/>
 </element>
 <element name="J1" library="SparkFun-Connectors" library_urn="urn:adsk.eagle:library:513" package="JST-5-PTH" package3d_urn="urn:adsk.eagle:package:38120/1" value="MKR" x="85" y="69" smashed="yes" rot="R270">
@@
 <attribute name="VALUE" x="73.349" y="61.698" size="0.6096" layer="27" font="vector" ratio="20"/>
 </element>
-<element name="A" library="wirepad" library_urn="urn:adsk.eagle:library:412" package="SMD1,27-2,54" package3d_urn="urn:adsk.eagle:package:30839/1" value="" x="21.5" y="31" smashed="yes">
-<attribute name="POPULARITY" value="15" x="21.5" y="31" size="1.778" layer="27" display="off"/>
-<attribute name="VALUE" x="21.5" y="31" size="0.0254" layer="27"/>
-</element>
-<element name="B" library="wirepad" library_urn="urn:adsk.eagle:library:412" package="SMD1,27-2,54" package3d_urn="urn:adsk.eagle:package:30839/1" value="" x="21.5" y="34" smashed="yes">
-<attribute name="POPULARITY" value="15" x="21.5" y="34" size="1.778" layer="27" display="off"/>
-<attribute name="VALUE" x="21.5" y="34" size="0.0254" layer="27"/>
-</element>
 <element name="SV3" library="pinhead" library_urn="urn:adsk.eagle:library:325" package="2X07" package3d_urn="urn:adsk.eagle:package:22478/2" value="Testport II" x="55.5" y="24" smashed="yes">
 <attribute name="NAME" x="65.5" y="24" size="1" layer="25" ratio="10" rot="R90" align="center"/>
@@
 <attribute name="POPULARITY" value="0" x="37" y="85.5" size="1.778" layer="28" rot="MR180" display="off"/>
 <attribute name="VALUE" x="33.317" y="91.469" size="1.27" layer="28" ratio="10" rot="MR180"/>
+</element>
+<element name="RZ0" library="rcl" library_urn="urn:adsk.eagle:library:334" package="M2012" package3d_urn="urn:adsk.eagle:package:23561/2" value="Inf" x="21.5" y="32.5" smashed="yes" rot="R90">
+<attribute name="NAME" x="21.5" y="30" size="1" layer="25" align="center"/>
+<attribute name="POPULARITY" value="0" x="21.5" y="32.5" size="1.778" layer="27" rot="R90" display="off"/>
+<attribute name="SPICEPREFIX" value="R" x="21.5" y="32.5" size="1.778" layer="27" rot="R90" display="off"/>
+<attribute name="VALUE" x="24.04" y="31.23" size="1.27" layer="27" rot="R90"/>
 </element>
 </elements>
@@
 <contactref element="K1" pad="1"/>
 <contactref element="JP4" pad="1"/>
-<contactref element="A" pad="1"/>
 <contactref element="RZ4**" pad="1"/>
+<contactref element="RZ0" pad="1"/>
 <wire x1="3.048" y1="51.3588" x2="3.048" y2="52.0446" width="1.016" layer="1"/>
 <wire x1="9.525" y1="44.8818" x2="3.048" y2="51.3588" width="1.016" layer="1"/>
@@
 <wire x1="3.048" y1="52.0446" x2="3" y2="52.05" width="1.016" layer="1"/>
 <wire x1="10.8966" y1="37.4904" x2="10.92" y2="37.46" width="1.016" layer="1"/>
-<wire x1="19.2024" y1="31.0134" x2="21.4884" y2="31.0134" width="1.016" layer="1"/>
-<wire x1="19.05" y1="31.1658" x2="19.2024" y2="31.0134" width="1.016" layer="1"/>
-<wire x1="21.4884" y1="31.0134" x2="21.5" y2="31" width="1.016" layer="1"/>
-<wire x1="19.05" y1="31.1658" x2="19" y2="31.23" width="1.016" layer="1"/>
+<wire x1="19.1262" y1="31.5468" x2="21.4884" y2="31.5468" width="1.016" layer="1"/>
+<wire x1="18.8214" y1="31.242" x2="19.1262" y2="31.5468" width="1.016" layer="1"/>
+<wire x1="21.4884" y1="31.5468" x2="21.5" y2="31.55" width="1.016" layer="1"/>
+<wire x1="18.8214" y1="31.242" x2="18.75" y2="31.23" width="1.016" layer="1"/>
 <wire x1="29.337" y1="24.003" x2="34.4424" y2="24.003" width="1.016" layer="1"/>
 <wire x1="25.2222" y1="28.1178" x2="29.337" y2="24.003" width="1.016" layer="16"/>
 <wire x1="23.6982" y1="29.6418" x2="25.2222" y2="28.1178" width="1.016" layer="1"/>
 <wire x1="22.9362" y1="29.6418" x2="23.6982" y2="29.6418" width="1.016" layer="1"/>
-<wire x1="21.8694" y1="30.7086" x2="22.9362" y2="29.6418" width="1.016" layer="1"/>
+<wire x1="21.717" y1="30.861" x2="22.9362" y2="29.6418" width="1.016" layer="1"/>
+<wire x1="21.717" y1="31.0896" x2="21.717" y2="30.861" width="1.016" layer="1"/>
 <wire x1="34.4424" y1="24.003" x2="34.46" y2="24" width="1.016" layer="1"/>
-<wire x1="21.8694" y1="30.7086" x2="21.5" y2="31" width="1.016" layer="1"/>
+<wire x1="21.717" y1="31.0896" x2="21.5" y2="31.55" width="1.016" layer="1"/>
 <wire x1="15.4686" y1="32.9184" x2="11.2776" y2="37.1094" width="1.016" layer="1"/>
-<wire x1="16.9926" y1="32.9184" x2="15.4686" y2="32.9184" width="1.016" layer="1"/>
-<wire x1="18.5166" y1="31.3944" x2="16.9926" y2="32.9184" width="1.016" layer="1"/>
+<wire x1="16.764" y1="32.9184" x2="15.4686" y2="32.9184" width="1.016" layer="1"/>
+<wire x1="18.288" y1="31.3944" x2="16.764" y2="32.9184" width="1.016" layer="1"/>
 <wire x1="11.2776" y1="37.1094" x2="10.92" y2="37.46" width="1.016" layer="1"/>
-<wire x1="18.5166" y1="31.3944" x2="19" y2="31.23" width="1.016" layer="1"/>
+<wire x1="18.288" y1="31.3944" x2="18.75" y2="31.23" width="1.016" layer="1"/>
 <via x="29.337" y="24.003" extent="1-16" drill="0.3048"/>
 <via x="25.2222" y="28.1178" extent="1-16" drill="0.3048"/>
@@
 <contactref element="K1" pad="5"/>
 <contactref element="JP4" pad="2"/>
-<contactref element="B" pad="1"/>
 <contactref element="RZ3**" pad="1"/>
 <contactref element="J3" pad="2"/>
+<contactref element="RZ0" pad="2"/>
 <wire x1="3.048" y1="45.9486" x2="3.048" y2="47.0154" width="1.016" layer="1"/>
 <wire x1="5.9436" y1="43.053" x2="3.048" y2="45.9486" width="1.016" layer="1"/>
 <wire x1="3.048" y1="47.0154" x2="3" y2="47.05" width="1.016" layer="1"/>
 <wire x1="5.9436" y1="43.053" x2="6" y2="43" width="1.016" layer="1"/>
-<wire x1="19.2024" y1="33.9852" x2="21.4884" y2="33.9852" width="1.016" layer="1"/>
-<wire x1="19.05" y1="33.8328" x2="19.2024" y2="33.9852" width="1.016" layer="1"/>
-<wire x1="21.4884" y1="33.9852" x2="21.5" y2="34" width="1.016" layer="1"/>
-<wire x1="19.05" y1="33.8328" x2="19" y2="33.77" width="1.016" layer="1"/>
-<wire x1="23.3934" y1="32.004" x2="23.3934" y2="31.0134" width="1.016" layer="1"/>
-<wire x1="21.7932" y1="33.6042" x2="23.0505" y2="32.3469" width="1.016" layer="1"/>
-<wire x1="23.0505" y1="32.3469" x2="23.3934" y2="32.004" width="1.016" layer="1"/>
+<wire x1="19.1262" y1="33.4518" x2="21.4884" y2="33.4518" width="1.016" layer="1"/>
+<wire x1="18.8214" y1="33.7566" x2="19.1262" y2="33.4518" width="1.016" layer="1"/>
+<wire x1="21.4884" y1="33.4518" x2="21.5" y2="33.45" width="1.016" layer="1"/>
+<wire x1="18.8214" y1="33.7566" x2="18.75" y2="33.77" width="1.016" layer="1"/>
+<wire x1="23.3934" y1="32.0802" x2="23.3934" y2="31.0134" width="1.016" layer="1"/>
+<wire x1="22.3266" y1="33.147" x2="23.0886" y2="32.385" width="1.016" layer="1"/>
+<wire x1="23.0886" y1="32.385" x2="23.3934" y2="32.0802" width="1.016" layer="1"/>
+<wire x1="21.9456" y1="33.147" x2="22.3266" y2="33.147" width="1.016" layer="1"/>
 <wire x1="23.3934" y1="31.0134" x2="23.46" y2="31" width="1.016" layer="1"/>
-<wire x1="21.7932" y1="33.6042" x2="21.5" y2="34" width="1.016" layer="1"/>
-<wire x1="21.1074" y1="34.4424" x2="21.1074" y2="37.4142" width="1.016" layer="1"/>
+<wire x1="21.9456" y1="33.147" x2="21.5" y2="33.45" width="1.016" layer="1"/>
+<wire x1="21.1074" y1="33.909" x2="21.1074" y2="37.4142" width="1.016" layer="1"/>
 <wire x1="21.1074" y1="37.4142" x2="21.08" y2="37.46" width="1.016" layer="1"/>
-<wire x1="21.1074" y1="34.4424" x2="21.5" y2="34" width="1.016" layer="1"/>
+<wire x1="21.1074" y1="33.909" x2="21.5" y2="33.45" width="1.016" layer="1"/>
+<wire x1="23.0886" y1="32.385" x2="24.6888" y2="33.9852" width="1.016" layer="1"/>
+<wire x1="24.6888" y1="33.9852" x2="24.73" y2="34" width="1.016" layer="1"/>
 <wire x1="21.1074" y1="37.4904" x2="21.1074" y2="42.5196" width="1.016" layer="16"/>
 <wire x1="21.1074" y1="42.5196" x2="21.08" y2="42.54" width="1.016" layer="16"/>
 <wire x1="21.1074" y1="37.4904" x2="21.08" y2="37.46" width="1.016" layer="16"/>
-<wire x1="23.0505" y1="32.3469" x2="24.6888" y2="33.9852" width="1.016" layer="1"/>
-<wire x1="24.6888" y1="33.9852" x2="24.73" y2="34" width="1.016" layer="1"/>
 <wire x1="18.669" y1="26.2128" x2="18.669" y2="25.6032" width="1.016" layer="16"/>
 <wire x1="23.3934" y1="30.9372" x2="18.669" y2="26.2128" width="1.016" layer="16"/>
