File: Peripherals/USBBox/hardware/logicboard/usbx-001.brd (EAGLE design)
At the start: 72 x 42 mm, 5 parts, among them J2 AUDIO_JACK_TRRSSMD_RA

Commit message: Routed.
Routing:
- net GND: track 0.00 -> 36.7 mm
- net D-: track 0.00 -> 32.0 mm
- net D+: track 0.00 -> 30.4 mm
- net VBUSR: track 0.00 -> 25.8 mm, vias 0 -> 2
- net VBUS: track 0.00 -> 5.59 mm
- removed copper zone on layer 16, net GND
Other:
- board text added: "121/000"
- board text added: "201/INF"
Changed lines of the file:
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@@
 <setting verticaltext="up"/>
 </settings>
-<grid distance="0.05" unitdist="mm" unit="mm" style="lines" multiple="2" display="yes" altdistance="50" altunitdist="mil" altunit="mil"/>
+<grid distance="1" unitdist="mm" unit="mm" style="lines" multiple="2" display="yes" altdistance="50" altunitdist="mil" altunit="mil"/>
 <layers>
 <layer number="1" name="Top" color="4" fill="1" visible="yes" active="yes"/>
@@
 PF8-2-5</text>
 <text x="11" y="12" size="1" layer="25" align="center">4-M2</text>
-<text x="9" y="24" size="1" layer="25" align="center">2012</text>
+<text x="36" y="32" size="1" layer="25" align="center">2012</text>
+<text x="40" y="30" size="1" layer="25" align="center">121/000</text>
+<text x="32" y="30" size="1" layer="25" align="center">201/INF</text>
 </plain>
 <attributes>
@@
 <clearance class="1" value="0.1524"/>
 </class>
-<class number="2" name="power" width="0.508" drill="0.1524">
+<class number="2" name="power" width="0.3048" drill="0.1524">
 <clearance class="2" value="0.1524"/>
 </class>
@@
 </element>
 <element name="R1" library="rcl" library_urn="urn:adsk.eagle:library:334" package="R2012" package3d_urn="urn:adsk.eagle:package:23543/2" value="120" x="40" y="32" smashed="yes" rot="R90">
-<attribute name="NAME" x="38.73" y="31.365" size="1.27" layer="25" rot="R90"/>
+<attribute name="NAME" x="42" y="32" size="1" layer="25" align="center"/>
 <attribute name="POPULARITY" value="0" x="40" y="32" size="1.778" layer="27" rot="R90" display="off"/>
 <attribute name="SPICEPREFIX" value="R" x="40" y="32" size="1.778" layer="27" rot="R90" display="off"/>
@@
 </element>
 <element name="R2" library="rcl" library_urn="urn:adsk.eagle:library:334" package="R2012" package3d_urn="urn:adsk.eagle:package:23543/2" value="200" x="32" y="32" smashed="yes" rot="R90">
-<attribute name="NAME" x="30.73" y="31.365" size="1.27" layer="25" rot="R90"/>
+<attribute name="NAME" x="30" y="32" size="1" layer="25" align="center"/>
 <attribute name="POPULARITY" value="0" x="32" y="32" size="1.778" layer="27" rot="R90" display="off"/>
 <attribute name="SPICEPREFIX" value="R" x="32" y="32" size="1.778" layer="27" rot="R90" display="off"/>
@@
 <contactref element="J1" pad="GND"/>
 <contactref element="J2" pad="RING2"/>
+<contactref element="R2" pad="2"/>
+<wire x1="34.7472" y1="35.6616" x2="34.7472" y2="37.2618" width="0.3048" layer="1"/>
+<wire x1="32.004" y1="32.9184" x2="34.7472" y2="35.6616" width="0.3048" layer="1"/>
+<wire x1="34.7472" y1="37.2618" x2="34.7" y2="37.275" width="0.3048" layer="1"/>
+<wire x1="32.004" y1="32.9184" x2="32" y2="32.85" width="0.3048" layer="1"/>
+<wire x1="32.6898" y1="5.9436" x2="32.6898" y2="5.2578" width="0.3048" layer="1"/>
+<wire x1="31.1658" y1="7.4676" x2="32.6898" y2="5.9436" width="0.3048" layer="1"/>
+<wire x1="31.1658" y1="8.9154" x2="31.1658" y2="7.4676" width="0.3048" layer="1"/>
+<wire x1="33.528" y1="11.2776" x2="31.1658" y2="8.9154" width="0.3048" layer="1"/>
+<wire x1="34.1376" y1="11.2776" x2="33.528" y2="11.2776" width="0.3048" layer="1"/>
+<wire x1="34.3662" y1="11.5062" x2="34.1376" y2="11.2776" width="0.3048" layer="1"/>
+<wire x1="34.3662" y1="30.7086" x2="34.3662" y2="11.5062" width="0.3048" layer="1"/>
+<wire x1="32.1564" y1="32.9184" x2="34.3662" y2="30.7086" width="0.3048" layer="1"/>
+<wire x1="32.6898" y1="5.2578" x2="32.75" y2="5.2" width="0.3048" layer="1"/>
+<wire x1="32.1564" y1="32.9184" x2="32" y2="32.85" width="0.3048" layer="1"/>
 <polygon width="0.2" layer="1">
-<vertex x="-2" y="-2"/>
-<vertex x="74" y="-2"/>
-<vertex x="74" y="44"/>
-<vertex x="-2" y="44"/>
+<vertex x="-1" y="-1"/>
+<vertex x="73" y="-1"/>
+<vertex x="73" y="43"/>
+<vertex x="-1" y="43"/>
 </polygon>
-<polygon width="0.2" layer="16">
-<vertex x="-3" y="-3"/>
-<vertex x="75" y="-3"/>
-<vertex x="75" y="45"/>
-<vertex x="-3" y="45"/>
-</polygon>
-<contactref element="R2" pad="2"/>
-<wire x1="32" y1="32.85" x2="34.7" y2="37.275" width="0" layer="19" extent="1-1"/>
-<wire x1="32.75" y1="5.2" x2="32" y2="32.85" width="0" layer="19" extent="1-1"/>
 </signal>
 <signal name="D-">
 <contactref element="J1" pad="D-"/>
 <contactref element="J2" pad="TIP"/>
-<wire x1="32.75" y1="12.2" x2="36.65" y2="37.275" width="0" layer="19" extent="1-1"/>
+<wire x1="36.576" y1="37.9476" x2="36.576" y2="37.338" width="0.1524" layer="1"/>
+<wire x1="35.9664" y1="38.5572" x2="36.576" y2="37.9476" width="0.1524" layer="1"/>
+<wire x1="33.7566" y1="38.5572" x2="35.9664" y2="38.5572" width="0.1524" layer="1"/>
+<wire x1="31.0134" y1="35.814" x2="33.7566" y2="38.5572" width="0.1524" layer="1"/>
+<wire x1="31.0134" y1="13.9446" x2="31.0134" y2="35.814" width="0.1524" layer="1"/>
+<wire x1="32.6898" y1="12.2682" x2="31.0134" y2="13.9446" width="0.1524" layer="1"/>
+<wire x1="36.576" y1="37.338" x2="36.65" y2="37.275" width="0.1524" layer="1"/>
+<wire x1="32.6898" y1="12.2682" x2="32.75" y2="12.2" width="0.1524" layer="1"/>
 </signal>
 <signal name="D+">
 <contactref element="J1" pad="D+"/>
 <contactref element="J2" pad="RING1"/>
-<wire x1="32.75" y1="8.2" x2="36" y2="37.275" width="0" layer="19" extent="1-1"/>
+<wire x1="35.9664" y1="11.8872" x2="35.9664" y2="37.2618" width="0.1524" layer="1"/>
+<wire x1="32.766" y1="8.6868" x2="35.9664" y2="11.8872" width="0.1524" layer="1"/>
+<wire x1="32.766" y1="8.2296" x2="32.766" y2="8.6868" width="0.1524" layer="1"/>
+<wire x1="35.9664" y1="37.2618" x2="36" y2="37.275" width="0.1524" layer="1"/>
+<wire x1="32.766" y1="8.2296" x2="32.75" y2="8.2" width="0.1524" layer="1"/>
 </signal>
 <signal name="VBUS" class="2">
 <contactref element="J1" pad="VBUS"/>
 <contactref element="R1" pad="2"/>
-<wire x1="40" y1="32.85" x2="37.3" y2="37.275" width="0" layer="19" extent="1-1"/>
+<wire x1="37.2618" y1="35.5854" x2="37.2618" y2="37.2618" width="0.3048" layer="1"/>
+<wire x1="39.9288" y1="32.9184" x2="37.2618" y2="35.5854" width="0.3048" layer="1"/>
+<wire x1="37.2618" y1="37.2618" x2="37.3" y2="37.275" width="0.3048" layer="1"/>
+<wire x1="39.9288" y1="32.9184" x2="40" y2="32.85" width="0.3048" layer="1"/>
 </signal>
 <signal name="VBUSR" class="2">
@@
 <contactref element="J2" pad="EARTH"/>
 <contactref element="R2" pad="1"/>
-<wire x1="32" y1="31.15" x2="40" y2="31.15" width="0" layer="19" extent="1-1"/>
-<wire x1="39.25" y1="13.3" x2="40" y2="31.15" width="0" layer="19" extent="1-1"/>
+<wire x1="33.0708" y1="31.0896" x2="32.004" y2="31.0896" width="0.3048" layer="1"/>
+<wire x1="33.2232" y1="30.9372" x2="33.0708" y2="31.0896" width="0.3048" layer="1"/>
+<wire x1="38.7858" y1="30.9372" x2="33.2232" y2="30.9372" width="0.3048" layer="16"/>
+<wire x1="39.7764" y1="30.9372" x2="39.243" y2="30.9372" width="0.3048" layer="1"/>
+<wire x1="39.243" y1="30.9372" x2="38.7858" y2="30.9372" width="0.3048" layer="1"/>
+<wire x1="39.9288" y1="31.0896" x2="39.7764" y2="30.9372" width="0.3048" layer="1"/>
+<wire x1="32.004" y1="31.0896" x2="32" y2="31.15" width="0.3048" layer="1"/>
+<wire x1="39.9288" y1="31.0896" x2="40" y2="31.15" width="0.3048" layer="1"/>
+<wire x1="39.243" y1="30.9372" x2="39.243" y2="13.335" width="0.3048" layer="1"/>
+<wire x1="39.243" y1="13.335" x2="39.25" y2="13.3" width="0.3048" layer="1"/>
+<via x="33.2232" y="30.9372" extent="1-16" drill="0.3048"/>
+<via x="38.7858" y="30.9372" extent="1-16" drill="0.3048"/>
 </signal>
 </signals>
