File: Peripherals/MIDIBox/hardware/logicboard/mbox-001.brd (EAGLE design)
At the start: 91 x 57 mm, 11 parts, among them J7 DIN5, J8 DIN5, J9 DIN5

Commit message: Fixed signal names and silk of MIDI Box.
Connections:
- net M1GND renamed M1SLV
- net M2GND renamed M2SLV
- net M3GND renamed M3SLV
- removed net M1RING: JJ7.TIP, S1.3, S1.4
- removed net M2RING: JJ8.TIP, S2.3, S2.4
- removed net M3RING: JJ9.TIP, S3.3, S3.4
- new net M1RNG: JJ7.RING, S1.1, S1.6
- new net M2RNG: JJ8.RING, S2.1, S2.6
- new net M3RNG: JJ9.RING, S3.1, S3.6
- net M1TIP: now also JJ7.TIP, S1.3, S1.4; no longer JJ7.RING, S1.1, S1.6
- net M2TIP: now also JJ8.TIP, S2.3, S2.4; no longer JJ8.RING, S2.1, S2.6
- net M3TIP: now also JJ9.TIP, S3.3, S3.4; no longer JJ9.RING, S3.1, S3.6
Routing:
- net M3RNG: track 0.00 -> 13.5 mm
- net M2RNG: track 0.00 -> 13.5 mm
- net M1RING: track 13.5 -> 0.00 mm
- net M1RNG: track 0.00 -> 13.5 mm
- net M2RING: track 13.4 -> 0.00 mm
- net M3RING: track 13.4 -> 0.00 mm
Changed lines of the file:
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@@
 <text x="45.5" y="25" size="1" layer="25" align="center">Type A (MIDI Standard): Tip=MIDI5, Ring=MIDI4; Type B: Tip=MIDI4, Ring=MIDI5; Sleeve=MIDI2</text>
 <text x="75" y="19" size="1" layer="25" align="center-left">NKK SS-22DP2</text>
-<text x="70.5" y="19" size="2" layer="25" align="center-left">B</text>
-<text x="59.5" y="19" size="2" layer="25" align="center-right">A</text>
-<text x="20.5" y="19" size="2" layer="25" align="center-right">A</text>
-<text x="40" y="19" size="2" layer="25" align="center-right">A</text>
-<text x="51" y="19" size="2" layer="25" align="center-left">B</text>
-<text x="31.5" y="19" size="2" layer="25" align="center-left">B</text>
+<text x="70.5" y="19" size="2" layer="25" align="center-left">A</text>
+<text x="59.5" y="19" size="2" layer="25" align="center-right">B</text>
+<text x="20.5" y="19" size="2" layer="25" align="center-right">B</text>
+<text x="40" y="19" size="2" layer="25" align="center-right">B</text>
+<text x="51" y="19" size="2" layer="25" align="center-left">A</text>
+<text x="31.5" y="19" size="2" layer="25" align="center-left">A</text>
 <text x="24" y="17.73" size="1" layer="25" align="center-right">1</text>
 <text x="45.5" y="16" size="1" layer="26" rot="MR0" align="center">RTN</text>
@@
 <wire x1="50.4444" y1="41.9862" x2="50.5" y2="42" width="0.1524" layer="1"/>
 </signal>
-<signal name="M1GND" class="2">
+<signal name="M1SLV" class="2">
 <contactref element="J7" pad="2"/>
 <contactref element="JJ7" pad="SLEEVE"/>
@@
 </polygon>
 </signal>
-<signal name="M3GND" class="2">
+<signal name="M3SLV" class="2">
 <contactref element="J9" pad="2"/>
 <contactref element="JJ9" pad="SLEEVE"/>
@@
 </polygon>
 </signal>
-<signal name="M2GND" class="2">
+<signal name="M2SLV" class="2">
 <contactref element="J8" pad="2"/>
 <contactref element="JJ8" pad="SLEEVE"/>
@@
 <wire x1="60.0456" y1="41.9862" x2="60" y2="42" width="0.1524" layer="1"/>
 </signal>
-<signal name="M1RING">
+<signal name="M1TIP">
 <contactref element="S1" pad="3"/>
 <contactref element="JJ7" pad="TIP"/>
@@
 <wire x1="67.5894" y1="17.6784" x2="67.54" y2="17.73" width="0.1524" layer="1"/>
 </signal>
-<signal name="M1TIP">
+<signal name="M1RNG">
 <contactref element="JJ7" pad="RING"/>
 <contactref element="S1" pad="6"/>
@@
 <wire x1="40.5384" y1="41.9862" x2="40.5" y2="42" width="0.1524" layer="16"/>
 </signal>
-<signal name="M2RING">
+<signal name="M2TIP">
 <contactref element="S2" pad="3"/>
 <contactref element="JJ8" pad="TIP"/>
@@
 <wire x1="48.0822" y1="17.6784" x2="48.04" y2="17.73" width="0.1524" layer="1"/>
 </signal>
-<signal name="M2TIP">
+<signal name="M2RNG">
 <contactref element="S2" pad="1"/>
 <contactref element="JJ8" pad="RING"/>
@@
 <wire x1="21.0312" y1="41.9862" x2="21" y2="42" width="0.1524" layer="1"/>
 </signal>
-<signal name="M3RING">
+<signal name="M3TIP">
 <contactref element="S3" pad="3"/>
 <contactref element="JJ9" pad="TIP"/>
@@
 <wire x1="28.575" y1="17.6784" x2="28.54" y2="17.73" width="0.1524" layer="1"/>
 </signal>
-<signal name="M3TIP">
+<signal name="M3RNG">
 <contactref element="S3" pad="1"/>
 <contactref element="S3" pad="6"/>
