File: Peripherals/MIDIBox/hardware/logicboard/mbox-001.sch (EAGLE design)
At the start: 11 parts, among them J7 DIN5, J8 DIN5, J9 DIN5

Commit message: Fixed signal names and silk of MIDI Box.
Connections:
- net M1GND renamed M1SLV
- net M2GND renamed M2SLV
- net M3GND renamed M3SLV
- removed net M1RING: JJ7.TIP, S11.O, S12.S
- removed net M2RING: JJ8.TIP, S21.O, S22.S
- removed net M3RING: JJ9.TIP, S31.O, S32.S
- new net M1RNG: JJ7.RING, S11.S, S12.O
- new net M2RNG: JJ8.RING, S21.S, S22.O
- new net M3RNG: JJ9.RING, S31.S, S32.O
- net M1TIP: now also JJ7.TIP, S11.O, S12.S; no longer JJ7.RING, S11.S, S12.O
- net M2TIP: now also JJ8.TIP, S21.O, S22.S; no longer JJ8.RING, S21.S, S22.O
- net M3TIP: now also JJ9.TIP, S31.O, S32.S; no longer JJ9.RING, S31.S, S32.O
Changed lines of the file:
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@@
 </segment>
 </net>
-<net name="M1GND" class="2">
+<net name="M1SLV" class="2">
 <segment>
 <pinref part="J7" gate="G$1" pin="2"/>
@@
 </segment>
 </net>
-<net name="M3GND" class="2">
+<net name="M3SLV" class="2">
 <segment>
 <pinref part="J9" gate="G$1" pin="2"/>
@@
 </segment>
 </net>
-<net name="M2GND" class="2">
+<net name="M2SLV" class="2">
 <segment>
 <pinref part="J8" gate="G$1" pin="2"/>
@@
 </segment>
 </net>
-<net name="M1RING" class="0">
+<net name="M1TIP" class="0">
 <segment>
 <pinref part="S1" gate="1" pin="O"/>
@@
 </segment>
 </net>
-<net name="M1TIP" class="0">
+<net name="M1RNG" class="0">
 <segment>
 <pinref part="JJ7" gate="G$1" pin="RING"/>
@@
 </segment>
 </net>
-<net name="M2RING" class="0">
+<net name="M2TIP" class="0">
 <segment>
 <pinref part="S2" gate="1" pin="O"/>
@@
 </segment>
 </net>
-<net name="M2TIP" class="0">
+<net name="M2RNG" class="0">
 <segment>
 <pinref part="S2" gate="1" pin="S"/>
@@
 </segment>
 </net>
-<net name="M3RING" class="0">
+<net name="M3TIP" class="0">
 <segment>
 <pinref part="S3" gate="1" pin="O"/>
@@
 </segment>
 </net>
-<net name="M3TIP" class="0">
+<net name="M3RNG" class="0">
 <segment>
 <pinref part="S3" gate="1" pin="S"/>
