File: 2gs/hardware/logicboard/p2gs-001.sch (EAGLE design)
At the start: 55 parts, among them J0 12V, J1 MKR, J7 DIN5, Q1 60V/32A/35mΩ, Q10 60V/32A/35mΩ, Q11 60V/32A/35mΩ, Q12 60V/32A/35mΩ, Q13 60V/32A/35mΩ, Q14 60V/32A/35mΩ, Q15 60V/32A/35mΩ, Q16 60V/32A/35mΩ, Q2 60V/32A/35mΩ, Q3 60V/32A/35mΩ, Q4 60V/32A/35mΩ, Q5 60V/32A/35mΩ, Q6 60V/32A/35mΩ, Q7 60V/32A/35mΩ, Q8 60V/32A/35mΩ, Q9 60V/32A/35mΩ, X1 ADAFRUIT-PCA9685

Commit message: Double Grove con.
Parts:
- added JG2: Grove/2, Connector:TWIG-4P-2.0'90D'
- JG1: value (none) -> Grove/1
- RN1, RN2: value (none) -> 10k
Connections:
- net GND: now also JG2.4
- net SCL: now also JG2.1
- net SDA: now also JG2.2
- net VCC: now also JG2.3
Other:
- moved on the sheet: JG1
Changed lines of the file:
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@@
 <part name="SUPPLY28" library="supply2" deviceset="GND" device=""/>
 <part name="SUPPLY30" library="supply2" deviceset="GND" device=""/>
-<part name="JG1" library="Connector" deviceset="TWIG-4P-2.0" device="'90D'"/>
-<part name="RN1" library="resistor-net" library_urn="urn:adsk.eagle:library:343" deviceset="RN08" device="" package3d_urn="urn:adsk.eagle:package:24977/1"/>
-<part name="RN2" library="resistor-net" library_urn="urn:adsk.eagle:library:343" deviceset="RN08" device="" package3d_urn="urn:adsk.eagle:package:24977/1"/>
+<part name="JG1" library="Connector" deviceset="TWIG-4P-2.0" device="'90D'" value="Grove/1"/>
+<part name="RN1" library="resistor-net" library_urn="urn:adsk.eagle:library:343" deviceset="RN08" device="" package3d_urn="urn:adsk.eagle:package:24977/1" value="10k"/>
+<part name="RN2" library="resistor-net" library_urn="urn:adsk.eagle:library:343" deviceset="RN08" device="" package3d_urn="urn:adsk.eagle:package:24977/1" value="10k"/>
 <part name="SUPPLY31" library="supply2" deviceset="GND" device=""/>
 <part name="SUPPLY32" library="supply2" deviceset="GND" device=""/>
+<part name="JG2" library="Connector" deviceset="TWIG-4P-2.0" device="'90D'" value="Grove/2"/>
 </parts>
 <sheets>
@@
 <instance part="SUPPLY28" gate="GND" x="154.94" y="106.68" smashed="yes"/>
 <instance part="SUPPLY30" gate="GND" x="175.26" y="106.68" smashed="yes"/>
-<instance part="JG1" gate="G$1" x="299.72" y="71.12" smashed="yes">
-<attribute name="NAME" x="298.45" y="76.2" size="1.27" layer="95"/>
-<attribute name="VALUE" x="302.26" y="67.31" size="1.27" layer="96" rot="R90"/>
+<instance part="JG1" gate="G$1" x="266.7" y="68.58" smashed="yes">
+<attribute name="NAME" x="265.43" y="73.66" size="1.27" layer="95"/>
+<attribute name="VALUE" x="269.24" y="64.77" size="1.27" layer="96" rot="R90"/>
 </instance>
 <instance part="RN1" gate="1" x="231.14" y="139.7" smashed="yes" rot="R90">
@@
 <instance part="SUPPLY31" gate="GND" x="231.14" y="127" smashed="yes"/>
 <instance part="SUPPLY32" gate="GND" x="246.38" y="127" smashed="yes"/>
+<instance part="JG2" gate="G$1" x="289.56" y="68.58" smashed="yes">
+<attribute name="NAME" x="288.29" y="73.66" size="1.27" layer="95"/>
+<attribute name="VALUE" x="292.1" y="64.77" size="1.27" layer="96" rot="R90"/>
+</instance>
 </instances>
 <busses>
@@
 <segment>
 <pinref part="JG1" gate="G$1" pin="4"/>
-<wire x1="295.91" y1="67.31" x2="289.56" y2="67.31" width="0.1524" layer="91"/>
-<label x="289.56" y="68.58" size="0.8128" layer="95"/>
+<wire x1="262.89" y1="64.77" x2="256.54" y2="64.77" width="0.1524" layer="91"/>
+<label x="256.54" y="66.04" size="0.8128" layer="95"/>
 </segment>
 <segment>
@@
 <wire x1="246.38" y1="134.62" x2="246.38" y2="129.54" width="0.1524" layer="91"/>
 <pinref part="SUPPLY32" gate="GND" pin="GND"/>
+</segment>
+<segment>
+<pinref part="JG2" gate="G$1" pin="4"/>
+<wire x1="285.75" y1="64.77" x2="279.4" y2="64.77" width="0.1524" layer="91"/>
+<label x="279.4" y="66.04" size="0.8128" layer="95"/>
 </segment>
 </net>
@@
 <segment>
 <pinref part="JG1" gate="G$1" pin="3"/>
-<wire x1="295.91" y1="69.85" x2="289.56" y2="69.85" width="0.1524" layer="91"/>
-<label x="284.48" y="71.12" size="0.8128" layer="95"/>
+<wire x1="262.89" y1="67.31" x2="256.54" y2="67.31" width="0.1524" layer="91"/>
+<label x="251.46" y="68.58" size="0.8128" layer="95"/>
+</segment>
+<segment>
+<pinref part="JG2" gate="G$1" pin="3"/>
+<wire x1="285.75" y1="67.31" x2="279.4" y2="67.31" width="0.1524" layer="91"/>
+<label x="274.32" y="68.58" size="0.8128" layer="95"/>
 </segment>
 </net>
@@
 <segment>
 <pinref part="JG1" gate="G$1" pin="2"/>
-<wire x1="295.91" y1="72.39" x2="289.56" y2="72.39" width="0.1524" layer="91"/>
-<label x="289.56" y="73.66" size="0.8128" layer="95"/>
+<wire x1="262.89" y1="69.85" x2="256.54" y2="69.85" width="0.1524" layer="91"/>
+<label x="256.54" y="71.12" size="0.8128" layer="95"/>
+</segment>
+<segment>
+<pinref part="JG2" gate="G$1" pin="2"/>
+<wire x1="285.75" y1="69.85" x2="279.4" y2="69.85" width="0.1524" layer="91"/>
+<label x="279.4" y="71.12" size="0.8128" layer="95"/>
 </segment>
 </net>
@@
 <segment>
 <pinref part="JG1" gate="G$1" pin="1"/>
-<wire x1="295.91" y1="74.93" x2="289.56" y2="74.93" width="0.1524" layer="91"/>
-<label x="289.56" y="76.2" size="0.8128" layer="95"/>
-</segment>
-</net>
+<wire x1="262.89" y1="72.39" x2="256.54" y2="72.39" width="0.1524" layer="91"/>
+<label x="256.54" y="73.66" size="0.8128" layer="95"/>
+</segment>
+<segment>
+<pinref part="JG2" gate="G$1" pin="1"/>
+<wire x1="285.75" y1="72.39" x2="279.4" y2="72.39" width="0.1524" layer="91"/>
+<label x="279.4" y="73.66" size="0.8128" layer="95"/>
+</segment>
+</net>
