File: Xvi/hardware/logicboard/pxvi-001.sch (EAGLE design)
At the start: 69 parts, among them J1 MKR, J5 SPI, J7 DIN5, Q1 60V/32A/35mΩ, Q10 60V/32A/35mΩ, Q11 60V/32A/35mΩ, Q12 60V/32A/35mΩ, Q13 60V/32A/35mΩ, Q14 60V/32A/35mΩ, Q15 60V/32A/35mΩ, Q16 60V/32A/35mΩ, Q2 60V/32A/35mΩ, Q3 60V/32A/35mΩ, Q4 60V/32A/35mΩ, Q5 60V/32A/35mΩ, Q6 60V/32A/35mΩ, Q7 60V/32A/35mΩ, Q8 60V/32A/35mΩ, Q9 60V/32A/35mΩ, U1 DS18B20, X1 ADAFRUIT-PCA9685

Commit message: Routed.
Parts:
- removed C10: 100n, rcl:C-EU025-024X044
- removed C11, C9: 100n, resistor:C-EU025-024X044
- removed C8: 10n, resistor:C-EU025-024X044
- removed F1: 1.8A, fuse:TE5
- removed JP1: PWRSEL, pinhead:PINHD-2X3
- removed R3: 1k, resistor:R-EU_0204/5
- removed RN2: 4.7k, resistor-net:RN04
Connections:
- removed net MIN: OK1A.VO1, RN2.2
- removed net N$10: X1.15
- removed net N$11: X1.16
- removed net N$12: X1.17
- removed net N$13: X1.18
- removed net N$14: X1.19
- removed net N$15: X1.20
- removed net N$16: X1.21
- removed net N$17: X1.22
- removed net N$18: X1.23
- removed net N$19: X1.24
- removed net N$20: X1.25
- removed net N$21: X1.26
- removed net N$22: X1.27
- removed net N$23: X1.28
- removed net N$8: X1.13
- removed net N$9: X1.14
- removed net NMO2RTN: RN2.5
- removed net NMORTN: RN2.4
- removed net NMTRTN: RN2.3
- removed net VCC/2: JP1.5, R3.2
- removed net VOUT: F1.2, JP1.4, JP1.6
- removed net VOUTRAW: C3.1, C4.1, D1.A, F1.1, V1.OUT
- net AREF: no longer C10.1, R3.1
- net GND: no longer C10.2, C11.2, C8.2, C9.2
- net MNTR: no longer RN3.5
- net PWM00: now also X1.13
- net PWM01: now also X1.14
- net PWM02: now also X1.15
- net PWM03: now also X1.16
- net PWM04: now also X1.17
- net PWM05: now also X1.18
- net PWM06: now also X1.19
- net PWM07: now also X1.20
- net PWM08: now also X1.21
- net PWM09: now also X1.22
- net PWM10: now also X1.23
- net PWM11: now also X1.24
- net PWM12: now also X1.25
- net PWM13: now also X1.26
- net PWM14: now also X1.27
- net PWM15: now also X1.28
- net RX: now also OK1A.VO1, RN3.5
- net V+: no longer JP1.1
- net VCC: now also C3.1, C4.1, D1.A, V1.OUT; no longer C11.1, C8.1, C9.1, JP1.3, RN2.1
- net VIN: no longer JP1.2
Other:
- moved on the sheet: C5

Commit message: Routed.
Parts:
- added X2: MKDSN1,5/2-5,08, con-phoenix-508:MKDSN1,5/2-5,08
- DD1, DD10, DD11, DD12, DD13, DD14, DD15, DD16, DD2, DD3, DD4, DD5, DD6, DD7, DD8, DD9: value 250mA/100V -> CGRM400-G; device SparkFun-DiscreteSemi:DIODE-BAS16J -> diode:CGRM4007-G
Connections:
- net GND: now also X2-2.KL
- net VCC: now also X2-1.KL

Commit message: Diodes -> back.
Parts:
- added DDUMMY: CGRM400-G, diode:CGRM4007-G
Connections:
- net GND: now also DDUMMY.A, DDUMMY.C
Changed lines of the file:
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@@
 <part name="P+18" library="supply1" library_urn="urn:adsk.eagle:library:371" deviceset="V+" device=""/>
 <part name="X2" library="con-phoenix-508" library_urn="urn:adsk.eagle:library:176" deviceset="MKDSN1,5/2-5,08" device="" package3d_urn="urn:adsk.eagle:package:9630/1"/>
+<part name="DDUMMY" library="diode" library_urn="urn:adsk.eagle:library:210" deviceset="CGRM400*-G" device="" package3d_urn="urn:adsk.eagle:package:43457/2" technology="7" value="CGRM400-G"/>
+<part name="SUPPLY33" library="supply2" deviceset="GND" device=""/>
 </parts>
 <sheets>
@@
 <attribute name="VALUE" x="114.3" y="191.897" size="1.778" layer="96"/>
 </instance>
+<instance part="DDUMMY" gate="G$1" x="248.92" y="30.48" smashed="yes" rot="R90">
+<attribute name="NAME" x="246.888" y="27.94" size="1.778" layer="95" font="vector" rot="R90"/>
+</instance>
+<instance part="SUPPLY33" gate="GND" x="248.92" y="7.62" smashed="yes"/>
 </instances>
 <busses>
@@
 <label x="88.9" y="68.58" size="0.8128" layer="95" xref="yes"/>
 </segment>
+<segment>
+<pinref part="DDUMMY" gate="G$1" pin="A"/>
+<wire x1="248.92" y1="27.94" x2="248.92" y2="25.4" width="0.1524" layer="91"/>
+<pinref part="DDUMMY" gate="G$1" pin="C"/>
+<wire x1="248.92" y1="25.4" x2="248.92" y2="10.16" width="0.1524" layer="91"/>
+<wire x1="248.92" y1="33.02" x2="248.92" y2="35.56" width="0.1524" layer="91"/>
+<wire x1="248.92" y1="35.56" x2="254" y2="35.56" width="0.1524" layer="91"/>
+<wire x1="254" y1="35.56" x2="254" y2="25.4" width="0.1524" layer="91"/>
+<wire x1="254" y1="25.4" x2="248.92" y2="25.4" width="0.1524" layer="91"/>
+<junction x="248.92" y="25.4"/>
+<pinref part="SUPPLY33" gate="GND" pin="GND"/>
+</segment>
 </net>

Commit message: Relay.
Parts:
- added C8: 10n, resistor:C-EU025-024X044
- added K1: G5V1, relay:G5V1
- added R2, R3: 1k, resistor:R-EU_0204/5
- added T1: 2SC1815, transistor:2SC1815
Connections:
- new net N$1: K11.2, T1.C
- new net N$2: R2.2, R3.2, T1.B
- new net N$4: K12.S, X2-2.KL
- net GND: now also C8.2, R3.1, T1.E, X2-1.KL; no longer X2-2.KL
- net RLY: now also R2.1
- net VCC: now also C8.1, K11.1, K12.P, K12.P@1; no longer X2-1.KL
Other:
- moved on the sheet: X2-1, X2-2
Changed lines of the file:
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@@
 <part name="DDUMMY" library="diode" library_urn="urn:adsk.eagle:library:210" deviceset="CGRM400*-G" device="" package3d_urn="urn:adsk.eagle:package:43457/2" technology="7" value="CGRM400-G"/>
 <part name="SUPPLY33" library="supply2" deviceset="GND" device=""/>
+<part name="T1" library="transistor" library_urn="urn:adsk.eagle:library:402" deviceset="2SC1815" device="" package3d_urn="urn:adsk.eagle:package:29929/2"/>
+<part name="K1" library="relay" library_urn="urn:adsk.eagle:library:339" deviceset="G5V1" device="" package3d_urn="urn:adsk.eagle:package:24341/1"/>
+<part name="SUPPLY34" library="supply2" library_urn="urn:adsk.eagle:library:372" deviceset="VCC" device=""/>
+<part name="SUPPLY35" library="supply2" deviceset="GND" device=""/>
+<part name="C8" library="resistor" library_urn="urn:adsk.eagle:library:348" deviceset="C-EU" device="025-024X044" package3d_urn="urn:adsk.eagle:package:23630/1" value="10n"/>
+<part name="SUPPLY36" library="supply2" deviceset="GND" device=""/>
+<part name="R2" library="resistor" library_urn="urn:adsk.eagle:library:348" deviceset="R-EU_" device="0204/5" package3d_urn="urn:adsk.eagle:package:23488/1" value="1k"/>
+<part name="R3" library="resistor" library_urn="urn:adsk.eagle:library:348" deviceset="R-EU_" device="0204/5" package3d_urn="urn:adsk.eagle:package:23488/1" value="1k"/>
+<part name="SUPPLY37" library="supply2" deviceset="GND" device=""/>
+<part name="SUPPLY38" library="supply2" library_urn="urn:adsk.eagle:library:372" deviceset="VCC" device=""/>
+<part name="SUPPLY39" library="supply2" deviceset="GND" device=""/>
 </parts>
 <sheets>
@@
 <attribute name="VALUE" x="233.68" y="43.18" size="1.778" layer="96"/>
 </instance>
-<instance part="X2" gate="-1" x="116.84" y="200.66" smashed="yes">
-<attribute name="NAME" x="119.888" y="199.771" size="1.778" layer="95"/>
-<attribute name="VALUE" x="114.3" y="196.977" size="1.778" layer="96"/>
-</instance>
-<instance part="X2" gate="-2" x="116.84" y="195.58" smashed="yes">
-<attribute name="NAME" x="119.888" y="194.691" size="1.778" layer="95"/>
-<attribute name="VALUE" x="114.3" y="191.897" size="1.778" layer="96"/>
+<instance part="X2" gate="-1" x="355.6" y="147.32" smashed="yes">
+<attribute name="NAME" x="358.648" y="146.431" size="1.778" layer="95"/>
+<attribute name="VALUE" x="353.06" y="143.637" size="1.778" layer="96"/>
+</instance>
+<instance part="X2" gate="-2" x="355.6" y="152.4" smashed="yes">
+<attribute name="NAME" x="358.648" y="151.511" size="1.778" layer="95"/>
+<attribute name="VALUE" x="353.06" y="148.717" size="1.778" layer="96"/>
 </instance>
 <instance part="DDUMMY" gate="G$1" x="248.92" y="30.48" smashed="yes" rot="R90">
@@
 </instance>
 <instance part="SUPPLY33" gate="GND" x="248.92" y="7.62" smashed="yes"/>
+<instance part="T1" gate="G$1" x="337.82" y="152.4" smashed="yes">
+<attribute name="NAME" x="327.66" y="160.02" size="1.778" layer="95"/>
+<attribute name="VALUE" x="327.66" y="157.48" size="1.778" layer="96"/>
+</instance>
+<instance part="K1" gate="1" x="340.36" y="165.1" smashed="yes">
+<attribute name="VALUE" x="341.63" y="168.021" size="1.778" layer="96"/>
+<attribute name="PART" x="341.63" y="170.18" size="1.778" layer="95"/>
+</instance>
+<instance part="K1" gate="2" x="358.14" y="162.56" smashed="yes">
+<attribute name="PART" x="360.68" y="162.56" size="1.778" layer="95"/>
+</instance>
+<instance part="SUPPLY34" gate="G$1" x="340.36" y="182.88" smashed="yes">
+<attribute name="VALUE" x="340.36" y="187.96" size="1.778" layer="96" align="bottom-center"/>
+</instance>
+<instance part="SUPPLY35" gate="GND" x="340.36" y="129.54" smashed="yes"/>
+<instance part="C8" gate="G$1" x="269.24" y="210.82" smashed="yes">
+<attribute name="NAME" x="266.7" y="210.82" size="1.778" layer="95" align="bottom-center"/>
+<attribute name="VALUE" x="266.7" y="205.74" size="1.778" layer="96" align="bottom-center"/>
+</instance>
+<instance part="SUPPLY36" gate="GND" x="269.24" y="198.12" smashed="yes"/>
+<instance part="R2" gate="G$1" x="325.12" y="152.4" smashed="yes">
+<attribute name="NAME" x="325.12" y="154.94" size="1.778" layer="95" align="center"/>
+<attribute name="VALUE" x="330.2" y="154.94" size="1.778" layer="96" align="center"/>
+</instance>
+<instance part="R3" gate="G$1" x="332.74" y="139.7" smashed="yes" rot="R90">
+<attribute name="NAME" x="330.2" y="139.7" size="1.778" layer="95" rot="R90" align="center"/>
+<attribute name="VALUE" x="330.2" y="144.78" size="1.778" layer="96" rot="R90" align="center"/>
+</instance>
+<instance part="SUPPLY37" gate="GND" x="332.74" y="129.54" smashed="yes"/>
+<instance part="SUPPLY38" gate="G$1" x="373.38" y="182.88" smashed="yes">
+<attribute name="VALUE" x="373.38" y="187.96" size="1.778" layer="96" align="bottom-center"/>
+</instance>
+<instance part="SUPPLY39" gate="GND" x="350.52" y="129.54" smashed="yes"/>
 </instances>
 <busses>
@@
 <junction x="63.5" y="187.96"/>
 <wire x1="45.72" y1="187.96" x2="63.5" y2="187.96" width="0.1524" layer="91"/>
-<pinref part="X2" gate="-2" pin="KL"/>
-<wire x1="114.3" y1="195.58" x2="111.76" y2="195.58" width="0.1524" layer="91"/>
-<wire x1="111.76" y1="195.58" x2="111.76" y2="187.96" width="0.1524" layer="91"/>
-<wire x1="111.76" y1="187.96" x2="99.06" y2="187.96" width="0.1524" layer="91"/>
-<junction x="99.06" y="187.96"/>
 </segment>
 <segment>
@@
 <junction x="248.92" y="25.4"/>
 <pinref part="SUPPLY33" gate="GND" pin="GND"/>
+</segment>
+<segment>
+<pinref part="T1" gate="G$1" pin="E"/>
+<wire x1="340.36" y1="147.32" x2="340.36" y2="132.08" width="0.1524" layer="91"/>
+<pinref part="SUPPLY35" gate="GND" pin="GND"/>
+</segment>
+<segment>
+<pinref part="C8" gate="G$1" pin="2"/>
+<wire x1="269.24" y1="205.74" x2="269.24" y2="200.66" width="0.1524" layer="91"/>
+<pinref part="SUPPLY36" gate="GND" pin="GND"/>
+</segment>
+<segment>
+<pinref part="R3" gate="G$1" pin="1"/>
+<wire x1="332.74" y1="134.62" x2="332.74" y2="132.08" width="0.1524" layer="91"/>
+<pinref part="SUPPLY37" gate="GND" pin="GND"/>
+</segment>
+<segment>
+<pinref part="X2" gate="-1" pin="KL"/>
+<wire x1="353.06" y1="147.32" x2="350.52" y2="147.32" width="0.1524" layer="91"/>
+<pinref part="SUPPLY39" gate="GND" pin="GND"/>
+<wire x1="350.52" y1="147.32" x2="350.52" y2="132.08" width="0.1524" layer="91"/>
 </segment>
 </net>
@@
 <junction x="241.3" y="220.98"/>
 <junction x="231.14" y="220.98"/>
+<wire x1="261.62" y1="220.98" x2="269.24" y2="220.98" width="0.1524" layer="91"/>
+<junction x="261.62" y="220.98"/>
+<pinref part="C8" gate="G$1" pin="1"/>
+<wire x1="269.24" y1="220.98" x2="269.24" y2="213.36" width="0.1524" layer="91"/>
 </segment>
 <segment>
@@
 <wire x1="99.06" y1="200.66" x2="99.06" y2="198.12" width="0.1524" layer="91"/>
 <wire x1="99.06" y1="243.84" x2="99.06" y2="200.66" width="0.1524" layer="91"/>
-<pinref part="X2" gate="-1" pin="KL"/>
-<wire x1="99.06" y1="200.66" x2="114.3" y2="200.66" width="0.1524" layer="91"/>
 </segment>
 <segment>
@@
 <wire x1="53.34" y1="139.7" x2="66.04" y2="139.7" width="0.1524" layer="91"/>
 </segment>
+<segment>
+<pinref part="SUPPLY34" gate="G$1" pin="VCC"/>
+<pinref part="K1" gate="1" pin="1"/>
+<wire x1="340.36" y1="180.34" x2="340.36" y2="170.18" width="0.1524" layer="91"/>
+</segment>
+<segment>
+<pinref part="K1" gate="2" pin="P@1"/>
+<wire x1="355.6" y1="160.02" x2="355.6" y2="157.48" width="0.1524" layer="91"/>
+<wire x1="355.6" y1="157.48" x2="358.14" y2="157.48" width="0.1524" layer="91"/>
+<pinref part="SUPPLY38" gate="G$1" pin="VCC"/>
+<wire x1="358.14" y1="157.48" x2="373.38" y2="157.48" width="0.1524" layer="91"/>
+<wire x1="373.38" y1="157.48" x2="373.38" y2="180.34" width="0.1524" layer="91"/>
+<pinref part="K1" gate="2" pin="P"/>
+<wire x1="358.14" y1="160.02" x2="358.14" y2="157.48" width="0.1524" layer="91"/>
+<junction x="358.14" y="157.48"/>
+</segment>
 </net>
 <net name="RST" class="0">
@@
 <wire x1="347.98" y1="93.98" x2="350.52" y2="93.98" width="0.1524" layer="91"/>
 <label x="350.52" y="93.98" size="0.8128" layer="95" xref="yes"/>
+</segment>
+<segment>
+<pinref part="R2" gate="G$1" pin="1"/>
+<wire x1="320.04" y1="152.4" x2="317.5" y2="152.4" width="0.1524" layer="91"/>
+<label x="317.5" y="152.4" size="0.8128" layer="95" rot="R180" xref="yes"/>
 </segment>
 </net>
@@
 </segment>
 </net>
+<net name="N$1" class="0">
+<segment>
+<pinref part="K1" gate="1" pin="2"/>
+<pinref part="T1" gate="G$1" pin="C"/>
+<wire x1="340.36" y1="160.02" x2="340.36" y2="157.48" width="0.1524" layer="91"/>
+</segment>
+</net>
+<net name="N$2" class="0">
+<segment>
+<pinref part="T1" gate="G$1" pin="B"/>
+<wire x1="335.28" y1="152.4" x2="332.74" y2="152.4" width="0.1524" layer="91"/>
+<pinref part="R2" gate="G$1" pin="2"/>
+<pinref part="R3" gate="G$1" pin="2"/>
+<wire x1="332.74" y1="152.4" x2="330.2" y2="152.4" width="0.1524" layer="91"/>
+<wire x1="332.74" y1="152.4" x2="332.74" y2="144.78" width="0.1524" layer="91"/>
+<junction x="332.74" y="152.4"/>
+</segment>
+</net>
+<net name="N$4" class="0">
+<segment>
+<pinref part="X2" gate="-2" pin="KL"/>
+<wire x1="353.06" y1="152.4" x2="350.52" y2="152.4" width="0.1524" layer="91"/>
+<wire x1="350.52" y1="152.4" x2="350.52" y2="167.64" width="0.1524" layer="91"/>
+<pinref part="K1" gate="2" pin="S"/>
+<wire x1="350.52" y1="167.64" x2="353.06" y2="167.64" width="0.1524" layer="91"/>
+</segment>
+</net>

Commit message: Qwiic con.
Parts:
- added J4, J6: QWIIC_RIGHT_ANGLE, SparkFun-Connectors:QWIIC_CONNECTORJS-1MM
Connections:
- net GND: now also J4.1, J6.1
- net SCL: now also J4.4, J6.4
- net SDA: now also J4.3, J6.3
- net VCC: now also J4.2, J6.2
Changed lines of the file:
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@@
 <layer number="56" name="wert" color="7" fill="1" visible="no" active="no"/>
 <layer number="57" name="tCAD" color="7" fill="1" visible="no" active="no"/>
+<layer number="58" name="bCAD" color="7" fill="1" visible="no" active="no"/>
 <layer number="59" name="tCarbon" color="7" fill="1" visible="no" active="no"/>
 <layer number="60" name="bCarbon" color="7" fill="1" visible="no" active="no"/>
@@
 <layer number="128" name="_bValues" color="7" fill="1" visible="yes" active="yes"/>
 <layer number="129" name="Mask" color="7" fill="1" visible="yes" active="yes"/>
+<layer number="130" name="SMDSTROOK" color="7" fill="1" visible="no" active="no"/>
 <layer number="131" name="tAdjust" color="7" fill="1" visible="no" active="yes"/>
 <layer number="132" name="bAdjust" color="7" fill="1" visible="no" active="yes"/>
+<layer number="133" name="bottom_silk" color="7" fill="1" visible="no" active="no"/>
+<layer number="134" name="silk_top" color="7" fill="1" visible="no" active="no"/>
+<layer number="135" name="silk_bottom" color="7" fill="1" visible="no" active="no"/>
+<layer number="136" name="silktop" color="7" fill="1" visible="no" active="no"/>
+<layer number="137" name="silkbottom" color="7" fill="1" visible="no" active="no"/>
+<layer number="138" name="EEE" color="7" fill="1" visible="no" active="no"/>
+<layer number="139" name="_tKeepout" color="7" fill="1" visible="no" active="no"/>
+<layer number="140" name="mbKeepout" color="7" fill="1" visible="no" active="no"/>
+<layer number="141" name="ASSEMBLY_TOP" color="7" fill="1" visible="no" active="no"/>
+<layer number="142" name="mbRestrict" color="7" fill="1" visible="no" active="no"/>
+<layer number="143" name="PLACE_BOUND_TOP" color="7" fill="1" visible="no" active="no"/>
 <layer number="144" name="Drill_legend" color="7" fill="1" visible="yes" active="yes"/>
+<layer number="145" name="DrillLegend_01-16" color="7" fill="1" visible="no" active="no"/>
+<layer number="146" name="DrillLegend_01-20" color="7" fill="1" visible="no" active="no"/>
+<layer number="147" name="PIN_NUMBER" color="7" fill="1" visible="no" active="no"/>
+<layer number="148" name="DrillLegend_01-20" color="7" fill="1" visible="no" active="no"/>
+<layer number="149" name="DrillLegend_02-15" color="7" fill="1" visible="no" active="no"/>
 <layer number="150" name="Notes" color="7" fill="1" visible="no" active="yes"/>
 <layer number="151" name="HeatSink" color="7" fill="1" visible="yes" active="yes"/>
@@
 <layer number="154" name="FabDoc2" color="2" fill="1" visible="no" active="no"/>
 <layer number="155" name="FabDoc3" color="7" fill="15" visible="no" active="no"/>
+<layer number="156" name="gesam-Maß" color="7" fill="1" visible="no" active="no"/>
+<layer number="157" name="FaceMchng" color="7" fill="1" visible="no" active="no"/>
+<layer number="158" name="FaceMMeas" color="7" fill="1" visible="no" active="no"/>
+<layer number="159" name="Geh-Bear2" color="7" fill="1" visible="no" active="no"/>
+<layer number="160" name="Topologie" color="7" fill="1" visible="no" active="no"/>
+<layer number="161" name="tomplace2" color="7" fill="1" visible="no" active="no"/>
+<layer number="166" name="AntennaArea" color="7" fill="1" visible="no" active="no"/>
+<layer number="168" name="4mmHeightArea" color="7" fill="1" visible="no" active="no"/>
+<layer number="191" name="mNets" color="7" fill="1" visible="no" active="no"/>
+<layer number="192" name="mBusses" color="7" fill="1" visible="no" active="no"/>
+<layer number="193" name="mPins" color="7" fill="1" visible="no" active="no"/>
+<layer number="194" name="mSymbols" color="7" fill="1" visible="no" active="no"/>
+<layer number="195" name="mNames" color="7" fill="1" visible="no" active="no"/>
+<layer number="196" name="mValues" color="7" fill="1" visible="no" active="no"/>
 <layer number="199" name="Contour" color="7" fill="1" visible="yes" active="yes"/>
 <layer number="200" name="200bmp" color="1" fill="10" visible="yes" active="yes"/>
@@
 <layer number="250" name="Descript" color="7" fill="1" visible="no" active="no"/>
 <layer number="251" name="SMDround" color="7" fill="1" visible="no" active="no"/>
+<layer number="252" name="BR-BS" color="7" fill="1" visible="no" active="no"/>
+<layer number="253" name="Extra" color="7" fill="1" visible="no" active="no"/>
 <layer number="254" name="cooling" color="7" fill="1" visible="yes" active="yes"/>
 <layer number="255" name="routoute" color="7" fill="1" visible="yes" active="yes"/>
@@
 <part name="SUPPLY38" library="supply2" library_urn="urn:adsk.eagle:library:372" deviceset="VCC" device=""/>
 <part name="SUPPLY39" library="supply2" deviceset="GND" device=""/>
+<part name="J4" library="SparkFun-Connectors" library_urn="urn:adsk.eagle:library:513" deviceset="QWIIC_CONNECTOR" device="JS-1MM" package3d_urn="urn:adsk.eagle:package:41390393/1" value="QWIIC_RIGHT_ANGLE"/>
+<part name="J6" library="SparkFun-Connectors" library_urn="urn:adsk.eagle:library:513" deviceset="QWIIC_CONNECTOR" device="JS-1MM" package3d_urn="urn:adsk.eagle:package:41390393/1" value="QWIIC_RIGHT_ANGLE"/>
+<part name="SUPPLY40" library="supply2" library_urn="urn:adsk.eagle:library:372" deviceset="VCC" device=""/>
+<part name="SUPPLY41" library="supply2" deviceset="GND" device=""/>
 </parts>
 <sheets>
@@
 </instance>
 <instance part="SUPPLY39" gate="GND" x="350.52" y="129.54" smashed="yes"/>
+<instance part="J4" gate="J1" x="215.9" y="139.7" smashed="yes">
+<attribute name="VALUE" x="210.82" y="134.366" size="1.778" layer="96" font="vector" align="top-left"/>
+<attribute name="NAME" x="210.82" y="147.574" size="1.778" layer="95" font="vector"/>
+</instance>
+<instance part="J6" gate="J1" x="215.9" y="116.84" smashed="yes">
+<attribute name="VALUE" x="210.82" y="111.506" size="1.778" layer="96" font="vector" align="top-left"/>
+<attribute name="NAME" x="210.82" y="124.714" size="1.778" layer="95" font="vector"/>
+</instance>
+<instance part="SUPPLY40" gate="G$1" x="246.38" y="149.86" smashed="yes">
+<attribute name="VALUE" x="246.38" y="154.94" size="1.778" layer="96" align="bottom-center"/>
+</instance>
+<instance part="SUPPLY41" gate="GND" x="246.38" y="132.08" smashed="yes"/>
 </instances>
 <busses>
@@
 <wire x1="350.52" y1="147.32" x2="350.52" y2="132.08" width="0.1524" layer="91"/>
 </segment>
+<segment>
+<pinref part="J4" gate="J1" pin="1"/>
+<wire x1="223.52" y1="137.16" x2="233.68" y2="137.16" width="0.1524" layer="91"/>
+<wire x1="233.68" y1="137.16" x2="246.38" y2="137.16" width="0.1524" layer="91"/>
+<wire x1="246.38" y1="137.16" x2="246.38" y2="134.62" width="0.1524" layer="91"/>
+<pinref part="J6" gate="J1" pin="1"/>
+<wire x1="223.52" y1="114.3" x2="233.68" y2="114.3" width="0.1524" layer="91"/>
+<wire x1="233.68" y1="114.3" x2="233.68" y2="137.16" width="0.1524" layer="91"/>
+<junction x="233.68" y="137.16"/>
+<pinref part="SUPPLY41" gate="GND" pin="GND"/>
+</segment>
 </net>
 <net name="VCC" class="2">
@@
 <junction x="358.14" y="157.48"/>
 </segment>
+<segment>
+<pinref part="J4" gate="J1" pin="2"/>
+<wire x1="223.52" y1="139.7" x2="231.14" y2="139.7" width="0.1524" layer="91"/>
+<pinref part="J6" gate="J1" pin="2"/>
+<wire x1="223.52" y1="116.84" x2="231.14" y2="116.84" width="0.1524" layer="91"/>
+<wire x1="231.14" y1="116.84" x2="231.14" y2="139.7" width="0.1524" layer="91"/>
+<junction x="231.14" y="139.7"/>
+<wire x1="231.14" y1="139.7" x2="246.38" y2="139.7" width="0.1524" layer="91"/>
+<wire x1="246.38" y1="139.7" x2="246.38" y2="147.32" width="0.1524" layer="91"/>
+<pinref part="SUPPLY40" gate="G$1" pin="VCC"/>
+</segment>
 </net>
 <net name="RST" class="0">
@@
 <label x="88.9" y="63.5" size="0.8128" layer="95" xref="yes"/>
 </segment>
+<segment>
+<pinref part="J4" gate="J1" pin="3"/>
+<wire x1="223.52" y1="142.24" x2="228.6" y2="142.24" width="0.1524" layer="91"/>
+<pinref part="J6" gate="J1" pin="3"/>
+<wire x1="228.6" y1="142.24" x2="238.76" y2="142.24" width="0.1524" layer="91"/>
+<wire x1="228.6" y1="142.24" x2="228.6" y2="119.38" width="0.1524" layer="91"/>
+<wire x1="228.6" y1="119.38" x2="223.52" y2="119.38" width="0.1524" layer="91"/>
+<junction x="228.6" y="142.24"/>
+<label x="238.76" y="142.24" size="0.8128" layer="95" xref="yes"/>
+</segment>
 </net>
 <net name="SCL" class="0">
@@
 <label x="88.9" y="60.96" size="0.8128" layer="95" xref="yes"/>
 </segment>
+<segment>
+<pinref part="J4" gate="J1" pin="4"/>
+<wire x1="223.52" y1="144.78" x2="226.06" y2="144.78" width="0.1524" layer="91"/>
+<pinref part="J6" gate="J1" pin="4"/>
+<wire x1="226.06" y1="144.78" x2="238.76" y2="144.78" width="0.1524" layer="91"/>
+<wire x1="223.52" y1="121.92" x2="226.06" y2="121.92" width="0.1524" layer="91"/>
+<wire x1="226.06" y1="121.92" x2="226.06" y2="144.78" width="0.1524" layer="91"/>
+<junction x="226.06" y="144.78"/>
+<label x="238.76" y="144.78" size="0.8128" layer="95" xref="yes"/>
+</segment>
 </net>
