File: Xvi/peripheral/candy/pcan-001.brd (EAGLE design)
At the start: 72 x 72 mm, 21 parts

Commit message: Optocoupler.
Parts:
- added JP1: Optorelay, pinhead:1X02
- added OK1: LTV816, optocoupler:DIL04
- added R1: 220, rcl:0204/5
Connections:
- new net N$17: OK1.1, R1.2
- new net N$19: JP1.2, OK1.3
- new net N$20: JP1.1, OK1.4
- net GND: now also OK1.2
- net MNTR: now also R1.1
Routing:
- net N$20: track 0.00 -> 53.8 mm
- net N$19: track 0.00 -> 50.9 mm
- net LD08: track 58.9 -> 75.2 mm
- net GND: track 0.00 -> 14.2 mm
- net VIN: track 148.6 -> 136.4 mm
- net N$15: track 68.9 -> 80.0 mm
- net LD03: track 66.2 -> 56.3 mm
- net N$11: track 35.0 -> 44.6 mm, vias 1 -> 0
- net MNTR: track 0.00 -> 8.59 mm
- net N$17: track 0.00 -> 8.53 mm
- net LD09: track 58.1 -> 64.0 mm
- net LD11: track 57.3 -> 63.2 mm
- net LD10: track 58.1 -> 62.3 mm
- net N$14: track 64.9 -> 60.9 mm, vias 0 -> 1
- net LD12: track 65.6 -> 62.2 mm
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
Commit message: Routing.
Routing:
- net LD15: track 57.3 -> 59.1 mm
Changed lines of the file:
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@@
 <contactref element="SV1" pad="31"/>
 <contactref element="RN2" pad="8"/>
-<wire x1="11.8872" y1="9.144" x2="6.2484" y2="9.144" width="0.1524" layer="1"/>
-<wire x1="13.4874" y1="10.7442" x2="11.8872" y2="9.144" width="0.1524" layer="1"/>
-<wire x1="52.197" y1="10.7442" x2="13.4874" y2="10.7442" width="0.1524" layer="1"/>
-<wire x1="59.6646" y1="18.2118" x2="52.197" y2="10.7442" width="0.1524" layer="1"/>
-<wire x1="6.2484" y1="9.144" x2="6.19" y2="9.11" width="0.1524" layer="1"/>
+<wire x1="59.6646" y1="18.2118" x2="51.4528" y2="10" width="0.1524" layer="1"/>
 <wire x1="59.6646" y1="18.2118" x2="59.73" y2="18.22" width="0.1524" layer="1"/>
+<wire x1="48" y1="10" x2="45" y2="7" width="0.1524" layer="1"/>
+<wire x1="51.4528" y1="10" x2="48" y2="10" width="0.1524" layer="1"/>
+<wire x1="8.3" y1="7" x2="6.19" y2="9.11" width="0.1524" layer="1"/>
+<wire x1="45" y1="7" x2="8.3" y2="7" width="0.1524" layer="1"/>
 </signal>
 <signal name="MNTR">
