File: Xvi/peripheral/candy/cndy-001.brd (EAGLE design)
At the start: 72 x 72 mm, 42 parts, among them K1 G5V1, T1 2SC1815

Commit message: Fixed some errors.
Parts:
- R1: value (none) -> 1k
- R2: value (none) -> 47k
- SV1: value (none) -> LightDrive
Changed lines of the file:
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@@
 <element name="LOGO1" library="SparkFun-Aesthetics" package="OSHW-LOGO-S_COPPER" value="OSHW-LOGOS-COPPER" x="36" y="62" smashed="yes"/>
 <element name="U$1" library="pineapple" package="PINEAPPLE450_SILK" value="PINEAPPLE450_SILK" x="36" y="8" smashed="yes"/>
-<element name="SV1" library="con-ml" library_urn="urn:adsk.eagle:library:164" package="ML34L" package3d_urn="urn:adsk.eagle:package:8689/1" value="" x="61" y="36" smashed="yes" rot="R270">
+<element name="SV1" library="con-ml" library_urn="urn:adsk.eagle:library:164" package="ML34L" package3d_urn="urn:adsk.eagle:package:8689/1" value="LightDrive" x="61" y="36" smashed="yes" rot="R270">
 <attribute name="MF" value="" x="61" y="36" size="1.778" layer="27" rot="R270" display="off"/>
 <attribute name="MPN" value="" x="61" y="36" size="1.778" layer="27" rot="R270" display="off"/>
@@
 <attribute name="VALUE" x="51.46" y="11.698" size="1.27" layer="27" ratio="10"/>
 </element>
-<element name="R1" library="rcl" library_urn="urn:adsk.eagle:library:334" package="0204/5" package3d_urn="urn:adsk.eagle:package:23488/1" value="" x="54" y="19" smashed="yes">
+<element name="R1" library="rcl" library_urn="urn:adsk.eagle:library:334" package="0204/5" package3d_urn="urn:adsk.eagle:package:23488/1" value="1k" x="54" y="19" smashed="yes">
 <attribute name="NAME" x="49" y="19" size="1" layer="25" ratio="10" align="center"/>
 <attribute name="POPULARITY" value="35" x="54" y="19" size="1.778" layer="27" display="off"/>
@@
 <attribute name="VALUE" x="51.8664" y="16.6886" size="0.9906" layer="27" ratio="10"/>
 </element>
-<element name="R2" library="rcl" library_urn="urn:adsk.eagle:library:334" package="0204/5" package3d_urn="urn:adsk.eagle:package:23488/1" value="" x="54" y="22" smashed="yes">
+<element name="R2" library="rcl" library_urn="urn:adsk.eagle:library:334" package="0204/5" package3d_urn="urn:adsk.eagle:package:23488/1" value="47k" x="54" y="22" smashed="yes">
 <attribute name="NAME" x="49" y="22" size="1" layer="25" ratio="10" align="center"/>
 <attribute name="POPULARITY" value="35" x="54" y="22" size="1.778" layer="27" display="off"/>
