File: Sweetio/hardware/logicboard/swt-001.brd (EAGLE design)
At the start: 91 x 90 mm, 44 parts, among them IC1 74ACT06N, J1 MKR, J10 THS, J16 MNTR, J2 GPIO, J5 SPI, J6 LED, J7 DIN5, J8 DIN5, J9 DIN5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

Commit message: Moved JP00.
Parts:
- added D4: (no value), SparkFun-DiscreteSemi:DIODE-1N4148
- moved JP00 14.2 mm to (6.00, 59.5), turned to 0 degrees
Connections:
- net N$2 renamed BASE
- net N$3 renamed COLLECTOR
- net SND renamed MNTRA
- removed net N$1: OK1.4, RN4.16
- removed net RTN: J16.1, OK1.3
- new net MNTRAA: D4.C, OK1.4, RN4.16
- new net MNTRK: D4.A, J16.1, OK1.3
Routing:
- net MNTRAA: track 0.00 -> 80.7 mm
- net VDD: track 354.6 -> 297.0 mm, vias 0 -> 4
- net TX: track 151.4 -> 95.1 mm, vias 1 -> 2
- net GPIO6: track 140.6 -> 94.9 mm, vias 3 -> 2
- net N$1: track 43.2 -> 0.00 mm
- net SCL: track 214.1 -> 172.2 mm, vias 4 -> 2
- net GPIO2: track 71.9 -> 110.0 mm, vias 2 -> 0
- net MNTRK: track 0.00 -> 30.0 mm
- net GND: track 451.3 -> 425.9 mm, vias 5 -> 3
- net NMORTN: track 110.5 -> 86.0 mm, vias 1 -> 4
- net RTN: track 22.4 -> 0.00 mm
- net DTCT0: track 65.8 -> 45.8 mm
- net GPIO8: track 89.4 -> 107.4 mm, vias 2 -> 0
- net NMO2RTN: track 137.0 -> 120.2 mm, vias 1 -> 2
- net SDA: track 179.3 -> 194.6 mm, vias 6 -> 4
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- added copper zone on layer 1, net GND
- added copper zone on layer 16, net GND
Other:
- board text added: "2-Grove"
- board text added: "4"
- board text added: "5"
- board text added: "74HCT05 (5V)"
- board text added: "A"
- board text added: "Configuration of X3"
- board text added: "Fan GND"
- board text added: "Fan Vcc"
- board text added: "Grove"
- board text added: "K"
- board text added: "LED0"
- board text added: "LED1"
- board text added: "MN"
- board text added: "OUT2"
- board text added: "RLY-A"
- board text added: "RLY-B"
- board text added: "Raspberry Pi Zero"
- board text added: "To RUN Pad (RPiZW2)"
- board text removed: "74HCT05"
- board text removed: "To RUN Pad"
- board text removed: "V+"

Commit message: RST switch.
Parts:
- removed JP6: LED, pinhead:1X03
- added LED0, LED1: (no value), led:CHIPLED_0603
- added S1: (no value), switch-omron:B3F-31XX
- moved LOGO1 1.00 mm to (45.5, 85.5)
- moved JP2 0.47 mm to (27.0, 40.0)
- moved H2 0.38 mm to (11.8, 50.2)
- moved H1 0.38 mm to (25.7, 36.2)
Connections:
- net GND: now also LED0.C, LED1.C, S1.1; no longer JP6.2
- net LED0A: now also LED0.A; no longer JP6.3
- net LED1A: now also LED1.A; no longer JP6.1
- net RST: now also S1.2
Routing:
- net GND: track 425.9 -> 0.00 mm, vias 3 -> 0
- net VDD: track 297.0 -> 0.00 mm, vias 4 -> 0
- net SDA: track 194.6 -> 0.00 mm, vias 4 -> 0
- net SCL: track 172.2 -> 0.00 mm, vias 2 -> 0
- net VCC: track 141.1 -> 0.00 mm, vias 2 -> 0
- net GPIO1: track 137.5 -> 0.00 mm, vias 3 -> 0
- net GPIO7: track 130.4 -> 0.00 mm
- net GPIO0: track 126.7 -> 0.00 mm, vias 4 -> 0
- net NMO2RTN: track 120.2 -> 0.00 mm, vias 2 -> 0
- net RX: track 118.1 -> 0.00 mm, vias 2 -> 0
- net NMTRTN: track 117.2 -> 0.00 mm, vias 2 -> 0
- net GPIO4: track 113.9 -> 0.00 mm, vias 2 -> 0
- net GPIO5: track 113.1 -> 0.00 mm, vias 2 -> 0
- net GPIO2: track 110.0 -> 0.00 mm
- net THS: track 109.6 -> 0.00 mm, vias 4 -> 0
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- removed copper zone on layer 1, net GND
- removed copper zone on layer 16, net GND
Other:
- board text added: "(2-1608)"
- board text added: "2-472"
- board text removed: "LED"

Commit message: RST Sw.
Routing:
- net GND: track 0.00 -> 471.9 mm, vias 0 -> 2
- net VDD: track 0.00 -> 316.9 mm, vias 0 -> 4
- net SDA: track 0.00 -> 198.7 mm, vias 0 -> 4
- net SCL: track 0.00 -> 170.2 mm, vias 0 -> 5
- net VCC: track 0.00 -> 145.2 mm, vias 0 -> 2
- net GPIO1: track 0.00 -> 140.4 mm, vias 0 -> 3
- net GPIO0: track 0.00 -> 140.3 mm, vias 0 -> 4
- net GPIO7: track 0.00 -> 124.9 mm, vias 0 -> 1
- net NMTRTN: track 0.00 -> 116.8 mm, vias 0 -> 1
- net RX: track 0.00 -> 116.5 mm, vias 0 -> 4
- net GPIO5: track 0.00 -> 109.1 mm, vias 0 -> 3
- net GPIO8: track 0.00 -> 107.4 mm
- net GPIO4: track 0.00 -> 106.9 mm, vias 0 -> 1
- net NMO2RTN: track 0.00 -> 106.2 mm, vias 0 -> 2
- net GPIO3: track 0.00 -> 104.3 mm, vias 0 -> 1
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