File: 0/hardware/logicboard/p0-001.brd (EAGLE design)
At the start: 91 x 57 mm, 31 parts, among them IC1 74ALS05N, IC2 LTC485N, IC3 LTC485N, J0 DC5V, J7 DIN5, J8 DIN5, J9 DIN5, X7 NELTRON-7810-XPXC, X9 NELTRON-7810-XPXC

Commit message: Silk.
Parts:
- moved D1 0.31 mm to (8.00, 20.0), turned to 180 degrees
Routing:
- net GND: track 213.7 -> 227.5 mm, vias 1 -> 0
- net MIRTN: track 88.6 -> 79.1 mm
- net VCC: track 149.3 -> 142.7 mm, vias 0 -> 2
- net N$1: track 66.0 -> 61.2 mm
- net NMIDIOUT: track 40.6 -> 36.3 mm
- net MISND: track 33.8 -> 30.1 mm, vias 0 -> 1
- net N$3: track 66.9 -> 68.0 mm
- net MIDITHRU: track 27.7 -> 28.8 mm, vias 1 -> 0
- net TX: track 88.0 -> 88.8 mm
- net MTSND: track 18.4 -> 17.6 mm
- net N$5: track 37.6 -> 38.2 mm
- net RX: track 51.3 -> 51.9 mm
Other:
- board text added: "L1"
- board text added: "L2"
- board text added: "L3"
- board text added: "Pineapple Zero 2.7.0-RC"
- board text added: "THR"
- board text removed: "Pineapple Zero 2.6.3-B"
