File: 0/hardware/logicboard/p0rx-001.brd (EAGLE design)
At the start: 91 x 57 mm, 23 parts, among them IC1 74ALS05N, IC2 LTC485N, IC3 LTC485N, IC4 LTC485N, J0 DC5V, J7 DIN5, J8 DIN5, J9 DIN5, X7 NELTRON-7810-XPXC

Commit message: Silk.
Connections:
- net MIRTN renamed MO1RTN
- net MORTN renamed MO3RTN
- net MTRTN renamed NO2RTN
- net N$10 renamed MO1SND
- net N$14 renamed MO2SND
- net N$15 renamed MO3SND
Changed lines of the file:
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@@
 <layer number="19" name="Unrouted" color="6" fill="1" visible="yes" active="yes"/>
 <layer number="20" name="Dimension" color="15" fill="1" visible="yes" active="yes"/>
-<layer number="21" name="tPlace" color="7" fill="1" visible="no" active="yes"/>
+<layer number="21" name="tPlace" color="7" fill="1" visible="yes" active="yes"/>
 <layer number="22" name="bPlace" color="7" fill="1" visible="yes" active="yes"/>
-<layer number="23" name="tOrigins" color="15" fill="1" visible="no" active="yes"/>
+<layer number="23" name="tOrigins" color="15" fill="1" visible="yes" active="yes"/>
 <layer number="24" name="bOrigins" color="15" fill="1" visible="yes" active="yes"/>
-<layer number="25" name="tNames" color="7" fill="1" visible="no" active="yes"/>
+<layer number="25" name="tNames" color="7" fill="1" visible="yes" active="yes"/>
 <layer number="26" name="bNames" color="7" fill="1" visible="yes" active="yes"/>
 <layer number="27" name="tValues" color="7" fill="1" visible="no" active="yes"/>
@@
 <wire x1="40.4622" y1="19.9644" x2="40.42" y2="20" width="0.3048" layer="16"/>
 </signal>
-<signal name="MIRTN">
+<signal name="MO1RTN">
 <contactref element="J7" pad="5"/>
 <contactref element="RN1" pad="2"/>
@@
 <wire x1="44.0436" y1="8.8392" x2="43.97" y2="8.8" width="0.1524" layer="1"/>
 </signal>
-<signal name="MTRTN">
+<signal name="NO2RTN">
 <contactref element="J8" pad="5"/>
 <contactref element="RN1" pad="4"/>
@@
 <wire x1="50.4444" y1="41.9862" x2="50.5" y2="42" width="0.1524" layer="1"/>
 </signal>
-<signal name="MORTN">
+<signal name="MO3RTN">
 <contactref element="J9" pad="5"/>
 <contactref element="RN1" pad="6"/>
@@
 <wire x1="66.5226" y1="19.9644" x2="66.54" y2="20" width="0.1524" layer="1"/>
 </signal>
-<signal name="N$10">
+<signal name="MO1SND">
 <contactref element="J7" pad="4"/>
 <contactref element="RN1" pad="1"/>
@@
 <wire x1="39.0906" y1="32.766" x2="39.15" y2="32.81" width="0.1524" layer="16"/>
 </signal>
-<signal name="N$14">
+<signal name="MO2SND">
 <contactref element="J8" pad="4"/>
 <contactref element="RN1" pad="3"/>
@@
 <wire x1="44.196" y1="32.8422" x2="44.23" y2="32.81" width="0.1524" layer="16"/>
 </signal>
-<signal name="N$15">
+<signal name="MO3SND">
 <contactref element="J9" pad="4"/>
 <contactref element="RN1" pad="5"/>

Commit message: Layout.
Parts:
- moved IC2 35.0 mm to (62.0, 29.0)
- moved C3 35.0 mm to (62.0, 36.0)
- moved R2 35.0 mm to (62.0, 20.0)
- moved IC1 13.0 mm to (24.0, 29.0)
- moved C2 13.0 mm to (24.0, 36.0)
- moved R1 13.0 mm to (24.0, 20.0)
- moved C4 9.00 mm to (73.0, 36.0)
- moved IC3 9.00 mm to (73.0, 29.0)
- moved R3 9.00 mm to (73.0, 20.0)
- moved C5 7.00 mm to (84.0, 36.0)
- moved IC4 7.00 mm to (84.0, 29.0)
- moved R4 7.00 mm to (84.0, 20.0)
Routing:
- net N$7: track 16.1 -> 55.0 mm
- net N$16: track 42.9 -> 18.3 mm
- net GND: track 225.1 -> 205.8 mm, vias 0 -> 1
- net N$1: track 48.8 -> 30.0 mm, vias 1 -> 0
- net N$8: track 46.9 -> 28.4 mm
- net RX+: track 48.6 -> 66.0 mm
- net N$2: track 48.0 -> 30.8 mm
- net N$11: track 38.3 -> 23.4 mm
- net N$17: track 47.4 -> 33.0 mm
- net N$3: track 44.3 -> 57.2 mm, vias 1 -> 0
- net N$12: track 32.4 -> 43.0 mm
- net MO3RTN: track 26.4 -> 36.8 mm
- net RX-: track 54.9 -> 65.2 mm
- net N$13: track 39.6 -> 49.0 mm
- net N$6: track 73.6 -> 66.8 mm, vias 1 -> 0
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
Commit message: Fixed layout.
Parts:
- moved IC1 0.50 mm to (24.0, 28.5)
- moved IC2 0.50 mm to (62.0, 28.5)
- moved IC3 0.50 mm to (73.0, 28.5)
- moved IC4 0.50 mm to (84.0, 28.5)
- moved RN1 0.50 mm to (45.5, 28.5)
- turned R2 to 180 degrees
- turned R3 to 180 degrees
- turned R4 to 180 degrees
Connections:
- net N$1 renamed RX1R
- net N$11 renamed MO1RTNRAW
- net N$12 renamed RX2+
- net N$13 renamed RX2-
- net N$16 renamed MO2RTNRAW
- net N$17 renamed MO3RTNRAW
- net N$18 renamed MNTRSND
- net N$19 renamed MNTRRTN
- net N$2 renamed RX2R
- net N$3 renamed RX3R
- net N$5 renamed RX3
- net N$6 renamed RX2
- net N$7 renamed RX1
- net N$8 renamed RX1+
- net N$9 renamed RX1-
- net RX+ renamed RX3+
- net RX- renamed RX3-
Routing:
- net GND: track 205.8 -> 219.7 mm, vias 1 -> 0
- net RX1: track 55.0 -> 42.4 mm, vias 0 -> 1
- net RX3: track 82.1 -> 70.6 mm
- net VCC: track 148.3 -> 138.4 mm, vias 0 -> 1
- net MO3RTNRAW: track 33.0 -> 25.0 mm, vias 0 -> 1
- net RX3+: track 66.0 -> 58.9 mm
- net RX3-: track 65.2 -> 58.6 mm
- net RX1-: track 35.5 -> 28.9 mm
- net RX2-: track 49.0 -> 42.7 mm
- net RX3R: track 57.2 -> 61.9 mm
- net RX1+: track 28.4 -> 31.9 mm
- net MO3SND: track 34.5 -> 37.8 mm
- net RX2+: track 43.0 -> 45.3 mm
- net MO1SND: track 34.8 -> 35.7 mm
- net RX2: track 66.8 -> 67.5 mm

Commit message: Redesign.
Parts:
- added C6, C7: 10n, rcl:C025-024X044
- added IC5, IC6: 74ALS05N, 74xx-us:DIL14
- added J10: DIN5, SparkFun-Connectors:DIN5-RA-PTH
- added R5: 100, rcl:0204/5
- IC1: value 74ALS05N -> LTC485N; device 74xx-us:DIL14 -> linear-technology:DIL08
- moved IC4 55.0 mm to (29.0, 28.5)
- moved IC1 38.0 mm to (62.0, 28.5)
- moved C2 19.9 mm to (18.0, 17.0)
- moved U$1 13.5 mm to (78.5, -3.00)
- moved IC2 11.0 mm to (73.0, 28.5)
- moved IC3 11.0 mm to (84.0, 28.5)
- moved R1 5.22 mm to (29.0, 18.5)
- moved R2 1.50 mm to (62.0, 21.5)
- moved R3 1.50 mm to (73.0, 21.5)
- moved R4 1.50 mm to (84.0, 21.5)
Connections:
- removed net MNTRRTN: RN1.9, X7.8
- removed net MNTRSND: RN1.10, X7.7
- new net MO4RTN: J10.5, RN1.8
- new net MO4SND: J10.4, RN1.7
- new net N$1: IC6.1, IC6.4, RN2.5
- new net N$2: IC4.1, IC6.3
- new net N$3: IC4.6, R5.1, X7.7
- new net N$5: IC4.7, R5.2, X7.8
- new net N$6: IC6.2, RN1.9
- net GND: now also C6.2, C7.2, IC1.2, IC1.3, IC1.4, IC1.5, IC5.7, IC6.11, IC6.13, IC6.5, IC6.7, IC6.9, J10.2; no longer IC1.7, RN1.8
- net MO1RTNRAW: now also IC5.2; no longer IC1.2
- net MO2RTNRAW: now also IC5.6; no longer IC1.6
- net MO3RTNRAW: now also IC5.10; no longer IC1.10
- net RX1: now also IC1.1, IC5.3; no longer IC1.3, IC2.1
- net RX1+: now also IC1.6; no longer IC2.6
- net RX1-: now also IC1.7; no longer IC2.7
- net RX1R: now also IC5.1, IC5.4; no longer IC1.1, IC1.4
- net RX2: now also IC2.1, IC5.13; no longer IC1.13, IC3.1
- net RX2+: now also IC2.6; no longer IC3.6
- net RX2-: now also IC2.7; no longer IC3.7
- net RX2R: now also IC5.12, IC5.5; no longer IC1.12, IC1.5
- net RX3: now also IC3.1, IC5.9; no longer IC1.9, IC4.1
- net RX3+: now also IC3.6; no longer IC4.6
- net RX3-: now also IC3.7; no longer IC4.7
- net RX3R: now also IC5.11, IC5.8; no longer IC1.11, IC1.8
- net VCC: now also C6.1, C7.1, IC1.8, IC5.14, IC6.14, RN1.10; no longer IC1.14, RN1.7
Routing:
- net GND: track 219.7 -> 0.00 mm
- net VCC: track 138.4 -> 0.00 mm, vias 1 -> 0
- net RX3: track 70.6 -> 0.00 mm
- net RX2: track 67.5 -> 0.00 mm
- net RX3R: track 61.9 -> 0.00 mm
- net RX3+: track 58.9 -> 0.00 mm
- net RX3-: track 58.6 -> 0.00 mm
- net RX2+: track 45.3 -> 0.00 mm
- net MO1RTN: track 43.8 -> 0.00 mm
- net RX2-: track 42.7 -> 0.00 mm
- net RX1: track 42.4 -> 0.00 mm, vias 1 -> 0
- net MO3SND: track 37.8 -> 0.00 mm, vias 1 -> 0
- net MO3RTN: track 36.7 -> 0.00 mm
- net MO1SND: track 35.7 -> 0.00 mm
- net RX1+: track 31.9 -> 0.00 mm
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- removed copper zone on layer 1, net GND
- removed copper zone on layer 16, net GND

Commit message: RX indicators.
Parts:
- added LED2, LED3, LED4, LED5: BLUE, led:LED3MM
- added R6, R7, R8, R9: 100, rcl:0204/5
- moved LOGO1 40.4 mm to (19.0, 5.00)
- moved RN2 1.50 mm to (45.5, 21.5)
- moved C3 0.50 mm to (62.0, 35.5)
- moved C4 0.50 mm to (73.0, 35.5)
- moved C5 0.50 mm to (84.0, 35.5)
- moved C6 0.50 mm to (29.0, 35.5)
Connections:
- new net N$10: LED5.A, R9.1
- new net N$11: IC6.6, LED2.K
- new net N$12: IC6.8, LED3.K
- new net N$13: IC6.10, LED4.K
- new net N$14: IC6.12, LED5.K
- new net N$7: LED2.A, R6.1
- new net N$8: LED3.A, R7.1
- new net N$9: LED4.A, R8.1
- net GND: no longer IC6.11, IC6.13, IC6.5, IC6.9
- net N$1: now also IC6.13
- net RX1R: now also IC6.5
- net RX2R: now also IC6.9
- net RX3R: now also IC6.11
- net VCC: now also R6.2, R7.2, R8.2, R9.2
Routing:
- net GND: track 0.00 -> 255.8 mm, vias 0 -> 2
- net VCC: track 0.00 -> 178.8 mm, vias 0 -> 2
- net N$1: track 0.00 -> 84.3 mm, vias 0 -> 1
- net RX2: track 0.00 -> 77.8 mm
- net RX3: track 0.00 -> 72.6 mm
- net RX1: track 0.00 -> 71.0 mm
- net RX3+: track 0.00 -> 70.9 mm
- net N$12: track 0.00 -> 69.2 mm, vias 0 -> 1
- net RX1R: track 0.00 -> 69.0 mm, vias 0 -> 2
- net N$6: track 0.00 -> 67.6 mm, vias 0 -> 1
- net N$11: track 0.00 -> 59.9 mm, vias 0 -> 2
- net RX3-: track 0.00 -> 56.6 mm
- net MO1SND: track 0.00 -> 54.0 mm, vias 0 -> 1
- net RX3R: track 0.00 -> 51.9 mm
- net N$13: track 0.00 -> 51.8 mm
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
Commit message: Layout.
Parts:
- R1, R6, R7, R8, R9: value 100 -> 102
- R2, R3, R4, R5: value 100 -> 101
- RN1: value (none) -> 221
- moved U$1 43.4 mm to (84.0, 40.0)
Other:
- board text added: "103"
- board text added: "2-7406"
- board text added: "MIDI OUT4"
- board text added: "OUT4"
- board text removed: "7406"
