File: 0/hardware/logicboard/p0tx-001.brd (EAGLE design)
At the start: 91 x 57 mm, 33 parts, among them IC1 LTC485N, IC2 LTC485N, IC3 LTC485N, J0 DC5V, J7 DIN5, J8 DIN5, J9 DIN5, X9 NELTRON-7810-XPXC

Commit message: Redesign.
Parts:
- removed LED2: YELLOW, led:LED3MM
- added C7: 10n, rcl:C025-024X044
- added IC4: LTC485N, linear-technology:DIL08
- added J10: DIN5, SparkFun-Connectors:DIN5-RA-PTH
- moved U$1 12.0 mm to (66.0, -10.0)
- moved D3 5.00 mm to (19.0, 21.0)
- moved D4 5.00 mm to (19.0, 18.5)
- moved OK2 5.00 mm to (19.0, 28.5)
- moved C3 4.00 mm to (20.0, 36.0)
- moved C2 1.00 mm to (7.00, 36.0)
- moved D1 1.00 mm to (7.00, 21.0)
- moved D2 1.00 mm to (7.00, 18.5)
- moved OK1 1.00 mm to (7.00, 28.5)
Connections:
- removed net MNTRRTN: D4.A, OK2.3, X9.8
- removed net MNTRSND: R4.1, X9.7
- removed net N$11: LED2.K, OK2.6
- removed net N$12: LED2.A, R6L2.1
- new net MI4RTN: D4.A, J10.5, OK2.3
- new net MI4SND: J10.4, R4.1
- new net N$6: IC4.4, OK2.6, RN2.5
- new net TX4+: IC4.6, X9.7
- new net TX4-: IC4.7, X9.8
- net GND: now also C7.2, IC4.5
- net VCC: now also C7.1, IC4.2, IC4.3, IC4.8; no longer R6L2.2
Routing:
- net GND: track 179.2 -> 0.00 mm, vias 1 -> 0
- net VCC: track 165.5 -> 0.00 mm
- net TX: track 95.7 -> 0.00 mm, vias 1 -> 0
- net N$5: track 95.5 -> 0.00 mm, vias 1 -> 0
- net N$10: track 85.9 -> 0.00 mm, vias 1 -> 0
- net MI1RTN: track 76.0 -> 0.00 mm
- net N$11: track 73.5 -> 0.00 mm
- net MI2RTN: track 56.9 -> 0.00 mm
- net TX3+: track 55.4 -> 0.00 mm, vias 1 -> 0
- net TX3-: track 52.9 -> 0.00 mm
- net N$12: track 46.9 -> 0.00 mm
- net N$7: track 46.2 -> 0.00 mm, vias 1 -> 0
- net TX2+: track 43.7 -> 0.00 mm
- net N$4: track 41.6 -> 0.00 mm
- net TX2-: track 39.1 -> 0.00 mm
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- removed copper zone on layer 1, net GND
- removed copper zone on layer 16, net GND
Other:
- board text removed: "CON"
- board text removed: "YLW"

Commit message: Layout.
Parts:
- removed R2, R3, R4: 220, rcl:0204/5
- removed R5L1, R6L2, R7X, R8X: 1k, rcl:0204/5
- added RN1: 221, resistor-dil:DIL16
- R1: value 220 -> 1k
- moved U$1 53.1 mm to (84.0, 40.0)
- moved LOGO1 40.4 mm to (19.0, 5.00)
- moved R1 12.6 mm to (29.0, 18.5), turned to 0 degrees
- moved C3 2.00 mm to (18.0, 36.0)
- moved C7 1.12 mm to (29.0, 35.5)
- moved IC4 1.00 mm to (29.0, 28.5)
- moved OK2 1.00 mm to (18.0, 28.5)
- moved RN2 1.00 mm to (45.5, 21.0)
- moved C2 0.50 mm to (6.50, 36.0)
- moved C4 0.50 mm to (62.0, 35.5)
- moved C5 0.50 mm to (73.0, 35.5)
- moved C6 0.50 mm to (84.0, 35.5)
- moved OK1 0.50 mm to (6.50, 28.5)
Connections:
- net MI1SND: now also RN1.1; no longer R1.1
- net MI2SND: now also RN1.2; no longer R2.1
- net MI3SND: now also RN1.3; no longer R3.1
- net MI4SND: now also RN1.4; no longer R4.1
- net MIDIIN: now also RN1.16; no longer R1.2
- net N$1: now also RN1.13; no longer R4.2
- net N$4: now also R1.1; no longer R5L1.1
- net N$7: now also RN1.15; no longer R2.2
- net N$8: now also RN1.14; no longer R3.2
- net VCC: now also R1.2; no longer R5L1.2
Routing:
- net GND: track 0.00 -> 182.5 mm
- net VCC: track 0.00 -> 172.7 mm
- net N$10: track 0.00 -> 98.5 mm, vias 0 -> 1
- net N$5: track 0.00 -> 86.5 mm, vias 0 -> 1
- net MI1RTN: track 0.00 -> 85.1 mm
- net TX: track 0.00 -> 80.1 mm, vias 0 -> 2
- net MI2RTN: track 0.00 -> 79.9 mm
- net TX3+: track 0.00 -> 59.0 mm
- net N$7: track 0.00 -> 57.1 mm
- net TX3-: track 0.00 -> 57.0 mm
- net MI4RTN: track 0.00 -> 55.1 mm
- net MIDIIN: track 0.00 -> 53.2 mm
- net TX2+: track 0.00 -> 48.8 mm
- net N$1: track 0.00 -> 42.6 mm, vias 0 -> 1
- net N$8: track 0.00 -> 41.9 mm
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Other:
- board text added: "4-LCT485"
- board text added: "IN4"
- board text added: "MIDI IN4"
- board text removed: "102"
- board text removed: "3-LCT485"
