File: 0/hardware/logicboard/p0rx-001.sch (EAGLE design)
At the start: 23 parts, among them IC1 74ALS05N, IC2 LTC485N, IC3 LTC485N, IC4 LTC485N, J0 DC5V, J7 DIN5, J8 DIN5, J9 DIN5, X7 NELTRON-7810-XPXC

Commit message: Silk.
Connections:
- net MIRTN renamed MO1RTN
- net MORTN renamed MO3RTN
- net MTRTN renamed NO2RTN
- net N$10 renamed MO1SND
- net N$14 renamed MO2SND
- net N$15 renamed MO3SND
Other:
- note added: "MIDI IN1"
- note added: "MIDI IN2"
- note added: "MIDI IN3"
- note removed: "MIDI IN"
- note removed: "MIDI OUT"
- note removed: "MIDI THRU"
Changed lines of the file:
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@@
 <plain>
 <text x="215.9" y="20.32" size="1.778" layer="94">Pineapple Zero 1.2.0</text>
-<text x="35.56" y="114.3" size="1.778" layer="94">MIDI IN</text>
-<text x="35.56" y="83.82" size="1.778" layer="94">MIDI THRU</text>
-<text x="35.56" y="53.34" size="1.778" layer="94">MIDI OUT</text>
+<text x="35.56" y="114.3" size="1.778" layer="94">MIDI IN1</text>
+<text x="35.56" y="83.82" size="1.778" layer="94">MIDI IN2</text>
+<text x="35.56" y="53.34" size="1.778" layer="94">MIDI IN3</text>
 </plain>
 <instances>
@@
 <attribute name="VALUE" x="84.455" y="107.315" size="1.778" layer="96"/>
 </instance>
-<instance part="SUPPLY22" gate="GND" x="7.62" y="86.36" smashed="yes">
-<attribute name="VALUE" x="5.715" y="83.185" size="1.778" layer="96"/>
-</instance>
-<instance part="SUPPLY23" gate="GND" x="7.62" y="48.26" smashed="yes">
-<attribute name="VALUE" x="5.715" y="45.085" size="1.778" layer="96"/>
+<instance part="SUPPLY22" gate="GND" x="7.62" y="91.44" smashed="yes">
+<attribute name="VALUE" x="5.715" y="88.265" size="1.778" layer="96"/>
+</instance>
+<instance part="SUPPLY23" gate="GND" x="7.62" y="60.96" smashed="yes">
+<attribute name="VALUE" x="5.715" y="57.785" size="1.778" layer="96"/>
 </instance>
 <instance part="RN2" gate="1" x="93.98" y="157.48" smashed="yes" rot="R270">
@@
 <attribute name="VALUE" x="81.915" y="135.255" size="1.778" layer="96"/>
 </instance>
-<instance part="SUPPLY33" gate="GND" x="7.62" y="116.84" smashed="yes">
-<attribute name="VALUE" x="5.715" y="113.665" size="1.778" layer="96"/>
+<instance part="SUPPLY33" gate="GND" x="7.62" y="119.38" smashed="yes">
+<attribute name="VALUE" x="5.715" y="116.205" size="1.778" layer="96"/>
 </instance>
 <instance part="RN1" gate="A" x="76.2" y="127" smashed="yes">
@@
 <pinref part="SUPPLY22" gate="GND" pin="GND"/>
 <wire x1="25.4" y1="106.68" x2="7.62" y2="106.68" width="0.1524" layer="91"/>
-<wire x1="7.62" y1="106.68" x2="7.62" y2="88.9" width="0.1524" layer="91"/>
+<wire x1="7.62" y1="106.68" x2="7.62" y2="93.98" width="0.1524" layer="91"/>
 </segment>
 <segment>
@@
 <wire x1="25.4" y1="73.66" x2="25.4" y2="76.2" width="0.1524" layer="91"/>
 <wire x1="25.4" y1="76.2" x2="7.62" y2="76.2" width="0.1524" layer="91"/>
-<wire x1="7.62" y1="76.2" x2="7.62" y2="50.8" width="0.1524" layer="91"/>
+<wire x1="7.62" y1="76.2" x2="7.62" y2="63.5" width="0.1524" layer="91"/>
 <pinref part="SUPPLY23" gate="GND" pin="GND"/>
 </segment>
@@
 <wire x1="25.4" y1="132.08" x2="25.4" y2="134.62" width="0.1524" layer="91"/>
 <wire x1="25.4" y1="134.62" x2="7.62" y2="134.62" width="0.1524" layer="91"/>
-<wire x1="7.62" y1="134.62" x2="7.62" y2="119.38" width="0.1524" layer="91"/>
+<wire x1="7.62" y1="134.62" x2="7.62" y2="121.92" width="0.1524" layer="91"/>
 <pinref part="SUPPLY33" gate="GND" pin="GND"/>
 </segment>
@@
 </segment>
 </net>
-<net name="MIRTN" class="0">
+<net name="MO1RTN" class="0">
 <segment>
 <pinref part="J7" gate="G$1" pin="5"/>
@@
 <wire x1="71.12" y1="121.92" x2="45.72" y2="121.92" width="0.1524" layer="91"/>
 <pinref part="RN1" gate="B" pin="1"/>
+<label x="48.26" y="121.92" size="1.778" layer="95"/>
 </segment>
 </net>
@@
 </segment>
 </net>
-<net name="MTRTN" class="0">
+<net name="NO2RTN" class="0">
 <segment>
 <pinref part="J8" gate="G$1" pin="5"/>
@@
 <wire x1="45.72" y1="93.98" x2="73.66" y2="93.98" width="0.1524" layer="91"/>
 <pinref part="RN1" gate="D" pin="1"/>
-</segment>
-</net>
-<net name="MORTN" class="0">
+<label x="48.26" y="93.98" size="1.778" layer="95"/>
+</segment>
+</net>
+<net name="MO3RTN" class="0">
 <segment>
 <pinref part="J9" gate="G$1" pin="5"/>
@@
 <wire x1="73.66" y1="63.5" x2="45.72" y2="63.5" width="0.1524" layer="91"/>
 <pinref part="RN1" gate="F" pin="1"/>
+<label x="48.26" y="63.5" size="1.778" layer="95"/>
 </segment>
 </net>
@@
 </segment>
 </net>
-<net name="N$10" class="0">
+<net name="MO1SND" class="0">
 <segment>
 <pinref part="J7" gate="G$1" pin="4"/>
 <wire x1="71.12" y1="127" x2="33.02" y2="127" width="0.1524" layer="91"/>
 <pinref part="RN1" gate="A" pin="1"/>
+<label x="48.26" y="127" size="1.778" layer="95"/>
 </segment>
 </net>
@@
 </segment>
 </net>
-<net name="N$14" class="0">
+<net name="MO2SND" class="0">
 <segment>
 <pinref part="J8" gate="G$1" pin="4"/>
 <wire x1="73.66" y1="99.06" x2="33.02" y2="99.06" width="0.1524" layer="91"/>
 <pinref part="RN1" gate="C" pin="1"/>
+<label x="48.26" y="99.06" size="1.778" layer="95"/>
 </segment>
 </net>
@@
 </segment>
 </net>
-<net name="N$15" class="0">
+<net name="MO3SND" class="0">
 <segment>
 <pinref part="J9" gate="G$1" pin="4"/>
 <wire x1="33.02" y1="68.58" x2="73.66" y2="68.58" width="0.1524" layer="91"/>
 <pinref part="RN1" gate="E" pin="1"/>
-</segment>
-</net>
+<label x="48.26" y="68.58" size="1.778" layer="95"/>
+</segment>
+</net>

Commit message: Fixed layout.
Connections:
- net N$1 renamed RX1R
- net N$11 renamed MO1RTNRAW
- net N$12 renamed RX2+
- net N$13 renamed RX2-
- net N$16 renamed MO2RTNRAW
- net N$17 renamed MO3RTNRAW
- net N$18 renamed MNTRSND
- net N$19 renamed MNTRRTN
- net N$2 renamed RX2R
- net N$3 renamed RX3R
- net N$5 renamed RX3
- net N$6 renamed RX2
- net N$7 renamed RX1
- net N$8 renamed RX1+
- net N$9 renamed RX1-
- net RX+ renamed RX3+
- net RX- renamed RX3-
Changed lines of the file:
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@@
 <part name="SUPPLY8" library="supply2" library_urn="urn:adsk.eagle:library:372" deviceset="GND" device=""/>
 <part name="SUPPLY5" library="supply2" library_urn="urn:adsk.eagle:library:372" deviceset="GND" device=""/>
-<part name="SUPPLY4" library="supply2" library_urn="urn:adsk.eagle:library:372" deviceset="VCC" device=""/>
 <part name="SUPPLY14" library="supply2" library_urn="urn:adsk.eagle:library:372" deviceset="GND" device=""/>
 <part name="SUPPLY11" library="supply2" library_urn="urn:adsk.eagle:library:372" deviceset="VCC" device=""/>
@@
 <part name="C4" library="rcl" library_urn="urn:adsk.eagle:library:334" deviceset="C-EU" device="025-024X044" package3d_urn="urn:adsk.eagle:package:23630/1" value="10n"/>
 <part name="C5" library="rcl" library_urn="urn:adsk.eagle:library:334" deviceset="C-EU" device="025-024X044" package3d_urn="urn:adsk.eagle:package:23630/1" value="10n"/>
-<part name="SUPPLY27" library="supply2" library_urn="urn:adsk.eagle:library:372" deviceset="GND" device=""/>
 <part name="LED1" library="led" library_urn="urn:adsk.eagle:library:259" deviceset="LED" device="3MM" package3d_urn="urn:adsk.eagle:package:15797/1" value="BLUE"/>
 <part name="SUPPLY28" library="supply2" library_urn="urn:adsk.eagle:library:372" deviceset="VCC" device=""/>
@@
 <attribute name="VALUE" x="140.335" y="47.625" size="1.778" layer="96"/>
 </instance>
-<instance part="SUPPLY4" gate="G$1" x="132.08" y="167.64" smashed="yes">
-<attribute name="VALUE" x="130.175" y="170.815" size="1.778" layer="96"/>
-</instance>
 <instance part="SUPPLY14" gate="GND" x="167.64" y="109.22" smashed="yes">
 <attribute name="VALUE" x="165.735" y="106.045" size="1.778" layer="96"/>
@@
 <attribute name="NAME" x="70.104" y="20.701" size="1.778" layer="95"/>
 <attribute name="VALUE" x="70.104" y="15.621" size="1.778" layer="96"/>
-</instance>
-<instance part="SUPPLY27" gate="GND" x="76.2" y="10.16" smashed="yes">
-<attribute name="VALUE" x="74.295" y="6.985" size="1.778" layer="96"/>
 </instance>
 <instance part="LED1" gate="G$1" x="25.4" y="20.32" smashed="yes">
@@
 </segment>
 <segment>
-<pinref part="SUPPLY27" gate="GND" pin="GND"/>
-<wire x1="76.2" y1="15.24" x2="76.2" y2="12.7" width="0.1524" layer="91"/>
-</segment>
-<segment>
 <pinref part="LED1" gate="G$1" pin="C"/>
 <pinref part="SUPPLY29" gate="GND" pin="GND"/>
@@
 </segment>
 </net>
-<net name="RX+" class="0">
+<net name="RX3+" class="0">
 <segment>
 <pinref part="IC4" gate="G$1" pin="A"/>
@@
 <wire x1="195.58" y1="60.96" x2="172.72" y2="60.96" width="0.1524" layer="91"/>
 <junction x="172.72" y="60.96"/>
-</segment>
-</net>
-<net name="RX-" class="0">
+<label x="200.66" y="109.22" size="1.778" layer="95"/>
+</segment>
+</net>
+<net name="RX3-" class="0">
 <segment>
 <pinref part="IC4" gate="G$1" pin="B"/>
@@
 <wire x1="198.12" y1="58.42" x2="187.96" y2="58.42" width="0.1524" layer="91"/>
 <junction x="187.96" y="58.42"/>
+<label x="200.66" y="106.68" size="1.778" layer="95"/>
 </segment>
 </net>
@@
 </segment>
 </net>
-<net name="N$1" class="0">
+<net name="RX1R" class="0">
 <segment>
 <pinref part="IC1" gate="B" pin="O"/>
@@
 </segment>
 </net>
-<net name="N$2" class="0">
+<net name="RX2R" class="0">
 <segment>
 <pinref part="IC1" gate="F" pin="O"/>
@@
 </segment>
 </net>
-<net name="N$3" class="0">
+<net name="RX3R" class="0">
 <segment>
 <pinref part="IC1" gate="D" pin="O"/>
@@
 </segment>
 </net>
-<net name="N$5" class="0">
+<net name="RX3" class="0">
 <segment>
 <pinref part="IC4" gate="G$1" pin="RO"/>
 <pinref part="IC1" gate="D" pin="I"/>
 <wire x1="144.78" y1="63.5" x2="139.7" y2="63.5" width="0.1524" layer="91"/>
-</segment>
-</net>
-<net name="N$6" class="0">
+<label x="139.7" y="63.5" size="1.778" layer="95"/>
+</segment>
+</net>
+<net name="RX2" class="0">
 <segment>
 <pinref part="IC3" gate="G$1" pin="RO"/>
 <pinref part="IC1" gate="F" pin="I"/>
 <wire x1="144.78" y1="93.98" x2="139.7" y2="93.98" width="0.1524" layer="91"/>
-</segment>
-</net>
-<net name="N$7" class="0">
+<label x="139.7" y="93.98" size="1.778" layer="95"/>
+</segment>
+</net>
+<net name="RX1" class="0">
 <segment>
 <pinref part="IC2" gate="G$1" pin="RO"/>
 <pinref part="IC1" gate="B" pin="I"/>
 <wire x1="144.78" y1="121.92" x2="139.7" y2="121.92" width="0.1524" layer="91"/>
-</segment>
-</net>
-<net name="N$8" class="0">
+<label x="139.7" y="121.92" size="1.778" layer="95"/>
+</segment>
+</net>
+<net name="RX1+" class="0">
 <segment>
 <pinref part="IC2" gate="G$1" pin="A"/>
@@
 <wire x1="172.72" y1="121.92" x2="172.72" y2="119.38" width="0.1524" layer="91"/>
 <junction x="172.72" y="119.38"/>
-</segment>
-</net>
-<net name="N$9" class="0">
+<label x="200.66" y="119.38" size="1.778" layer="95"/>
+</segment>
+</net>
+<net name="RX1-" class="0">
 <segment>
 <pinref part="IC2" gate="G$1" pin="B"/>
@@
 <wire x1="187.96" y1="121.92" x2="187.96" y2="116.84" width="0.1524" layer="91"/>
 <junction x="187.96" y="116.84"/>
-</segment>
-</net>
-<net name="N$12" class="0">
+<label x="200.66" y="116.84" size="1.778" layer="95"/>
+</segment>
+</net>
+<net name="RX2+" class="0">
 <segment>
 <pinref part="IC3" gate="G$1" pin="A"/>
@@
 <wire x1="172.72" y1="93.98" x2="172.72" y2="91.44" width="0.1524" layer="91"/>
 <junction x="172.72" y="91.44"/>
-</segment>
-</net>
-<net name="N$13" class="0">
+<label x="200.66" y="114.3" size="1.778" layer="95"/>
+</segment>
+</net>
+<net name="RX2-" class="0">
 <segment>
 <pinref part="X7" gate="G$1" pin="4"/>
@@
 <wire x1="187.96" y1="93.98" x2="187.96" y2="88.9" width="0.1524" layer="91"/>
 <junction x="187.96" y="88.9"/>
+<label x="200.66" y="111.76" size="1.778" layer="95"/>
 </segment>
 </net>
@@
 </segment>
 </net>
-<net name="N$11" class="0">
+<net name="MO1RTNRAW" class="0">
 <segment>
 <pinref part="IC1" gate="A" pin="O"/>
@@
 </segment>
 </net>
-<net name="N$16" class="0">
+<net name="MO2RTNRAW" class="0">
 <segment>
 <pinref part="IC1" gate="C" pin="O"/>
@@
 </segment>
 </net>
-<net name="N$17" class="0">
+<net name="MO3RTNRAW" class="0">
 <segment>
 <pinref part="IC1" gate="E" pin="O"/>
@@
 </segment>
 </net>
-<net name="N$18" class="0">
+<net name="MNTRSND" class="0">
 <segment>
 <pinref part="X7" gate="G$1" pin="7"/>
@@
 </segment>
 </net>
-<net name="N$19" class="0">
+<net name="MNTRRTN" class="0">
 <segment>
 <pinref part="X7" gate="G$1" pin="8"/>

Commit message: Redesign.
Parts:
- added C6, C7: 10n, rcl:C-EU025-024X044
- added IC5, IC6: 74ALS05N, 74xx-us:74ALS05N
- added J10: DIN5, SparkFun-Connectors:DIN5
- added R5: 100, rcl:R-EU_0204/5
- IC1: value 74ALS05N -> LTC485N; device 74xx-us:74ALS05N -> linear-technology:LTC485N
Connections:
- removed net MNTRRTN: RN1H.2, X7.8
- removed net MNTRSND: RN1G.2, X7.7
- new net MO4RTN: J10.5, RN1H.1
- new net MO4SND: J10.4, RN1G.1
- new net N$1: IC6A.I, IC6B.O, RN2.5
- new net N$2: IC4.RO, IC6B.I
- new net N$3: IC4.A, R5.1, X7.7
- new net N$5: IC4.B, R5.2, X7.8
- new net N$6: IC6A.O, RN1H.2
- net GND: now also C6.2, C7.2, IC1.!RE, IC1.DE, IC1.DI, IC1.GND, IC6C.I, IC6D.I, IC6E.I, IC6F.I, J10.2; no longer RN1H.1
- net MO1RTNRAW: now also IC5A.O; no longer IC1A.O
- net MO2RTNRAW: now also IC5C.O; no longer IC1C.O
- net MO3RTNRAW: now also IC5E.O; no longer IC1E.O
- net RX1: now also IC1.RO, IC5B.I; no longer IC1B.I, IC2.RO
- net RX1+: now also IC1.A; no longer IC2.A
- net RX1-: now also IC1.B; no longer IC2.B
- net RX1R: now also IC5A.I, IC5B.O; no longer IC1A.I, IC1B.O
- net RX2: now also IC2.RO, IC5F.I; no longer IC1F.I, IC3.RO
- net RX2+: now also IC2.A; no longer IC3.A
- net RX2-: now also IC2.B; no longer IC3.B
- net RX2R: now also IC5C.I, IC5F.O; no longer IC1C.I, IC1F.O
- net RX3: now also IC3.RO, IC5D.I; no longer IC1D.I, IC4.RO
- net RX3+: now also IC3.A; no longer IC4.A
- net RX3-: now also IC3.B; no longer IC4.B
- net RX3R: now also IC5D.O, IC5E.I; no longer IC1D.O, IC1E.I
- net VCC: now also C6.1, C7.1, IC1.VCC, RN1G.2; no longer RN1G.1
Other:
- moved on the sheet: C1, C2, C3, C4, C5, IC2, IC3, IC4, LED1, R1, RN1G, RN1H

Commit message: RX indicators.
Parts:
- added LED2, LED3, LED4, LED5: BLUE, led:LED3MM
- added R6, R7, R8, R9: 100, rcl:R-EU_0204/5
Connections:
- new net N$10: LED5.A, R9.1
- new net N$11: IC6C.O, LED2.C
- new net N$12: IC6D.O, LED3.C
- new net N$13: IC6E.O, LED4.C
- new net N$14: IC6F.O, LED5.C
- new net N$7: LED2.A, R6.1
- new net N$8: LED3.A, R7.1
- new net N$9: LED4.A, R8.1
- net GND: no longer IC6C.I, IC6D.I, IC6E.I, IC6F.I
- net N$1: now also IC6F.I
- net RX1R: now also IC6C.I
- net RX2R: now also IC6D.I
- net RX3R: now also IC6E.I
- net VCC: now also R6.2, R7.2, R8.2, R9.2
Other:
- moved on the sheet: IC3, IC4, IC5D, IC5E, IC6A, IC6B, IC6C, IC6D, IC6E, IC6F, J10, J9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

Commit message: Layout.
Parts:
- R1, R6, R7, R8, R9: value 100 -> 102
- R2, R3, R4, R5: value 100 -> 101
- RN1: value (none) -> 221
Other:
- moved on the sheet: IC5D
Changed lines of the file:
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@@
 <part name="SUPPLY28" library="supply2" library_urn="urn:adsk.eagle:library:372" deviceset="VCC" device=""/>
 <part name="SUPPLY29" library="supply2" library_urn="urn:adsk.eagle:library:372" deviceset="GND" device=""/>
-<part name="R4" library="rcl" library_urn="urn:adsk.eagle:library:334" deviceset="R-EU_" device="0204/5" package3d_urn="urn:adsk.eagle:package:23488/1" value="100"/>
+<part name="R4" library="rcl" library_urn="urn:adsk.eagle:library:334" deviceset="R-EU_" device="0204/5" package3d_urn="urn:adsk.eagle:package:23488/1" value="101"/>
 <part name="X7" library="con-rj45" deviceset="NELTRON-7810-XPXC" device=""/>
 <part name="IC2" library="linear-technology" library_urn="urn:adsk.eagle:library:261" deviceset="LTC485" device="N" package3d_urn="urn:adsk.eagle:package:16059/1"/>
@@
 <part name="SUPPLY25" library="supply2" library_urn="urn:adsk.eagle:library:372" deviceset="VCC" device=""/>
 <part name="SUPPLY30" library="supply2" library_urn="urn:adsk.eagle:library:372" deviceset="GND" device=""/>
-<part name="R2" library="rcl" library_urn="urn:adsk.eagle:library:334" deviceset="R-EU_" device="0204/5" package3d_urn="urn:adsk.eagle:package:23488/1" value="100"/>
-<part name="R3" library="rcl" library_urn="urn:adsk.eagle:library:334" deviceset="R-EU_" device="0204/5" package3d_urn="urn:adsk.eagle:package:23488/1" value="100"/>
+<part name="R2" library="rcl" library_urn="urn:adsk.eagle:library:334" deviceset="R-EU_" device="0204/5" package3d_urn="urn:adsk.eagle:package:23488/1" value="101"/>
+<part name="R3" library="rcl" library_urn="urn:adsk.eagle:library:334" deviceset="R-EU_" device="0204/5" package3d_urn="urn:adsk.eagle:package:23488/1" value="101"/>
 <part name="SUPPLY32" library="supply2" library_urn="urn:adsk.eagle:library:372" deviceset="VCC" device=""/>
 <part name="SUPPLY33" library="supply2" library_urn="urn:adsk.eagle:library:372" deviceset="GND" device=""/>
-<part name="RN1" library="resistor-dil" library_urn="urn:adsk.eagle:library:342" deviceset="8R-N" device="" package3d_urn="urn:adsk.eagle:package:922/2"/>
-<part name="R1" library="rcl" library_urn="urn:adsk.eagle:library:334" deviceset="R-EU_" device="0204/5" package3d_urn="urn:adsk.eagle:package:23488/1" value="100"/>
+<part name="RN1" library="resistor-dil" library_urn="urn:adsk.eagle:library:342" deviceset="8R-N" device="" package3d_urn="urn:adsk.eagle:package:922/2" value="221"/>
+<part name="R1" library="rcl" library_urn="urn:adsk.eagle:library:334" deviceset="R-EU_" device="0204/5" package3d_urn="urn:adsk.eagle:package:23488/1" value="102"/>
 <part name="IC4" library="linear-technology" library_urn="urn:adsk.eagle:library:261" deviceset="LTC485" device="N" package3d_urn="urn:adsk.eagle:package:16059/1"/>
 <part name="IC6" library="74xx-us" library_urn="urn:adsk.eagle:library:88" deviceset="74*05" device="N" package3d_urn="urn:adsk.eagle:package:16407/2" technology="ALS"/>
-<part name="R5" library="rcl" library_urn="urn:adsk.eagle:library:334" deviceset="R-EU_" device="0204/5" package3d_urn="urn:adsk.eagle:package:23488/1" value="100"/>
+<part name="R5" library="rcl" library_urn="urn:adsk.eagle:library:334" deviceset="R-EU_" device="0204/5" package3d_urn="urn:adsk.eagle:package:23488/1" value="101"/>
 <part name="C6" library="rcl" library_urn="urn:adsk.eagle:library:334" deviceset="C-EU" device="025-024X044" package3d_urn="urn:adsk.eagle:package:23630/1" value="10n"/>
 <part name="C7" library="rcl" library_urn="urn:adsk.eagle:library:334" deviceset="C-EU" device="025-024X044" package3d_urn="urn:adsk.eagle:package:23630/1" value="10n"/>
@@
 <part name="LED4" library="led" library_urn="urn:adsk.eagle:library:259" deviceset="LED" device="3MM" package3d_urn="urn:adsk.eagle:package:15797/1" value="BLUE"/>
 <part name="LED5" library="led" library_urn="urn:adsk.eagle:library:259" deviceset="LED" device="3MM" package3d_urn="urn:adsk.eagle:package:15797/1" value="BLUE"/>
-<part name="R6" library="rcl" library_urn="urn:adsk.eagle:library:334" deviceset="R-EU_" device="0204/5" package3d_urn="urn:adsk.eagle:package:23488/1" value="100"/>
-<part name="R7" library="rcl" library_urn="urn:adsk.eagle:library:334" deviceset="R-EU_" device="0204/5" package3d_urn="urn:adsk.eagle:package:23488/1" value="100"/>
-<part name="R8" library="rcl" library_urn="urn:adsk.eagle:library:334" deviceset="R-EU_" device="0204/5" package3d_urn="urn:adsk.eagle:package:23488/1" value="100"/>
-<part name="R9" library="rcl" library_urn="urn:adsk.eagle:library:334" deviceset="R-EU_" device="0204/5" package3d_urn="urn:adsk.eagle:package:23488/1" value="100"/>
+<part name="R6" library="rcl" library_urn="urn:adsk.eagle:library:334" deviceset="R-EU_" device="0204/5" package3d_urn="urn:adsk.eagle:package:23488/1" value="102"/>
+<part name="R7" library="rcl" library_urn="urn:adsk.eagle:library:334" deviceset="R-EU_" device="0204/5" package3d_urn="urn:adsk.eagle:package:23488/1" value="102"/>
+<part name="R8" library="rcl" library_urn="urn:adsk.eagle:library:334" deviceset="R-EU_" device="0204/5" package3d_urn="urn:adsk.eagle:package:23488/1" value="102"/>
+<part name="R9" library="rcl" library_urn="urn:adsk.eagle:library:334" deviceset="R-EU_" device="0204/5" package3d_urn="urn:adsk.eagle:package:23488/1" value="102"/>
 <part name="SUPPLY41" library="supply2" library_urn="urn:adsk.eagle:library:372" deviceset="VCC" device=""/>
 </parts>
@@
 <attribute name="VALUE" x="93.98" y="88.9" size="1.778" layer="96" rot="MR0"/>
 </instance>
-<instance part="IC5" gate="D" x="127" y="66.04" smashed="yes" rot="R180">
-<attribute name="NAME" x="124.46" y="62.865" size="1.778" layer="95" rot="R180"/>
-<attribute name="VALUE" x="124.46" y="71.12" size="1.778" layer="96" rot="R180"/>
+<instance part="IC5" gate="D" x="129.54" y="66.04" smashed="yes" rot="R180">
+<attribute name="NAME" x="127" y="62.865" size="1.778" layer="95" rot="R180"/>
+<attribute name="VALUE" x="127" y="71.12" size="1.778" layer="96" rot="R180"/>
 </instance>
 <instance part="IC5" gate="E" x="96.52" y="66.04" smashed="yes" rot="R180">
@@
 <pinref part="IC5" gate="D" pin="O"/>
 <pinref part="IC5" gate="E" pin="I"/>
-<wire x1="116.84" y1="66.04" x2="114.3" y2="66.04" width="0.1524" layer="91"/>
+<wire x1="119.38" y1="66.04" x2="114.3" y2="66.04" width="0.1524" layer="91"/>
 <pinref part="RN2" gate="1" pin="4"/>
 <wire x1="114.3" y1="66.04" x2="109.22" y2="66.04" width="0.1524" layer="91"/>
@@
 <pinref part="IC3" gate="G$1" pin="RO"/>
 <pinref part="IC5" gate="D" pin="I"/>
-<wire x1="144.78" y1="66.04" x2="137.16" y2="66.04" width="0.1524" layer="91"/>
+<wire x1="144.78" y1="66.04" x2="139.7" y2="66.04" width="0.1524" layer="91"/>
 <label x="139.7" y="63.5" size="1.778" layer="95"/>
 </segment>
