File: 0/hardware/logicboard/p0rx-001.sch (EAGLE design)
At the start: 37 parts, among them IC1 LTC485N, IC2 LTC485N, IC3 LTC485N, IC4 LTC485N, IC5 74ALS05N, IC6 74ALS05N, J0 DC5V, J10 DIN5, J7 DIN5, J8 DIN5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

Commit message: Replaced Rs with RN.
Parts:
- removed R6, R7, R8, R9: 102, rcl:R-EU_0204/5
- added RN3: 1k, resistor-net:RN04
Connections:
- net N$10: now also RN3.5; no longer R9.1
- net N$7: now also RN3.2; no longer R6.1
- net N$8: now also RN3.3; no longer R7.1
- net N$9: now also RN3.4; no longer R8.1
- net VCC: now also RN3.1; no longer R6.2, R7.2, R8.2, R9.2
Changed lines of the file:
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@@
 <part name="LED4" library="led" library_urn="urn:adsk.eagle:library:259" deviceset="LED" device="3MM" package3d_urn="urn:adsk.eagle:package:15797/1" value="BLUE"/>
 <part name="LED5" library="led" library_urn="urn:adsk.eagle:library:259" deviceset="LED" device="3MM" package3d_urn="urn:adsk.eagle:package:15797/1" value="BLUE"/>
-<part name="R6" library="rcl" library_urn="urn:adsk.eagle:library:334" deviceset="R-EU_" device="0204/5" package3d_urn="urn:adsk.eagle:package:23488/1" value="102"/>
-<part name="R7" library="rcl" library_urn="urn:adsk.eagle:library:334" deviceset="R-EU_" device="0204/5" package3d_urn="urn:adsk.eagle:package:23488/1" value="102"/>
-<part name="R8" library="rcl" library_urn="urn:adsk.eagle:library:334" deviceset="R-EU_" device="0204/5" package3d_urn="urn:adsk.eagle:package:23488/1" value="102"/>
-<part name="R9" library="rcl" library_urn="urn:adsk.eagle:library:334" deviceset="R-EU_" device="0204/5" package3d_urn="urn:adsk.eagle:package:23488/1" value="102"/>
 <part name="SUPPLY41" library="supply2" library_urn="urn:adsk.eagle:library:372" deviceset="VCC" device=""/>
+<part name="RN3" library="resistor-net" library_urn="urn:adsk.eagle:library:343" deviceset="RN04" device="" package3d_urn="urn:adsk.eagle:package:24976/1" value="1k"/>
 </parts>
 <sheets>
@@
 <attribute name="VALUE" x="71.755" y="140.208" size="1.778" layer="96" rot="R90"/>
 </instance>
-<instance part="R6" gate="G$1" x="50.8" y="154.94" smashed="yes" rot="R90">
-<attribute name="NAME" x="49.3014" y="151.13" size="1.778" layer="95" rot="R90"/>
-<attribute name="VALUE" x="54.102" y="151.13" size="1.778" layer="96" rot="R90"/>
-</instance>
-<instance part="R7" gate="G$1" x="55.88" y="154.94" smashed="yes" rot="R90">
-<attribute name="NAME" x="54.3814" y="151.13" size="1.778" layer="95" rot="R90"/>
-<attribute name="VALUE" x="59.182" y="151.13" size="1.778" layer="96" rot="R90"/>
-</instance>
-<instance part="R8" gate="G$1" x="60.96" y="154.94" smashed="yes" rot="R90">
-<attribute name="NAME" x="59.4614" y="151.13" size="1.778" layer="95" rot="R90"/>
-<attribute name="VALUE" x="64.262" y="151.13" size="1.778" layer="96" rot="R90"/>
-</instance>
-<instance part="R9" gate="G$1" x="66.04" y="154.94" smashed="yes" rot="R90">
-<attribute name="NAME" x="64.5414" y="151.13" size="1.778" layer="95" rot="R90"/>
-<attribute name="VALUE" x="69.342" y="151.13" size="1.778" layer="96" rot="R90"/>
-</instance>
-<instance part="SUPPLY41" gate="G$1" x="50.8" y="167.64" smashed="yes">
-<attribute name="VALUE" x="48.895" y="170.815" size="1.778" layer="96"/>
+<instance part="SUPPLY41" gate="G$1" x="38.1" y="167.64" smashed="yes">
+<attribute name="VALUE" x="36.195" y="170.815" size="1.778" layer="96"/>
+</instance>
+<instance part="RN3" gate="1" x="45.72" y="157.48" smashed="yes">
+<attribute name="NAME" x="43.18" y="160.02" size="1.778" layer="95"/>
+<attribute name="VALUE" x="43.18" y="153.162" size="1.778" layer="96"/>
 </instance>
 </instances>
@@
 <segment>
 <pinref part="SUPPLY41" gate="G$1" pin="VCC"/>
-<pinref part="R6" gate="G$1" pin="2"/>
-<wire x1="50.8" y1="165.1" x2="50.8" y2="162.56" width="0.1524" layer="91"/>
-<wire x1="50.8" y1="162.56" x2="50.8" y2="160.02" width="0.1524" layer="91"/>
-<wire x1="50.8" y1="162.56" x2="55.88" y2="162.56" width="0.1524" layer="91"/>
-<junction x="50.8" y="162.56"/>
-<pinref part="R9" gate="G$1" pin="2"/>
-<wire x1="55.88" y1="162.56" x2="60.96" y2="162.56" width="0.1524" layer="91"/>
-<wire x1="60.96" y1="162.56" x2="66.04" y2="162.56" width="0.1524" layer="91"/>
-<wire x1="66.04" y1="162.56" x2="66.04" y2="160.02" width="0.1524" layer="91"/>
-<pinref part="R8" gate="G$1" pin="2"/>
-<wire x1="60.96" y1="160.02" x2="60.96" y2="162.56" width="0.1524" layer="91"/>
-<junction x="60.96" y="162.56"/>
-<pinref part="R7" gate="G$1" pin="2"/>
-<wire x1="55.88" y1="160.02" x2="55.88" y2="162.56" width="0.1524" layer="91"/>
-<junction x="55.88" y="162.56"/>
+<wire x1="38.1" y1="165.1" x2="38.1" y2="157.48" width="0.1524" layer="91"/>
+<pinref part="RN3" gate="1" pin="1"/>
+<wire x1="38.1" y1="157.48" x2="40.64" y2="157.48" width="0.1524" layer="91"/>
 </segment>
 </net>
@@
 <net name="N$7" class="0">
 <segment>
-<pinref part="R6" gate="G$1" pin="1"/>
 <pinref part="LED2" gate="G$1" pin="A"/>
-<wire x1="50.8" y1="149.86" x2="50.8" y2="147.32" width="0.1524" layer="91"/>
+<wire x1="50.8" y1="157.48" x2="50.8" y2="147.32" width="0.1524" layer="91"/>
+<pinref part="RN3" gate="1" pin="2"/>
 </segment>
 </net>
 <net name="N$8" class="0">
 <segment>
-<pinref part="R7" gate="G$1" pin="1"/>
 <pinref part="LED3" gate="G$1" pin="A"/>
-<wire x1="55.88" y1="149.86" x2="55.88" y2="147.32" width="0.1524" layer="91"/>
+<wire x1="55.88" y1="157.48" x2="55.88" y2="147.32" width="0.1524" layer="91"/>
+<pinref part="RN3" gate="1" pin="3"/>
 </segment>
 </net>
 <net name="N$9" class="0">
 <segment>
-<pinref part="R8" gate="G$1" pin="1"/>
 <pinref part="LED4" gate="G$1" pin="A"/>
-<wire x1="60.96" y1="149.86" x2="60.96" y2="147.32" width="0.1524" layer="91"/>
+<wire x1="60.96" y1="157.48" x2="60.96" y2="147.32" width="0.1524" layer="91"/>
+<pinref part="RN3" gate="1" pin="4"/>
 </segment>
 </net>
 <net name="N$10" class="0">
 <segment>
-<pinref part="R9" gate="G$1" pin="1"/>
 <pinref part="LED5" gate="G$1" pin="A"/>
-<wire x1="66.04" y1="149.86" x2="66.04" y2="147.32" width="0.1524" layer="91"/>
-</segment>
-</net>
+<wire x1="66.04" y1="157.48" x2="66.04" y2="147.32" width="0.1524" layer="91"/>
+<pinref part="RN3" gate="1" pin="5"/>
+</segment>
+</net>

Commit message: Fixed wiring of 0.
Connections:
- removed net N$3: IC4.A, R5.1, X7.7
- removed net N$5: IC4.B, R5.2, X7.8
- new net RX4+: IC4.A, R5.1, X7.8
- new net RX4-: IC4.B, R5.2, X7.7
- net RX1+: now also X7.4; no longer X7.1
- net RX1-: now also X7.5; no longer X7.2
- net RX2+: now also X7.6; no longer X7.3
- net RX2-: now also X7.3; no longer X7.4
- net RX3+: now also X7.2; no longer X7.5
- net RX3-: now also X7.1; no longer X7.6
Other:
- moved on the sheet: X7
Changed lines of the file:
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@@
 <attribute name="VALUE" x="176.53" y="62.738" size="1.778" layer="96"/>
 </instance>
-<instance part="X7" gate="G$1" x="226.06" y="109.22" smashed="yes">
-<attribute name="NAME" x="229.87" y="119.888" size="1.778" layer="95"/>
-<attribute name="VALUE" x="229.87" y="98.298" size="1.778" layer="96"/>
+<instance part="X7" gate="G$1" x="226.06" y="116.84" smashed="yes">
+<attribute name="NAME" x="229.87" y="127.508" size="1.778" layer="95"/>
+<attribute name="VALUE" x="229.87" y="105.918" size="1.778" layer="96"/>
 </instance>
 <instance part="IC2" gate="G$1" x="154.94" y="91.44" smashed="yes">
@@
 </segment>
 <segment>
-<wire x1="228.6" y1="96.52" x2="228.6" y2="93.98" width="0.1524" layer="91"/>
+<wire x1="228.6" y1="104.14" x2="228.6" y2="93.98" width="0.1524" layer="91"/>
 <wire x1="228.6" y1="93.98" x2="226.06" y2="93.98" width="0.1524" layer="91"/>
-<wire x1="226.06" y1="93.98" x2="226.06" y2="96.52" width="0.1524" layer="91"/>
+<wire x1="226.06" y1="93.98" x2="226.06" y2="104.14" width="0.1524" layer="91"/>
 <pinref part="SUPPLY26" gate="GND" pin="GND"/>
 <wire x1="226.06" y1="93.98" x2="226.06" y2="91.44" width="0.1524" layer="91"/>
@@
 <pinref part="IC3" gate="G$1" pin="A"/>
 <wire x1="165.1" y1="63.5" x2="172.72" y2="63.5" width="0.1524" layer="91"/>
-<label x="167.64" y="60.96" size="1.778" layer="95"/>
+<label x="167.64" y="63.5" size="1.778" layer="95"/>
 <pinref part="R4" gate="G$1" pin="1"/>
 <wire x1="175.26" y1="66.04" x2="172.72" y2="66.04" width="0.1524" layer="91"/>
 <wire x1="172.72" y1="66.04" x2="172.72" y2="63.5" width="0.1524" layer="91"/>
-<pinref part="X7" gate="G$1" pin="5"/>
-<wire x1="223.52" y1="109.22" x2="195.58" y2="109.22" width="0.1524" layer="91"/>
-<wire x1="195.58" y1="109.22" x2="195.58" y2="63.5" width="0.1524" layer="91"/>
+<wire x1="195.58" y1="124.46" x2="195.58" y2="63.5" width="0.1524" layer="91"/>
 <wire x1="195.58" y1="63.5" x2="172.72" y2="63.5" width="0.1524" layer="91"/>
 <junction x="172.72" y="63.5"/>
-<label x="200.66" y="109.22" size="1.778" layer="95"/>
+<pinref part="X7" gate="G$1" pin="2"/>
+<wire x1="223.52" y1="124.46" x2="195.58" y2="124.46" width="0.1524" layer="91"/>
+<label x="205.74" y="124.46" size="1.778" layer="95"/>
 </segment>
 </net>
@@
 <segment>
 <pinref part="IC3" gate="G$1" pin="B"/>
-<label x="167.64" y="58.42" size="1.778" layer="95"/>
+<label x="167.64" y="60.96" size="1.778" layer="95"/>
 <pinref part="R4" gate="G$1" pin="2"/>
 <wire x1="187.96" y1="60.96" x2="165.1" y2="60.96" width="0.1524" layer="91"/>
 <wire x1="185.42" y1="66.04" x2="187.96" y2="66.04" width="0.1524" layer="91"/>
 <wire x1="187.96" y1="66.04" x2="187.96" y2="60.96" width="0.1524" layer="91"/>
-<pinref part="X7" gate="G$1" pin="6"/>
-<wire x1="223.52" y1="106.68" x2="198.12" y2="106.68" width="0.1524" layer="91"/>
-<wire x1="198.12" y1="106.68" x2="198.12" y2="60.96" width="0.1524" layer="91"/>
+<wire x1="198.12" y1="127" x2="198.12" y2="60.96" width="0.1524" layer="91"/>
 <wire x1="198.12" y1="60.96" x2="187.96" y2="60.96" width="0.1524" layer="91"/>
 <junction x="187.96" y="60.96"/>
-<label x="200.66" y="106.68" size="1.778" layer="95"/>
+<pinref part="X7" gate="G$1" pin="1"/>
+<wire x1="223.52" y1="127" x2="198.12" y2="127" width="0.1524" layer="91"/>
+<label x="205.74" y="127" size="1.778" layer="95"/>
 </segment>
 </net>
@@
 <segment>
 <pinref part="IC1" gate="G$1" pin="A"/>
-<pinref part="X7" gate="G$1" pin="1"/>
 <wire x1="165.1" y1="119.38" x2="172.72" y2="119.38" width="0.1524" layer="91"/>
 <pinref part="R2" gate="G$1" pin="1"/>
-<wire x1="172.72" y1="119.38" x2="223.52" y2="119.38" width="0.1524" layer="91"/>
 <wire x1="175.26" y1="121.92" x2="172.72" y2="121.92" width="0.1524" layer="91"/>
 <wire x1="172.72" y1="121.92" x2="172.72" y2="119.38" width="0.1524" layer="91"/>
+<wire x1="172.72" y1="119.38" x2="223.52" y2="119.38" width="0.1524" layer="91"/>
 <junction x="172.72" y="119.38"/>
-<label x="200.66" y="119.38" size="1.778" layer="95"/>
+<pinref part="X7" gate="G$1" pin="4"/>
+<label x="205.74" y="119.38" size="1.778" layer="95"/>
+<label x="167.64" y="119.38" size="1.778" layer="95"/>
 </segment>
 </net>
@@
 <segment>
 <pinref part="IC1" gate="G$1" pin="B"/>
-<pinref part="X7" gate="G$1" pin="2"/>
 <wire x1="165.1" y1="116.84" x2="187.96" y2="116.84" width="0.1524" layer="91"/>
 <pinref part="R2" gate="G$1" pin="2"/>
-<wire x1="187.96" y1="116.84" x2="223.52" y2="116.84" width="0.1524" layer="91"/>
 <wire x1="185.42" y1="121.92" x2="187.96" y2="121.92" width="0.1524" layer="91"/>
 <wire x1="187.96" y1="121.92" x2="187.96" y2="116.84" width="0.1524" layer="91"/>
+<pinref part="X7" gate="G$1" pin="5"/>
+<wire x1="187.96" y1="116.84" x2="223.52" y2="116.84" width="0.1524" layer="91"/>
 <junction x="187.96" y="116.84"/>
-<label x="200.66" y="116.84" size="1.778" layer="95"/>
+<label x="205.74" y="116.84" size="1.778" layer="95"/>
+<label x="167.64" y="116.84" size="1.778" layer="95"/>
 </segment>
 </net>
@@
 <wire x1="172.72" y1="91.44" x2="190.5" y2="91.44" width="0.1524" layer="91"/>
 <wire x1="190.5" y1="91.44" x2="190.5" y2="114.3" width="0.1524" layer="91"/>
-<pinref part="X7" gate="G$1" pin="3"/>
-<wire x1="190.5" y1="114.3" x2="223.52" y2="114.3" width="0.1524" layer="91"/>
 <pinref part="R3" gate="G$1" pin="1"/>
 <wire x1="175.26" y1="93.98" x2="172.72" y2="93.98" width="0.1524" layer="91"/>
 <wire x1="172.72" y1="93.98" x2="172.72" y2="91.44" width="0.1524" layer="91"/>
 <junction x="172.72" y="91.44"/>
-<label x="200.66" y="114.3" size="1.778" layer="95"/>
+<pinref part="X7" gate="G$1" pin="6"/>
+<wire x1="223.52" y1="114.3" x2="190.5" y2="114.3" width="0.1524" layer="91"/>
+<label x="205.74" y="114.3" size="1.778" layer="95"/>
+<label x="167.64" y="91.44" size="1.778" layer="95"/>
 </segment>
 </net>
 <net name="RX2-" class="0">
 <segment>
-<pinref part="X7" gate="G$1" pin="4"/>
-<wire x1="223.52" y1="111.76" x2="193.04" y2="111.76" width="0.1524" layer="91"/>
-<wire x1="193.04" y1="111.76" x2="193.04" y2="88.9" width="0.1524" layer="91"/>
+<wire x1="193.04" y1="121.92" x2="193.04" y2="88.9" width="0.1524" layer="91"/>
 <pinref part="IC2" gate="G$1" pin="B"/>
 <wire x1="193.04" y1="88.9" x2="187.96" y2="88.9" width="0.1524" layer="91"/>
@@
 <wire x1="187.96" y1="93.98" x2="187.96" y2="88.9" width="0.1524" layer="91"/>
 <junction x="187.96" y="88.9"/>
-<label x="200.66" y="111.76" size="1.778" layer="95"/>
+<pinref part="X7" gate="G$1" pin="3"/>
+<wire x1="223.52" y1="121.92" x2="193.04" y2="121.92" width="0.1524" layer="91"/>
+<label x="205.74" y="121.92" size="1.778" layer="95"/>
+<label x="167.64" y="88.9" size="1.778" layer="95"/>
 </segment>
 </net>
@@
 </segment>
 </net>
-<net name="N$3" class="0">
+<net name="RX4+" class="0">
 <segment>
 <pinref part="IC4" gate="G$1" pin="A"/>
 <wire x1="165.1" y1="35.56" x2="172.72" y2="35.56" width="0.1524" layer="91"/>
 <wire x1="172.72" y1="35.56" x2="200.66" y2="35.56" width="0.1524" layer="91"/>
-<wire x1="200.66" y1="35.56" x2="200.66" y2="104.14" width="0.1524" layer="91"/>
-<pinref part="X7" gate="G$1" pin="7"/>
-<wire x1="200.66" y1="104.14" x2="223.52" y2="104.14" width="0.1524" layer="91"/>
+<wire x1="200.66" y1="35.56" x2="200.66" y2="109.22" width="0.1524" layer="91"/>
 <pinref part="R5" gate="G$1" pin="1"/>
 <wire x1="175.26" y1="38.1" x2="172.72" y2="38.1" width="0.1524" layer="91"/>
 <wire x1="172.72" y1="38.1" x2="172.72" y2="35.56" width="0.1524" layer="91"/>
 <junction x="172.72" y="35.56"/>
-</segment>
-</net>
-<net name="N$5" class="0">
-<segment>
 <pinref part="X7" gate="G$1" pin="8"/>
-<wire x1="223.52" y1="101.6" x2="203.2" y2="101.6" width="0.1524" layer="91"/>
+<wire x1="223.52" y1="109.22" x2="200.66" y2="109.22" width="0.1524" layer="91"/>
+<label x="205.74" y="109.22" size="1.778" layer="95"/>
+<label x="167.64" y="35.56" size="1.778" layer="95"/>
+</segment>
+</net>
+<net name="RX4-" class="0">
+<segment>
 <pinref part="IC4" gate="G$1" pin="B"/>
-<wire x1="203.2" y1="101.6" x2="203.2" y2="33.02" width="0.1524" layer="91"/>
+<wire x1="203.2" y1="111.76" x2="203.2" y2="33.02" width="0.1524" layer="91"/>
 <wire x1="203.2" y1="33.02" x2="187.96" y2="33.02" width="0.1524" layer="91"/>
 <pinref part="R5" gate="G$1" pin="2"/>
@@
 <wire x1="187.96" y1="38.1" x2="187.96" y2="33.02" width="0.1524" layer="91"/>
 <junction x="187.96" y="33.02"/>
-</segment>
-</net>
+<pinref part="X7" gate="G$1" pin="7"/>
+<wire x1="223.52" y1="111.76" x2="203.2" y2="111.76" width="0.1524" layer="91"/>
+<label x="205.74" y="111.76" size="1.778" layer="95"/>
+<label x="167.64" y="33.02" size="1.778" layer="95"/>
+</segment>
+</net>
