File: 0b/hardware/logicboard/p0b-002.brd (EAGLE design)
At the start: 70 x 41 mm, 30 parts, among them IC1 7404D, IC4 LTC485S, IC5 LTC485S, J0 DC5V, J7 DIN5, J9 DIN5, X7 NELTRON-7810-XPXC

Commit message: Now 0b are divided in type a (straight) and type b (cross).
Connections:
- net RX+: now also X7.2; no longer X7.6
- net RX-: now also X7.1; no longer X7.3
- net TX+: now also X7.6; no longer X7.2
- net TX-: now also X7.3; no longer X7.1
Routing:
- net RX: track 88.8 -> 64.6 mm, vias 0 -> 2
- net RX-: track 60.3 -> 42.1 mm, vias 3 -> 2
- net RX+: track 42.8 -> 59.3 mm, vias 1 -> 0
- net MIRTN: track 45.0 -> 56.5 mm, vias 3 -> 0
- net VCC: track 143.2 -> 153.3 mm
- net GND: track 230.9 -> 224.9 mm
- net NMIDIOUT: track 16.2 -> 18.8 mm
- net MIDIINGND: track 50.9 -> 49.0 mm
- net TX+: track 37.0 -> 35.3 mm, vias 2 -> 1
- net TX-: track 40.2 -> 41.5 mm
- net MIDIOUTGND: track 28.1 -> 26.9 mm
- net MIDIOUTV+: track 31.0 -> 29.8 mm
- net MIDIINV+: track 50.1 -> 51.0 mm
- net MORTN: track 34.8 -> 34.0 mm, vias 1 -> 0
- net MOSND: vias 0 -> 2
Other:
- board text added: "B"
- board text added: "TYPE B"
- board text removed: "A"
- board text removed: "TYPE A"
