File: Peripherals/PixelDrive/hardware/logicboard/pxdr-001.brd (EAGLE design)
At the start: 92 x 58 mm, 10 parts

Commit message: First try.
Parts:
- removed SV0: (no value), con-ml:ML34L
- removed SV3: (no value), con-ml:ML14L
- added J1: (no value), SparkFun-Connectors:JST-4-PTH
- added J2: (no value), SparkFun-Connectors:JST-5-PTH
- added J3: (no value), SparkFun-Connectors:JST-3-PTH
- added SV2: (no value), con-ml:ML40L
- moved LED1 14.3 mm to (63.0, 48.0)
- moved R1 14.3 mm to (73.0, 48.0)
- moved R2 11.0 mm to (22.0, 42.0)
- moved C2 10.4 mm to (52.0, 45.0)
- moved C1 6.32 mm to (52.0, 48.0)
Connections:
- removed net GB00: SV0.1, SV3.1
- removed net GB01: SV0.3, SV3.3
- removed net GB02: SV0.5, SV3.7
- removed net GB03: SV0.7, SV3.9
- removed net GB04: SV0.9, SV3.11
- removed net GB05: SV0.11, SV3.2
- removed net GB06: SV0.13, SV3.4
- removed net GB07: SV0.15, SV3.6
- removed net GB08: SV0.19, SV3.8
- removed net GB09: SV0.21, SV3.10
- removed net GB10: SV0.23, SV3.12
- removed net GB11: SV0.25, SV3.14
- removed net GB12: SV0.27, SV1.2
- removed net GB13: SV0.29, SV1.6
- removed net GB14: SV0.31, SV1.10
- removed net GB15: SV0.33, SV1.14
- new net NP1: SV1.2, SV2.2
- new net NP10: J1.4, SV2.29
- new net NP11: J2.2, SV2.32
- new net NP12: J2.3, SV2.35
- new net NP13: J2.4, SV2.38
- new net NP14: J3.2, SV2.40
- new net NP2: SV1.6, SV2.5
- new net NP3: SV1.10, SV2.8
- new net NP4: SV1.14, SV2.11
- new net NP5: SV1.3, SV2.14
- new net NP6: SV1.7, SV2.17
- new net NP7: SV1.11, SV2.20
- new net NP8: SV1.15, SV2.23
- new net NP9: J1.3, SV2.26
- net GND: now also J1.1, J2.1, J3.1, SV2.1, SV2.10, SV2.13, SV2.16, SV2.19, SV2.22, SV2.25, SV2.28, SV2.31, SV2.34, SV2.37, SV2.4, SV2.7; no longer SV0.10, SV0.12, SV0.14, SV0.16, SV0.18, SV0.2, SV0.20, SV0.22, SV0.24, SV0.26, SV0.28, SV0.30, SV0.32, SV0.34, SV0.4, SV0.6, SV0.8, SV3.5
- net VCC: now also J1.2, J2.5, J3.3; no longer SV3.13
- net VCC/2: now also SV2.12, SV2.15, SV2.18, SV2.21, SV2.24, SV2.27, SV2.3, SV2.30, SV2.33, SV2.36, SV2.39, SV2.6, SV2.9
Routing:
- net VCC/2: track 30.5 -> 140.7 mm
- net NP13: track 0.00 -> 88.8 mm
- net NP14: track 0.00 -> 85.3 mm
- net NP1: track 0.00 -> 77.7 mm
- net NP12: track 0.00 -> 70.0 mm
- net NP2: track 0.00 -> 63.3 mm
- net GB11: track 61.3 -> 0.00 mm
- net NP5: track 0.00 -> 58.2 mm
- net NP11: track 0.00 -> 58.1 mm, vias 0 -> 2
- net GB10: track 57.1 -> 0.00 mm
- net NP10: track 0.00 -> 57.1 mm
- net NP3: track 0.00 -> 54.8 mm
- net GB09: track 54.4 -> 0.00 mm
- net GB04: track 53.0 -> 0.00 mm
- net NP9: track 0.00 -> 51.9 mm, vias 0 -> 1
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- removed copper zone on layer 1, net GND
- removed copper zone on layer 16, net GND
Other:
- board text added: "1-Wire"
- board text added: "GPIO"
- board text added: "GeekPort II"
- board text added: "MKR"
- board text added: "PixelDrive"
- board text added: "PixelDrive 0.0.0-X"
- board text removed: "GeekBox 1.0.0-RC"
- board text removed: "To GeekPort II"
- board text removed: "To RIGOL MSO5000"
- board text removed: "To TestPort II"

Commit message: Second shot.
Parts:
- moved R1 14.1 mm to (63.0, 38.0)
- moved R2 11.7 mm to (33.0, 38.0)
Connections:
- removed net NP11: J2.2, SV2.32
- removed net NP12: J2.3, SV2.35
- removed net NP13: J2.4, SV2.38
- removed net NP14: J3.2, SV2.40
- new net DIGITAL7: J2.4, SV2.32
- new net SCL: J2.3, SV2.36
- new net SDA: J2.2, SV2.35
- new net THS: J3.2, SV2.39
- net GND: now also SV2.38; no longer SV2.37
- net VCC: now also SV2.33, SV2.37, SV2.40
- net VCC/2: no longer SV2.33, SV2.36, SV2.39
Routing:
- net SDA: track 0.00 -> 100.7 mm
- net VCC: track 32.6 -> 126.5 mm, vias 0 -> 1
- net THS: track 0.00 -> 89.3 mm
- net NP13: track 88.8 -> 0.00 mm
- net NP14: track 85.3 -> 0.00 mm
- net SCL: track 0.00 -> 83.2 mm
- net DIGITAL7: track 0.00 -> 74.5 mm
- net GND: track 184.7 -> 256.8 mm, vias 0 -> 1
- net NP12: track 70.0 -> 0.00 mm
- net NP11: track 58.1 -> 0.00 mm, vias 2 -> 0
- net VCC/2: track 140.7 -> 123.2 mm, vias 0 -> 1
- net NP9: track 51.9 -> 64.5 mm, vias 1 -> 0
- net VCC2LED: track 17.6 -> 28.4 mm
- net NP1: track 77.7 -> 88.1 mm
- net NP10: track 57.1 -> 63.1 mm
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
Commit message: Third shot.
Connections:
- net DIGITAL7 renamed NP11
- removed net THS: J3.2, SV2.39
- new net NP12: J3.2, SV2.35
- net GND: now also SV2.37; no longer SV2.38
- net SCL: now also SV2.39; no longer SV2.36
- net SDA: now also SV2.38; no longer SV2.35
- net VCC: no longer SV2.33, SV2.37
- net VCC/2: now also SV2.33, SV2.36
Routing:
- net NP12: track 0.00 -> 96.2 mm
- net THS: track 89.3 -> 0.00 mm
- net GND: track 256.8 -> 188.7 mm, vias 1 -> 0
- net VCC/2: track 123.2 -> 154.7 mm
- net SDA: track 100.7 -> 82.6 mm
- net NP1: track 88.1 -> 71.6 mm
- net VCC: track 126.5 -> 113.9 mm
- net NP5: track 62.6 -> 57.2 mm
- net SCL: track 83.2 -> 77.9 mm
- net NP11: track 74.5 -> 78.7 mm, vias 0 -> 1
- net NP2: track 57.9 -> 60.5 mm
- net NP3: track 55.9 -> 54.3 mm, vias 1 -> 0
- net VCC2LED: track 28.4 -> 26.9 mm
- net NP9: track 64.5 -> 65.6 mm

Commit message: Fixed some errors.
Parts:
- C1, C2: value (none) -> 104
- J1: value (none) -> GPIO
- J2: value (none) -> MKR
- J3: value (none) -> 1-Wire
- LED1: value (none) -> GRN; device led:LED3MM -> led:Q62902-B152
- LED2: value (none) -> BLU; device led:LED3MM -> led:Q62902-B152
- SV2: value (none) -> LightDrive
- moved LED1 44.4 mm to (19.0, 54.0), turned to 90 degrees
- moved R1 44.0 mm to (19.0, 36.0), turned to 90 degrees
- moved C2 26.4 mm to (28.0, 34.0)
- moved C1 26.0 mm to (28.0, 38.0)
- moved R2 18.1 mm to (15.0, 36.0), turned to 90 degrees
- moved J1 2.00 mm to (54.0, 52.0)
- moved J2 2.00 mm to (65.0, 52.0)
- moved J3 2.00 mm to (75.0, 52.0)
- moved SV1 2.00 mm to (35.0, 47.0)
- moved LED2 1.00 mm to (15.0, 54.0), turned to 90 degrees
Routing:
- net GND: track 188.7 -> 170.1 mm
- net SCL: track 77.9 -> 94.7 mm
- net NP3: track 54.3 -> 69.4 mm
- net VCC/2: track 154.7 -> 139.8 mm, vias 1 -> 0
- net NP2: track 60.5 -> 72.7 mm
- net NP12: track 96.2 -> 85.3 mm
- net NP1: track 71.6 -> 82.3 mm
- net NP9: track 65.6 -> 55.4 mm
- net VCC2LED: track 26.9 -> 18.6 mm
- net SDA: track 82.6 -> 89.2 mm
- net NP11: track 78.7 -> 72.5 mm, vias 1 -> 0
- net VCCLED: track 12.3 -> 18.1 mm
- net VCC: track 113.9 -> 109.5 mm, vias 1 -> 0
- net NP7: track 44.9 -> 49.1 mm
- net NP10: track 63.5 -> 59.4 mm
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Other:
- board text added: "1Wire"
- board text added: "2-102"
- board text added: "2-104"
- board text added: "BLU"
- board text added: "GRN"
- board text removed: "1-Wire"
- board text removed: "102"
- board text removed: "104"
