File: Peripherals/PixelDrive/hardware/logicboard/pxdr-001.sch (EAGLE design)
At the start: 10 parts

Commit message: First try.
Parts:
- removed SV0: (no value), con-ml:ML34LE
- removed SV3: (no value), con-ml:ML14LE
- added J1: (no value), SparkFun-Connectors:CONN_04JST-PTH
- added J2: (no value), SparkFun-Connectors:CONN_05JST
- added J3: (no value), SparkFun-Connectors:CONN_03JST-PTH
- added SV2: (no value), con-ml:ML40LE
Connections:
- removed net GB00: SV0-1.S, SV3-1.S
- removed net GB01: SV0-3.S, SV3-3.S
- removed net GB02: SV0-5.S, SV3-7.S
- removed net GB03: SV0-7.S, SV3-9.S
- removed net GB04: SV0-9.S, SV3-11.S
- removed net GB05: SV0-11.S, SV3-2.S
- removed net GB06: SV0-13.S, SV3-4.S
- removed net GB07: SV0-15.S, SV3-6.S
- removed net GB08: SV0-19.S, SV3-8.S
- removed net GB09: SV0-21.S, SV3-10.S
- removed net GB10: SV0-23.S, SV3-12.S
- removed net GB11: SV0-25.S, SV3-14.S
- removed net GB12: SV0-27.S, SV1-2.S
- removed net GB13: SV0-29.S, SV1-6.S
- removed net GB14: SV0-31.S, SV1-10.S
- removed net GB15: SV0-33.S, SV1-14.S
- new net NP1: SV1-2.S, SV2-2.S
- new net NP10: J1.4, SV2-29.S
- new net NP11: J2.2, SV2-32.S
- new net NP12: J2.3, SV2-35.S
- new net NP13: J2.4, SV2-38.S
- new net NP14: J3.2, SV2-40.S
- new net NP2: SV1-6.S, SV2-5.S
- new net NP3: SV1-10.S, SV2-8.S
- new net NP4: SV1-14.S, SV2-11.S
- new net NP5: SV1-3.S, SV2-14.S
- new net NP6: SV1-7.S, SV2-17.S
- new net NP7: SV1-11.S, SV2-20.S
- new net NP8: SV1-15.S, SV2-23.S
- new net NP9: J1.3, SV2-26.S
- net GND: now also J1.1, J2.1, J3.1, SV2-1.S, SV2-10.S, SV2-13.S, SV2-16.S, SV2-19.S, SV2-22.S, SV2-25.S, SV2-28.S, SV2-31.S, SV2-34.S, SV2-37.S, SV2-4.S, SV2-7.S; no longer SV0-10.S, SV0-12.S, SV0-14.S, SV0-16.S, SV0-18.S, SV0-2.S, SV0-20.S, SV0-22.S, SV0-24.S, SV0-26.S, SV0-28.S, SV0-30.S, SV0-32.S, SV0-34.S, SV0-4.S, SV0-6.S, SV0-8.S, SV3-5.S
- net VCC: now also J1.2, J2.5, J3.3; no longer SV3-13.S
- net VCC/2: now also SV2-12.S, SV2-15.S, SV2-18.S, SV2-21.S, SV2-24.S, SV2-27.S, SV2-3.S, SV2-30.S, SV2-33.S, SV2-36.S, SV2-39.S, SV2-6.S, SV2-9.S

Commit message: Second shot.
Connections:
- removed net NP11: J2.2, SV2-32.S
- removed net NP12: J2.3, SV2-35.S
- removed net NP13: J2.4, SV2-38.S
- removed net NP14: J3.2, SV2-40.S
- new net DIGITAL7: J2.4, SV2-32.S
- new net SCL: J2.3, SV2-36.S
- new net SDA: J2.2, SV2-35.S
- new net THS: J3.2, SV2-39.S
- net GND: now also SV2-38.S; no longer SV2-37.S
- net VCC: now also SV2-33.S, SV2-37.S, SV2-40.S
- net VCC/2: no longer SV2-33.S, SV2-36.S, SV2-39.S
Changed lines of the file:
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@@
 </segment>
 <segment>
-<pinref part="SV2" gate="-37" pin="S"/>
-<wire x1="38.1" y1="58.42" x2="35.56" y2="58.42" width="0.1524" layer="91"/>
-<label x="35.56" y="58.42" size="0.8128" layer="95" rot="R180" xref="yes"/>
+<pinref part="SV2" gate="-38" pin="S"/>
+<wire x1="38.1" y1="53.34" x2="35.56" y2="53.34" width="0.1524" layer="91"/>
+<label x="35.56" y="53.34" size="0.8128" layer="95" rot="R180" xref="yes"/>
 </segment>
 </net>
@@
 <label x="35.56" y="93.98" size="0.8128" layer="95" rot="R180" xref="yes"/>
 </segment>
-<segment>
-<pinref part="SV2" gate="-33" pin="S"/>
-<wire x1="38.1" y1="78.74" x2="35.56" y2="78.74" width="0.1524" layer="91"/>
-<label x="35.56" y="78.74" size="0.8128" layer="95" rot="R180" xref="yes"/>
-</segment>
-<segment>
-<pinref part="SV2" gate="-36" pin="S"/>
-<wire x1="38.1" y1="63.5" x2="35.56" y2="63.5" width="0.1524" layer="91"/>
-<label x="35.56" y="63.5" size="0.8128" layer="95" rot="R180" xref="yes"/>
-</segment>
-<segment>
-<pinref part="SV2" gate="-39" pin="S"/>
-<wire x1="38.1" y1="48.26" x2="35.56" y2="48.26" width="0.1524" layer="91"/>
-<label x="35.56" y="48.26" size="0.8128" layer="95" rot="R180" xref="yes"/>
-</segment>
 </net>
 <net name="NP1" class="0">
@@
 <wire x1="38.1" y1="99.06" x2="35.56" y2="99.06" width="0.1524" layer="91"/>
 <label x="35.56" y="99.06" size="0.8128" layer="95" rot="R180" xref="yes"/>
-</segment>
-</net>
-<net name="NP11" class="0">
-<segment>
-<pinref part="J2" gate="J1" pin="2"/>
-<wire x1="165.1" y1="137.16" x2="162.56" y2="137.16" width="0.1524" layer="91"/>
-<label x="162.56" y="137.16" size="0.8128" layer="95" rot="R180" xref="yes"/>
-</segment>
-<segment>
-<pinref part="SV2" gate="-32" pin="S"/>
-<wire x1="38.1" y1="83.82" x2="35.56" y2="83.82" width="0.1524" layer="91"/>
-<label x="35.56" y="83.82" size="0.8128" layer="95" rot="R180" xref="yes"/>
-</segment>
-</net>
-<net name="NP12" class="0">
-<segment>
-<pinref part="J2" gate="J1" pin="3"/>
-<wire x1="165.1" y1="134.62" x2="162.56" y2="134.62" width="0.1524" layer="91"/>
-<label x="162.56" y="134.62" size="0.8128" layer="95" rot="R180" xref="yes"/>
-</segment>
-<segment>
-<pinref part="SV2" gate="-35" pin="S"/>
-<wire x1="38.1" y1="68.58" x2="35.56" y2="68.58" width="0.1524" layer="91"/>
-<label x="35.56" y="68.58" size="0.8128" layer="95" rot="R180" xref="yes"/>
-</segment>
-</net>
-<net name="NP13" class="0">
-<segment>
-<pinref part="J2" gate="J1" pin="4"/>
-<wire x1="165.1" y1="132.08" x2="162.56" y2="132.08" width="0.1524" layer="91"/>
-<label x="162.56" y="132.08" size="0.8128" layer="95" rot="R180" xref="yes"/>
-</segment>
-<segment>
-<pinref part="SV2" gate="-38" pin="S"/>
-<wire x1="38.1" y1="53.34" x2="35.56" y2="53.34" width="0.1524" layer="91"/>
-<label x="35.56" y="53.34" size="0.8128" layer="95" rot="R180" xref="yes"/>
-</segment>
-</net>
-<net name="NP14" class="0">
-<segment>
-<pinref part="J3" gate="J1" pin="2"/>
-<wire x1="165.1" y1="114.3" x2="162.56" y2="114.3" width="0.1524" layer="91"/>
-<label x="162.56" y="114.3" size="0.8128" layer="95" rot="R180" xref="yes"/>
-</segment>
-<segment>
-<pinref part="SV2" gate="-40" pin="S"/>
-<wire x1="38.1" y1="43.18" x2="35.56" y2="43.18" width="0.1524" layer="91"/>
-<label x="35.56" y="43.18" size="0.8128" layer="95" rot="R180" xref="yes"/>
 </segment>
 </net>
@@
 <label x="162.56" y="111.76" size="0.8128" layer="95" rot="R180" xref="yes"/>
 </segment>
-</net>
+<segment>
+<pinref part="SV2" gate="-33" pin="S"/>
+<wire x1="38.1" y1="78.74" x2="35.56" y2="78.74" width="0.1524" layer="91"/>
+<label x="35.56" y="78.74" size="0.8128" layer="95" rot="R180" xref="yes"/>
+</segment>
+<segment>
+<pinref part="SV2" gate="-37" pin="S"/>
+<wire x1="38.1" y1="58.42" x2="35.56" y2="58.42" width="0.1524" layer="91"/>
+<label x="35.56" y="58.42" size="0.8128" layer="95" rot="R180" xref="yes"/>
+</segment>
+<segment>
+<pinref part="SV2" gate="-40" pin="S"/>
+<wire x1="38.1" y1="43.18" x2="35.56" y2="43.18" width="0.1524" layer="91"/>
+<label x="35.56" y="43.18" size="0.8128" layer="95" rot="R180" xref="yes"/>
+</segment>
+</net>
+<net name="DIGITAL7" class="0">
+<segment>
+<pinref part="SV2" gate="-32" pin="S"/>
+<wire x1="38.1" y1="83.82" x2="35.56" y2="83.82" width="0.1524" layer="91"/>
+<label x="35.56" y="83.82" size="0.8128" layer="95" rot="R180" xref="yes"/>
+</segment>
+<segment>
+<pinref part="J2" gate="J1" pin="4"/>
+<wire x1="165.1" y1="132.08" x2="162.56" y2="132.08" width="0.1524" layer="91"/>
+<label x="162.56" y="132.08" size="0.8128" layer="95" rot="R180" xref="yes"/>
+</segment>
+</net>
+<net name="SDA" class="0">
+<segment>
+<pinref part="SV2" gate="-35" pin="S"/>
+<wire x1="38.1" y1="68.58" x2="35.56" y2="68.58" width="0.1524" layer="91"/>
+<label x="35.56" y="68.58" size="0.8128" layer="95" rot="R180" xref="yes"/>
+</segment>
+<segment>
+<pinref part="J2" gate="J1" pin="2"/>
+<wire x1="165.1" y1="137.16" x2="162.56" y2="137.16" width="0.1524" layer="91"/>
+<label x="162.56" y="137.16" size="0.8128" layer="95" rot="R180" xref="yes"/>
+</segment>
+</net>
+<net name="SCL" class="0">
+<segment>
+<pinref part="SV2" gate="-36" pin="S"/>
+<wire x1="38.1" y1="63.5" x2="35.56" y2="63.5" width="0.1524" layer="91"/>
+<label x="35.56" y="63.5" size="0.8128" layer="95" rot="R180" xref="yes"/>
+</segment>
+<segment>
+<pinref part="J2" gate="J1" pin="3"/>
+<wire x1="165.1" y1="134.62" x2="162.56" y2="134.62" width="0.1524" layer="91"/>
+<label x="162.56" y="134.62" size="0.8128" layer="95" rot="R180" xref="yes"/>
+</segment>
+</net>
+<net name="THS" class="0">
+<segment>
+<pinref part="SV2" gate="-39" pin="S"/>
+<wire x1="38.1" y1="48.26" x2="35.56" y2="48.26" width="0.1524" layer="91"/>
+<label x="35.56" y="48.26" size="0.8128" layer="95" rot="R180" xref="yes"/>
+</segment>
+<segment>
+<pinref part="J3" gate="J1" pin="2"/>
+<wire x1="165.1" y1="114.3" x2="162.56" y2="114.3" width="0.1524" layer="91"/>
+<label x="162.56" y="114.3" size="0.8128" layer="95" rot="R180" xref="yes"/>
+</segment>
+</net>

Commit message: Third shot.
Connections:
- net DIGITAL7 renamed NP11
- removed net THS: J3.2, SV2-39.S
- new net NP12: J3.2, SV2-35.S
- net GND: now also SV2-37.S; no longer SV2-38.S
- net SCL: now also SV2-39.S; no longer SV2-36.S
- net SDA: now also SV2-38.S; no longer SV2-35.S
- net VCC: no longer SV2-33.S, SV2-37.S
- net VCC/2: now also SV2-33.S, SV2-36.S
Changed lines of the file:
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@@
 </segment>
 <segment>
-<pinref part="SV2" gate="-38" pin="S"/>
-<wire x1="38.1" y1="53.34" x2="35.56" y2="53.34" width="0.1524" layer="91"/>
-<label x="35.56" y="53.34" size="0.8128" layer="95" rot="R180" xref="yes"/>
+<pinref part="SV2" gate="-37" pin="S"/>
+<wire x1="38.1" y1="58.42" x2="35.56" y2="58.42" width="0.1524" layer="91"/>
+<label x="35.56" y="58.42" size="0.8128" layer="95" rot="R180" xref="yes"/>
 </segment>
 </net>
@@
 <label x="35.56" y="93.98" size="0.8128" layer="95" rot="R180" xref="yes"/>
 </segment>
+<segment>
+<pinref part="SV2" gate="-33" pin="S"/>
+<wire x1="38.1" y1="78.74" x2="35.56" y2="78.74" width="0.1524" layer="91"/>
+<label x="35.56" y="78.74" size="0.8128" layer="95" rot="R180" xref="yes"/>
+</segment>
+<segment>
+<pinref part="SV2" gate="-36" pin="S"/>
+<wire x1="38.1" y1="63.5" x2="35.56" y2="63.5" width="0.1524" layer="91"/>
+<label x="35.56" y="63.5" size="0.8128" layer="95" rot="R180" xref="yes"/>
+</segment>
 </net>
 <net name="NP1" class="0">
@@
 </segment>
 <segment>
-<pinref part="SV2" gate="-33" pin="S"/>
-<wire x1="38.1" y1="78.74" x2="35.56" y2="78.74" width="0.1524" layer="91"/>
-<label x="35.56" y="78.74" size="0.8128" layer="95" rot="R180" xref="yes"/>
-</segment>
-<segment>
-<pinref part="SV2" gate="-37" pin="S"/>
-<wire x1="38.1" y1="58.42" x2="35.56" y2="58.42" width="0.1524" layer="91"/>
-<label x="35.56" y="58.42" size="0.8128" layer="95" rot="R180" xref="yes"/>
-</segment>
-<segment>
 <pinref part="SV2" gate="-40" pin="S"/>
 <wire x1="38.1" y1="43.18" x2="35.56" y2="43.18" width="0.1524" layer="91"/>
@@
 </segment>
 </net>
-<net name="DIGITAL7" class="0">
+<net name="SDA" class="0">
+<segment>
+<pinref part="J2" gate="J1" pin="2"/>
+<wire x1="165.1" y1="137.16" x2="162.56" y2="137.16" width="0.1524" layer="91"/>
+<label x="162.56" y="137.16" size="0.8128" layer="95" rot="R180" xref="yes"/>
+</segment>
+<segment>
+<pinref part="SV2" gate="-38" pin="S"/>
+<wire x1="38.1" y1="53.34" x2="35.56" y2="53.34" width="0.1524" layer="91"/>
+<label x="35.56" y="53.34" size="0.8128" layer="95" rot="R180" xref="yes"/>
+</segment>
+</net>
+<net name="SCL" class="0">
+<segment>
+<pinref part="J2" gate="J1" pin="3"/>
+<wire x1="165.1" y1="134.62" x2="162.56" y2="134.62" width="0.1524" layer="91"/>
+<label x="162.56" y="134.62" size="0.8128" layer="95" rot="R180" xref="yes"/>
+</segment>
+<segment>
+<pinref part="SV2" gate="-39" pin="S"/>
+<wire x1="38.1" y1="48.26" x2="35.56" y2="48.26" width="0.1524" layer="91"/>
+<label x="35.56" y="48.26" size="0.8128" layer="95" rot="R180" xref="yes"/>
+</segment>
+</net>
+<net name="NP11" class="0">
+<segment>
+<pinref part="J2" gate="J1" pin="4"/>
+<wire x1="165.1" y1="132.08" x2="162.56" y2="132.08" width="0.1524" layer="91"/>
+<label x="162.56" y="132.08" size="0.8128" layer="95" rot="R180" xref="yes"/>
+</segment>
 <segment>
 <pinref part="SV2" gate="-32" pin="S"/>
@@
 <label x="35.56" y="83.82" size="0.8128" layer="95" rot="R180" xref="yes"/>
 </segment>
-<segment>
-<pinref part="J2" gate="J1" pin="4"/>
-<wire x1="165.1" y1="132.08" x2="162.56" y2="132.08" width="0.1524" layer="91"/>
-<label x="162.56" y="132.08" size="0.8128" layer="95" rot="R180" xref="yes"/>
-</segment>
-</net>
-<net name="SDA" class="0">
+</net>
+<net name="NP12" class="0">
+<segment>
+<pinref part="J3" gate="J1" pin="2"/>
+<wire x1="165.1" y1="114.3" x2="162.56" y2="114.3" width="0.1524" layer="91"/>
+<label x="162.56" y="114.3" size="0.8128" layer="95" rot="R180" xref="yes"/>
+</segment>
 <segment>
 <pinref part="SV2" gate="-35" pin="S"/>
@@
 <label x="35.56" y="68.58" size="0.8128" layer="95" rot="R180" xref="yes"/>
 </segment>
-<segment>
-<pinref part="J2" gate="J1" pin="2"/>
-<wire x1="165.1" y1="137.16" x2="162.56" y2="137.16" width="0.1524" layer="91"/>
-<label x="162.56" y="137.16" size="0.8128" layer="95" rot="R180" xref="yes"/>
-</segment>
-</net>
-<net name="SCL" class="0">
-<segment>
-<pinref part="SV2" gate="-36" pin="S"/>
-<wire x1="38.1" y1="63.5" x2="35.56" y2="63.5" width="0.1524" layer="91"/>
-<label x="35.56" y="63.5" size="0.8128" layer="95" rot="R180" xref="yes"/>
-</segment>
-<segment>
-<pinref part="J2" gate="J1" pin="3"/>
-<wire x1="165.1" y1="134.62" x2="162.56" y2="134.62" width="0.1524" layer="91"/>
-<label x="162.56" y="134.62" size="0.8128" layer="95" rot="R180" xref="yes"/>
-</segment>
-</net>
-<net name="THS" class="0">
-<segment>
-<pinref part="SV2" gate="-39" pin="S"/>
-<wire x1="38.1" y1="48.26" x2="35.56" y2="48.26" width="0.1524" layer="91"/>
-<label x="35.56" y="48.26" size="0.8128" layer="95" rot="R180" xref="yes"/>
-</segment>
-<segment>
-<pinref part="J3" gate="J1" pin="2"/>
-<wire x1="165.1" y1="114.3" x2="162.56" y2="114.3" width="0.1524" layer="91"/>
-<label x="162.56" y="114.3" size="0.8128" layer="95" rot="R180" xref="yes"/>
-</segment>
-</net>
+</net>

Commit message: Fixed some errors.
Parts:
- C1, C2: value (none) -> 104
- J1: value (none) -> GPIO
- J2: value (none) -> MKR
- J3: value (none) -> 1-Wire
- LED1: value (none) -> GRN; device led:LED3MM -> led:LEDB152
- LED2: value (none) -> BLU; device led:LED3MM -> led:LEDB152
- SV2: value (none) -> LightDrive
Changed lines of the file:
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@@
 <part name="SUPPLY2" library="supply2" library_urn="urn:adsk.eagle:library:372" deviceset="GND" device=""/>
 <part name="R1" library="rcl" library_urn="urn:adsk.eagle:library:334" deviceset="R-EU_" device="0204/5" package3d_urn="urn:adsk.eagle:package:23488/1" value="1k"/>
-<part name="LED1" library="led" library_urn="urn:adsk.eagle:library:259" deviceset="LED" device="3MM" package3d_urn="urn:adsk.eagle:package:15797/1"/>
+<part name="LED1" library="led" library_urn="urn:adsk.eagle:library:259" deviceset="LED" device="B152" package3d_urn="urn:adsk.eagle:package:15803/1" value="GRN"/>
 <part name="SUPPLY4" library="supply2" library_urn="urn:adsk.eagle:library:372" deviceset="GND" device=""/>
 <part name="SV1" library="con-ml" library_urn="urn:adsk.eagle:library:164" deviceset="ML16LE" device="" package3d_urn="urn:adsk.eagle:package:8682/1"/>
 <part name="R2" library="rcl" library_urn="urn:adsk.eagle:library:334" deviceset="R-EU_" device="0204/5" package3d_urn="urn:adsk.eagle:package:23488/1" value="1k"/>
-<part name="LED2" library="led" library_urn="urn:adsk.eagle:library:259" deviceset="LED" device="3MM" package3d_urn="urn:adsk.eagle:package:15797/1"/>
-<part name="C1" library="rcl" library_urn="urn:adsk.eagle:library:334" deviceset="C-EU" device="025-025X050" package3d_urn="urn:adsk.eagle:package:23629/2"/>
-<part name="C2" library="rcl" library_urn="urn:adsk.eagle:library:334" deviceset="C-EU" device="025-025X050" package3d_urn="urn:adsk.eagle:package:23629/2"/>
+<part name="LED2" library="led" library_urn="urn:adsk.eagle:library:259" deviceset="LED" device="B152" package3d_urn="urn:adsk.eagle:package:15803/1" value="BLU"/>
+<part name="C1" library="rcl" library_urn="urn:adsk.eagle:library:334" deviceset="C-EU" device="025-025X050" package3d_urn="urn:adsk.eagle:package:23629/2" value="104"/>
+<part name="C2" library="rcl" library_urn="urn:adsk.eagle:library:334" deviceset="C-EU" device="025-025X050" package3d_urn="urn:adsk.eagle:package:23629/2" value="104"/>
 <part name="SUPPLY5" library="supply2" library_urn="urn:adsk.eagle:library:372" deviceset="GND" device=""/>
 <part name="SUPPLY6" library="supply2" library_urn="urn:adsk.eagle:library:372" deviceset="GND" device=""/>
-<part name="J1" library="SparkFun-Connectors" library_urn="urn:adsk.eagle:library:513" deviceset="CONN_04" device="JST-PTH" package3d_urn="urn:adsk.eagle:package:38101/2"/>
-<part name="J2" library="SparkFun-Connectors" library_urn="urn:adsk.eagle:library:513" deviceset="CONN_05" device="JST" package3d_urn="urn:adsk.eagle:package:38120/2"/>
-<part name="SV2" library="con-ml" library_urn="urn:adsk.eagle:library:164" deviceset="ML40LE" device="" package3d_urn="urn:adsk.eagle:package:8688/1"/>
-<part name="J3" library="SparkFun-Connectors" library_urn="urn:adsk.eagle:library:513" deviceset="CONN_03" device="JST-PTH" package3d_urn="urn:adsk.eagle:package:38069/2"/>
+<part name="J1" library="SparkFun-Connectors" library_urn="urn:adsk.eagle:library:513" deviceset="CONN_04" device="JST-PTH" package3d_urn="urn:adsk.eagle:package:38101/2" value="GPIO"/>
+<part name="J2" library="SparkFun-Connectors" library_urn="urn:adsk.eagle:library:513" deviceset="CONN_05" device="JST" package3d_urn="urn:adsk.eagle:package:38120/2" value="MKR"/>
+<part name="SV2" library="con-ml" library_urn="urn:adsk.eagle:library:164" deviceset="ML40LE" device="" package3d_urn="urn:adsk.eagle:package:8688/1" value="LightDrive"/>
+<part name="J3" library="SparkFun-Connectors" library_urn="urn:adsk.eagle:library:513" deviceset="CONN_03" device="JST-PTH" package3d_urn="urn:adsk.eagle:package:38069/2" value="1-Wire"/>
 </parts>
 <sheets>
