File: Vii2/hardware/logicboard/p7ii-001.brd (EAGLE design)
At the start: 91 x 90 mm, 76 parts, among them IC1 74LS06N, IC2 4066N, J1 MKR, J10 1-Wire, J2 GPIO, J20 GPIO, J3 Vcc, J4** RLY2, J5 SPI, J6 LED, J7 DIN5, J8 DIN5, J9 DIN5, K1 G5V1, Q1 220mA/50V/3.5Ω, Q2 220mA/50V/3.5Ω, T1 2SC1815

Commit message: 1st try.
Parts:
- removed C10: 100n, rcl:C025-024X044
- removed C5, C7: 10n, resistor:C025-024X044
- removed D2: (no value), SparkFun-DiscreteSemi:DIODE-1N4148
- removed IC1: 74LS06N, 74xx-us:DIL14
- removed IC2: 4066N, 40xx:DIL14
- removed J4**: RLY2, SparkFun-Connectors:JST-3-PTH-NS
- removed J8, J9: DIN5, SparkFun-Connectors:DIN5-RA-PTH
- removed JP4: RLYJMP, jumper:JP1
- removed K1: G5V1, relay:G5V1
- removed R1: 1k, resistor:0204/5
- removed R2: 47k, resistor:0204/5
- removed RN1: 10k, resistor-net:RN-5
- removed RN2: 4.7k, resistor-net:RN-5
- removed RN4: 220, resistor-dil:DIL16
- removed RZ0, RZ01, RZ02, RZ03, RZ04, RZ3**, RZ4**: Inf, rcl:M2012
- removed SV3: Testport II, pinhead:2X07
- removed T1: 2SC1815, transistor:TO92-ECB
- added D10, D4, D5, D6, D7, D8, D9: 200mA/100V/1V, SparkFun-DiscreteSemi:DIODE-1N4148
- added Q3, Q4, Q5, Q6, Q7, Q8, Q9: 60V/32A/35mΩ, SparkFun-DiscreteSemi:TO220V
- added SV2: (no value), con-ml:ML34L
- R3: value 1k -> 220
- S2: value MIDIPHANTOM -> (none); device switch-dil:DIP04YL -> switch-dil:DIP02YL
- SV1: device con-ml:ML16L -> con-ml:ML14
- moved J7 96.9 mm to (62.0, 90.0), turned to 180 degrees
- moved SV1 55.4 mm to (55.5, 24.0)
- moved R4 32.2 mm to (16.0, 37.0)
- moved R5 32.2 mm to (16.0, 40.0)
- moved D3 28.5 mm to (26.0, 40.0), turned to 0 degrees
- moved OK1 24.0 mm to (37.0, 35.0)
- moved C6 23.5 mm to (44.0, 35.0)
- moved R3 22.9 mm to (26.0, 37.0), turned to 0 degrees
- moved S2 2.54 mm to (6.50, 20.0)
Connections:
- removed net ANLG0R: IC2.2, RZ01.1, SV1.3
- removed net ANLG1R: IC2.3, RZ02.1, SV1.7
- removed net ANLG2R: IC2.9, RZ03.1, SV1.11
- removed net ANLG3R: IC2.10, RZ04.1, SV1.15
- removed net MIDIOUTGND: J8.1, J9.1, S2.3
- removed net MIDIOUTV+: J8.3, J9.3, S2.4
- removed net MNTRA: OK1.4, RN4.16
- removed net MO2RTN: RN4.9
- removed net MO2RTNRAW: IC1.12, RN4.8
- removed net MO2SND: RN4.10
- removed net MORTN: J9.5, RN4.13
- removed net MORTNRAW: IC1.10, RN4.4
- removed net MOSND: J9.4, RN4.14
- removed net MTRTN: J8.5, RN4.11
- removed net MTRTNRAW: IC1.8, RN4.6
- removed net MTSND: J8.4, RN4.12
- removed net NMO2RTN: IC1.13, IC1.6, RN2.5
- removed net NMORTN: IC1.11, IC1.4, RN2.4
- removed net NMTRTN: IC1.2, IC1.9, RN2.3
- removed net RLYDRV: R1.1, R2.2, T1.B
- removed net RLYOUT: J4**.1, K1.10
- removed net RLYOUT1: J4**.2, RZ3**.2
- removed net RLYOUT2: J4**.3, RZ4**.2
- removed net RLYSNK: D2.A, K1.9, T1.C
- removed net VOUTRAW: C3.1, C4.1, D1.A, J3.2, JP4.1, K1.5, K1.6, RZ0.2, RZ3**.1, V1.OUT
- removed net VOUTRAW2: F1.1, JP4.2, K1.1, RZ0.1, RZ4**.1
- new net LD00: D4.A, Q3.2, SV2.1
- new net LD01: D5.A, Q4.2, SV2.3
- new net LD02: D6.A, Q5.2, SV2.5
- new net LD03: D7.A, Q6.2, SV2.7
- new net LD04: D8.A, Q7.2, SV2.9
- new net LD05: D9.A, Q8.2, SV2.11
- new net LD06: D10.A, Q9.2, SV2.13
- new net N$2: F1.1, J0.3
- net ANLG0: no longer IC2.1, RN1.2, RZ01.2
- net ANLG1: no longer IC2.4, RN1.3, RZ02.2
- net ANLG2: no longer IC2.8, RN1.4, RZ03.2
- net ANLG3: no longer IC2.11, RN1.5, RZ04.2
- net AREF: no longer C10.1, R3.1
- net D7GATE: now also SV1.4; no longer IC2.12, IC2.13, IC2.5, IC2.6, SV3.11
- net DTCT0: now also Q5.1, SV1.7; no longer SV1.2, SV3.8
- net DTCT1: now also Q6.1, SV1.5; no longer SV1.6, SV3.10
- net DTCT2: now also Q7.1, SV1.3; no longer SV1.10, SV3.12
- net DTCT3: now also SV1.1; no longer SV1.14, SV3.14
- net GND: now also OK1.4, Q3.3, Q4.3, Q5.3, Q6.3, Q7.3, Q8.3, Q9.3, S2.4, SV1.10, SV2.34; no longer C10.2, C5.2, C7.2, IC1.7, IC2.7, J8.2, J9.2, R2.1, RN1.1, S2.6, S2.8, SV1.1, SV1.13, SV1.5, SV1.9, SV3.5, T1.E
- net GPIO0: now also Q4.1, SV1.13; no longer SV3.2
- net GPIO1: now also SV1.11; no longer SV3.4
- net LED0: now also Q9.1
- net LED1: now also Q8.1
- net MIDIINSND: now also R3.1; no longer RN4.2
- net MISND: now also R3.2; no longer RN4.15
- net MNTR: now also SV2.33; no longer OK1.6, RN3.5
- net RLY: no longer R1.2
- net RX: now also RN3.5, SV1.12; no longer IC1.1, RN2.2, SV3.3
- net SCL: now also Q3.1, SV1.6; no longer SV3.9
- net SDA: now also SV1.8; no longer SV3.7
- net THS: now also SV1.9; no longer SV3.6
- net TX: now also SV1.14; no longer IC1.3, IC1.5, SV3.1
- net V+: now also F1.2, S2.3; no longer J0.3, S2.5, S2.7
- net VCC: now also SV1.2; no longer C5.1, C7.1, D2.C, IC1.14, IC2.14, K1.2, RN2.1, RN4.3, RN4.5, RN4.7, SV3.13
- net VCC/2: now also D10.C, D4.C, D5.C, D6.C, D7.C, D8.C, D9.C, SV2.10, SV2.12, SV2.14, SV2.16, SV2.18, SV2.2, SV2.20, SV2.22, SV2.24, SV2.26, SV2.28, SV2.30, SV2.32, SV2.4, SV2.6, SV2.8; no longer R3.2, RN4.1, SV1.12, SV1.16, SV1.4, SV1.8
- net VOUT: now also C3.1, C4.1, D1.A, J3.2, V1.OUT; no longer F1.2
Routing:
- net MIDIINV+: track 12.9 -> 128.1 mm, vias 0 -> 3
- net ANLG3: track 103.5 -> 0.00 mm, vias 4 -> 0
- net RLYOUT: track 102.5 -> 0.00 mm, vias 2 -> 0
- net RLYOUT1: track 92.8 -> 0.00 mm, vias 2 -> 0
- net N$2: track 0.00 -> 90.1 mm, vias 0 -> 5
- net RLYOUT2: track 89.4 -> 0.00 mm, vias 4 -> 0
- net VOUT: track 57.4 -> 146.0 mm, vias 0 -> 3
- net ANLG2: track 77.2 -> 0.00 mm, vias 6 -> 0
- net LD00: track 0.00 -> 76.2 mm, vias 0 -> 1
- net MTRTN: track 75.8 -> 0.00 mm, vias 1 -> 0
- net NMTRTN: track 72.2 -> 0.00 mm, vias 1 -> 0
- net LD01: track 0.00 -> 70.8 mm
- net VOUTRAW: track 70.2 -> 0.00 mm, vias 3 -> 0
- net MIDIOUTGND: track 69.1 -> 0.00 mm, vias 1 -> 0
- net MIDIINGND: track 25.6 -> 93.3 mm, vias 0 -> 2
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- removed copper zone on layer 1, net GND
- removed copper zone on layer 16, net GND
Other:
- board text added: "2.0.0-X"
- board text added: "Pineapple Vii"
- board text removed: "00"
- board text removed: "01"
- board text removed: "02"
- board text removed: "03"
- board text removed: "2-M2.5"
- board text removed: "2.9.1-GM"
- board text removed: "4066"
- board text removed: "473"
- board text removed: "7406"
- board text removed: "A0"
- board text removed: "A1"
- board text removed: "A2"
- board text removed: "A3"
- board text removed: "AREF"
- board text removed: "Do not forget installing RN2 to use MIDI"
- board text removed: "G5V-1"
- board text removed: "GeekPort II"
- board text removed: "LED00"
- board text removed: "LED00 monitors Vcc/2"
- board text removed: "Min. requirement for MIDI IN"
- board text removed: "Min. requirement for MIDI OUT"
- board text removed: "NO"
- board text removed: "O2"
- board text removed: "Pineapple IIb"
- board text removed: "RX"
- board text removed: "T"
- board text removed: "TH"
- board text removed: "THRU"
- board text removed: "TX"
- board text removed: "TestPort II"
- board text removed: "To use J4**"

Commit message: Trial. Needs re-number of some parts.
Connections:
- removed net N$2: F1.1, J0.3
- new net VIN0: C1.1, C2.1, D1.C, F1.2, V1.IN
- net V+: now also F1.1, J0.3; no longer C1.1, C2.1, D1.C, F1.2, V1.IN
Routing:
- net N$2: track 90.1 -> 0.00 mm, vias 5 -> 0
- net VCC: track 348.9 -> 271.8 mm
- net V+: track 148.7 -> 203.3 mm
- net VIN0: track 0.00 -> 45.3 mm
- net GND: track 419.8 -> 454.0 mm, vias 6 -> 1
- net GPIO1: track 176.7 -> 150.0 mm, vias 3 -> 6
- net LED0: track 118.2 -> 143.2 mm
- net MIDIINGND: track 93.3 -> 114.0 mm, vias 2 -> 3
- net MIRTN: track 104.8 -> 85.1 mm, vias 0 -> 2
- net LED0A: track 105.7 -> 90.1 mm, vias 2 -> 3
- net SCL: track 207.3 -> 192.5 mm, vias 5 -> 6
- net LED1: track 106.8 -> 95.1 mm, vias 2 -> 3
- net RX: track 93.2 -> 103.7 mm, vias 4 -> 1
- net SDA: track 207.1 -> 198.2 mm, vias 7 -> 8
- net MOSI: track 73.5 -> 81.9 mm, vias 1 -> 0
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- added copper zone on layer 1, net GND
- added copper zone on layer 16, net GND
Other:
- board text added: "LightDrive (1-7)"
- board text added: "MIDI Phantom"
- board text added: "TestPort II"
- board text removed: "I/O"
- board text removed: "Phantom"
