File: Vii2/hardware/logicboard/p7ii-001.brd (EAGLE design)
At the start: 91 x 90 mm, 66 parts, among them J1 MKR, J10 1-Wire, J2 GPIO, J20 GPIO, J3 Vcc, J5 SPI, J6 LED, J7 DIN5, Q1 220mA/50V/3.5Ω, Q2 220mA/50V/3.5Ω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

Commit message: Renumbered.
Parts:
- removed Q3: 60V/32A/35mΩ, SparkFun-DiscreteSemi:TO220V
- added Q10: 60V/32A/35mΩ, SparkFun-DiscreteSemi:TO220V
- moved Q4 6.00 mm to (62.0, 67.0)
- moved Q5 6.00 mm to (62.0, 61.0)
- moved Q6 6.00 mm to (62.0, 55.0)
- moved Q7 6.00 mm to (62.0, 49.0)
- moved Q8 6.00 mm to (62.0, 43.0)
- moved Q9 6.00 mm to (62.0, 37.0)
Connections:
- net DTCT0: now also Q6.1; no longer Q5.1
- net DTCT1: now also Q7.1; no longer Q6.1
- net DTCT2: now also Q8.1; no longer Q7.1
- net GND: now also Q10.3; no longer Q3.3
- net GPIO0: now also Q5.1; no longer Q4.1
- net LD00: now also Q4.2; no longer Q3.2
- net LD01: now also Q5.2; no longer Q4.2
- net LD02: now also Q6.2; no longer Q5.2
- net LD03: now also Q7.2; no longer Q6.2
- net LD04: now also Q8.2; no longer Q7.2
- net LD05: now also Q9.2; no longer Q8.2
- net LD06: now also Q10.2; no longer Q9.2
- net LED0: now also Q10.1; no longer Q9.1
- net LED1: now also Q9.1; no longer Q8.1
- net SCL: now also Q4.1; no longer Q3.1
Other:
- board text added: "03PWM"
- board text added: "05PWM"
- board text added: "06PWM"
- board text added: "09PWM"
- board text added: "10PWM"
- board text added: "11PWM"
- board text added: "13PWM"
