File: Vii2/hardware/logicboard/p7ii-001.sch (EAGLE design)
At the start: 76 parts, among them IC1 74LS06N, IC2 4066N, J1 MKR, J10 1-Wire, J2 GPIO, J20 GPIO, J3 Vcc, J4** RLY2, J5 SPI, J6 LED, J7 DIN5, J8 DIN5, J9 DIN5, K1 G5V1, Q1 220mA/50V/3.5Ω, Q2 220mA/50V/3.5Ω, T1 2SC1815

Commit message: 1st try.
Parts:
- removed C10: 100n, rcl:C-EU025-024X044
- removed C5, C7: 10n, resistor:C-EU025-024X044
- removed D2: DIODE-1N4148, SparkFun-DiscreteSemi:DIODE-1N4148
- removed IC1: 74LS06N, 74xx-us:74LS06N
- removed IC2: 4066N, 40xx:4066N
- removed J4**: RLY2, SparkFun-Connectors:CONN_03JST-PTH-NS
- removed J8, J9: DIN5, SparkFun-Connectors:DIN5
- removed JP4: RLYJMP, jumper:JP1E
- removed K1: G5V1, relay:G5V1
- removed R1: 1k, resistor:R-EU_0204/5
- removed R2: 47k, resistor:R-EU_0204/5
- removed RN1: 10k, resistor-net:RN04
- removed RN2: 4.7k, resistor-net:RN04
- removed RN4: 220, resistor-dil:8R-N
- removed RZ0, RZ01, RZ02, RZ03, RZ04, RZ3**, RZ4**: Inf, rcl:R-EU_M2012
- removed SV3: Testport II, pinhead:PINHD-2X7
- removed T1: 2SC1815, transistor:2SC1815
- added D10, D4, D5, D6, D7, D8, D9: 200mA/100V/1V, SparkFun-DiscreteSemi:DIODE-1N4148
- added Q3, Q4, Q5, Q6, Q7, Q8, Q9: 60V/32A/35mΩ, SparkFun-DiscreteSemi:MOSFET-NCH-FQP30N06L
- added SV2: (no value), con-ml:ML34L
- R3: value 1k -> 220
- S2: value MIDIPHANTOM -> (none); device switch-dil:DIP04YL -> switch-dil:DIP02YL
- SV1: device con-ml:ML16LE -> con-ml:ML14
Connections:
- removed net ANLG0R: IC2A.B, RZ01.1, SV1-3.S
- removed net ANLG1R: IC2B.B, RZ02.1, SV1-7.S
- removed net ANLG2R: IC2C.B, RZ03.1, SV1-11.S
- removed net ANLG3R: IC2D.B, RZ04.1, SV1-15.S
- removed net MIDIOUTGND: J8.1, J9.1, S2.3
- removed net MIDIOUTV+: J8.3, J9.3, S2.4
- removed net MNTRA: OK1B.A2, RN4A.2
- removed net MO2RTN: RN4H.2
- removed net MO2RTNRAW: IC1F.O, RN4H.1
- removed net MO2SND: RN4G.2
- removed net MORTN: J9.5, RN4D.2
- removed net MORTNRAW: IC1E.O, RN4D.1
- removed net MOSND: J9.4, RN4C.2
- removed net MTRTN: J8.5, RN4F.2
- removed net MTRTNRAW: IC1D.O, RN4F.1
- removed net MTSND: J8.4, RN4E.2
- removed net NMO2RTN: IC1C.O, IC1F.I, RN2.5
- removed net NMORTN: IC1B.O, IC1E.I, RN2.4
- removed net NMTRTN: IC1A.O, IC1D.I, RN2.3
- removed net RLYDRV: R1.1, R2.2, T1.B
- removed net RLYOUT: J4**.1, K12.S
- removed net RLYOUT1: J4**.2, RZ3**.2
- removed net RLYOUT2: J4**.3, RZ4**.2
- removed net RLYSNK: D2.A, K11.2, T1.C
- removed net VOUTRAW: C3.1, C4.1, D1.A, J3.2, JP4.1, K12.P, K12.P@1, RZ0.2, RZ3**.1, V1.OUT
- removed net VOUTRAW2: F1.1, JP4.2, K12.O, RZ0.1, RZ4**.1
- new net LD00: D4.A, Q3.D, SV2.1
- new net LD01: D5.A, Q4.D, SV2.3
- new net LD02: D6.A, Q5.D, SV2.5
- new net LD03: D7.A, Q6.D, SV2.7
- new net LD04: D8.A, Q7.D, SV2.9
- new net LD05: D9.A, Q8.D, SV2.11
- new net LD06: D10.A, Q9.D, SV2.13
- new net N$2: F1.1, J0.3
- net ANLG0: no longer IC2A.A, RN1.2, RZ01.2
- net ANLG1: no longer IC2B.A, RN1.3, RZ02.2
- net ANLG2: no longer IC2C.A, RN1.4, RZ03.2
- net ANLG3: no longer IC2D.A, RN1.5, RZ04.2
- net AREF: no longer C10.1, R3.1
- net D7GATE: now also SV1.4; no longer IC2A.C, IC2B.C, IC2C.C, IC2D.C, SV3.11
- net DTCT0: now also Q5.G, SV1.7; no longer SV1-2.S, SV3.8
- net DTCT1: now also Q6.G, SV1.5; no longer SV1-6.S, SV3.10
- net DTCT2: now also Q7.G, SV1.3; no longer SV1-10.S, SV3.12
- net DTCT3: now also SV1.1; no longer SV1-14.S, SV3.14
- net GND: now also OK1B.A2, Q3.S, Q4.S, Q5.S, Q6.S, Q7.S, Q8.S, Q9.S, S2.4, SV1.10, SV2.34; no longer C10.2, C5.2, C7.2, IC2P.VSS, J8.2, J9.2, R2.1, RN1.1, S2.6, S2.8, SV1-1.S, SV1-13.S, SV1-5.S, SV1-9.S, SV3.5, T1.E
- net GPIO0: now also Q4.G, SV1.13; no longer SV3.2
- net GPIO1: now also SV1.11; no longer SV3.4
- net LED0: now also Q9.G
- net LED1: now also Q8.G
- net MIDIINSND: now also R3.1; no longer RN4B.1
- net MISND: now also R3.2; no longer RN4B.2
- net MNTR: now also SV2.33; no longer OK1B.VO2, RN3.5
- net RLY: no longer R1.2
- net RX: now also RN3.5, SV1.12; no longer IC1A.I, RN2.2, SV3.3
- net SCL: now also Q3.G, SV1.6; no longer SV3.9
- net SDA: now also SV1.8; no longer SV3.7
- net THS: now also SV1.9; no longer SV3.6
- net TX: now also SV1.14; no longer IC1B.I, IC1C.I, SV3.1
- net V+: now also F1.2, S2.3; no longer J0.3, S2.5, S2.7
- net VCC: now also SV1.2; no longer C5.1, C7.1, D2.C, IC2P.VDD, K11.1, RN2.1, RN4C.1, RN4E.1, RN4G.1, SV3.13
- net VCC/2: now also D10.C, D4.C, D5.C, D6.C, D7.C, D8.C, D9.C, SV2.10, SV2.12, SV2.14, SV2.16, SV2.18, SV2.2, SV2.20, SV2.22, SV2.24, SV2.26, SV2.28, SV2.30, SV2.32, SV2.4, SV2.6, SV2.8; no longer R3.2, RN4A.1, SV1-12.S, SV1-16.S, SV1-4.S, SV1-8.S
- net VOUT: now also C3.1, C4.1, D1.A, J3.2, V1.OUT; no longer F1.2
Other:
- moved on the sheet: C1, C2, C3, C4, D3, F1, OK1A, OK1B, R3, RN3, V1

Commit message: Trial. Needs re-number of some parts.
Connections:
- removed net N$2: F1.1, J0.3
- new net VIN0: C1.1, C2.1, D1.C, F1.2, V1.IN
- net V+: now also F1.1, J0.3; no longer C1.1, C2.1, D1.C, F1.2, V1.IN
Other:
- moved on the sheet: F1
Changed lines of the file:
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@@
 <attribute name="VALUE" x="101.6" y="190.5" size="1.778" layer="96" align="bottom-center"/>
 </instance>
-<instance part="F1" gate="1" x="50.8" y="200.66" smashed="yes">
-<attribute name="NAME" x="50.8" y="203.2" size="1.778" layer="95" align="bottom-center"/>
-<attribute name="VALUE" x="50.8" y="198.12" size="1.778" layer="96" align="bottom-center"/>
+<instance part="F1" gate="1" x="60.96" y="200.66" smashed="yes">
+<attribute name="NAME" x="60.96" y="203.2" size="1.778" layer="95" align="bottom-center"/>
+<attribute name="VALUE" x="60.96" y="198.12" size="1.778" layer="96" align="bottom-center"/>
 </instance>
 <instance part="H1" gate="G$1" x="27.94" y="137.16" smashed="yes"/>
@@
 <attribute name="VALUE" x="60.96" y="241.3" size="1.778" layer="96" rot="R90"/>
 </instance>
-<instance part="P+3" gate="1" x="58.42" y="246.38" smashed="yes">
-<attribute name="VALUE" x="55.88" y="243.84" size="1.778" layer="96" rot="R90"/>
+<instance part="P+3" gate="1" x="45.72" y="246.38" smashed="yes">
+<attribute name="VALUE" x="43.18" y="243.84" size="1.778" layer="96" rot="R90"/>
 </instance>
 <instance part="J6" gate="J$1" x="66.04" y="20.32" smashed="yes">
@@
 <attribute name="NAME" x="63.5" y="25.908" size="1.778" layer="95" font="vector"/>
 </instance>
-<instance part="SUPPLY8" gate="G$1" x="60.96" y="248.92" smashed="yes">
-<attribute name="VALUE" x="60.96" y="254" size="1.778" layer="96" align="bottom-center"/>
+<instance part="SUPPLY8" gate="G$1" x="55.88" y="243.84" smashed="yes">
+<attribute name="VALUE" x="55.88" y="248.92" size="1.778" layer="96" align="bottom-center"/>
 </instance>
 <instance part="SUPPLY10" gate="G$1" x="119.38" y="53.34" smashed="yes">
@@
 <wire x1="45.72" y1="195.58" x2="45.72" y2="187.96" width="0.1524" layer="91"/>
 <junction x="45.72" y="195.58"/>
-<wire x1="45.72" y1="187.96" x2="60.96" y2="187.96" width="0.1524" layer="91"/>
+<wire x1="45.72" y1="187.96" x2="50.8" y2="187.96" width="0.1524" layer="91"/>
 <junction x="76.2" y="187.96"/>
 <pinref part="JP5" gate="A" pin="1"/>
-<wire x1="60.96" y1="187.96" x2="76.2" y2="187.96" width="0.1524" layer="91"/>
-<wire x1="33.02" y1="231.14" x2="60.96" y2="231.14" width="0.1524" layer="91"/>
-<wire x1="60.96" y1="231.14" x2="60.96" y2="187.96" width="0.1524" layer="91"/>
-<junction x="60.96" y="187.96"/>
+<wire x1="50.8" y1="187.96" x2="76.2" y2="187.96" width="0.1524" layer="91"/>
+<wire x1="33.02" y1="231.14" x2="50.8" y2="231.14" width="0.1524" layer="91"/>
+<wire x1="50.8" y1="231.14" x2="50.8" y2="187.96" width="0.1524" layer="91"/>
+<junction x="50.8" y="187.96"/>
 </segment>
 <segment>
@@
 <pinref part="JP1" gate="A" pin="3"/>
 <pinref part="JP5" gate="A" pin="2"/>
-<wire x1="33.02" y1="233.68" x2="60.96" y2="233.68" width="0.1524" layer="91"/>
+<wire x1="33.02" y1="233.68" x2="55.88" y2="233.68" width="0.1524" layer="91"/>
 <pinref part="SUPPLY8" gate="G$1" pin="VCC"/>
-<wire x1="60.96" y1="233.68" x2="81.28" y2="233.68" width="0.1524" layer="91"/>
-<wire x1="60.96" y1="246.38" x2="60.96" y2="233.68" width="0.1524" layer="91"/>
-<junction x="60.96" y="233.68"/>
+<wire x1="55.88" y1="233.68" x2="81.28" y2="233.68" width="0.1524" layer="91"/>
+<wire x1="55.88" y1="241.3" x2="55.88" y2="233.68" width="0.1524" layer="91"/>
+<junction x="55.88" y="233.68"/>
 <label x="66.04" y="233.68" size="1.778" layer="95"/>
 </segment>
@@
 <segment>
 <pinref part="JP1" gate="A" pin="1"/>
-<wire x1="81.28" y1="236.22" x2="58.42" y2="236.22" width="0.1524" layer="91"/>
+<wire x1="81.28" y1="236.22" x2="45.72" y2="236.22" width="0.1524" layer="91"/>
 <pinref part="P+3" gate="1" pin="V+"/>
-<wire x1="58.42" y1="243.84" x2="58.42" y2="236.22" width="0.1524" layer="91"/>
-<junction x="58.42" y="236.22"/>
+<wire x1="45.72" y1="243.84" x2="45.72" y2="236.22" width="0.1524" layer="91"/>
+<junction x="45.72" y="236.22"/>
 <pinref part="JP5" gate="A" pin="3"/>
-<wire x1="33.02" y1="236.22" x2="58.42" y2="236.22" width="0.1524" layer="91"/>
+<wire x1="33.02" y1="236.22" x2="45.72" y2="236.22" width="0.1524" layer="91"/>
 <label x="66.04" y="236.22" size="1.778" layer="95"/>
-<pinref part="C1" gate="G$1" pin="1"/>
-<pinref part="D1" gate="G$1" pin="C"/>
-<wire x1="83.82" y1="205.74" x2="91.44" y2="205.74" width="0.1524" layer="91"/>
-<pinref part="V1" gate="1" pin="IN"/>
-<wire x1="86.36" y1="200.66" x2="83.82" y2="200.66" width="0.1524" layer="91"/>
-<pinref part="C2" gate="G$1" pin="1"/>
-<wire x1="83.82" y1="198.12" x2="83.82" y2="200.66" width="0.1524" layer="91"/>
-<junction x="83.82" y="200.66"/>
-<wire x1="83.82" y1="200.66" x2="83.82" y2="205.74" width="0.1524" layer="91"/>
-<wire x1="83.82" y1="200.66" x2="76.2" y2="200.66" width="0.1524" layer="91"/>
-<wire x1="76.2" y1="200.66" x2="76.2" y2="198.12" width="0.1524" layer="91"/>
-<label x="78.74" y="200.66" size="1.778" layer="95"/>
-<pinref part="F1" gate="1" pin="2"/>
-<wire x1="76.2" y1="200.66" x2="58.42" y2="200.66" width="0.1524" layer="91"/>
-<junction x="76.2" y="200.66"/>
-<wire x1="58.42" y1="200.66" x2="55.88" y2="200.66" width="0.1524" layer="91"/>
-<wire x1="58.42" y1="236.22" x2="58.42" y2="200.66" width="0.1524" layer="91"/>
-<junction x="58.42" y="200.66"/>
+<pinref part="J0" gate="G$1" pin="3"/>
+<pinref part="F1" gate="1" pin="1"/>
+<wire x1="55.88" y1="200.66" x2="45.72" y2="200.66" width="0.1524" layer="91"/>
+<wire x1="45.72" y1="200.66" x2="38.1" y2="200.66" width="0.1524" layer="91"/>
+<wire x1="45.72" y1="200.66" x2="45.72" y2="236.22" width="0.1524" layer="91"/>
+<junction x="45.72" y="200.66"/>
+<junction x="45.72" y="236.22"/>
 </segment>
 <segment>
@@
 </segment>
 </net>
-<net name="N$2" class="4">
-<segment>
-<pinref part="J0" gate="G$1" pin="3"/>
-<pinref part="F1" gate="1" pin="1"/>
-<wire x1="45.72" y1="200.66" x2="38.1" y2="200.66" width="0.1524" layer="91"/>
-</segment>
-</net>
+<net name="VIN0" class="4">
+<segment>
+<pinref part="F1" gate="1" pin="2"/>
+<pinref part="C1" gate="G$1" pin="1"/>
+<pinref part="D1" gate="G$1" pin="C"/>
+<wire x1="83.82" y1="205.74" x2="91.44" y2="205.74" width="0.1524" layer="91"/>
+<pinref part="V1" gate="1" pin="IN"/>
+<wire x1="86.36" y1="200.66" x2="83.82" y2="200.66" width="0.1524" layer="91"/>
+<pinref part="C2" gate="G$1" pin="1"/>
+<wire x1="83.82" y1="198.12" x2="83.82" y2="200.66" width="0.1524" layer="91"/>
+<junction x="83.82" y="200.66"/>
+<wire x1="83.82" y1="200.66" x2="83.82" y2="205.74" width="0.1524" layer="91"/>
+<wire x1="83.82" y1="200.66" x2="76.2" y2="200.66" width="0.1524" layer="91"/>
+<wire x1="76.2" y1="200.66" x2="76.2" y2="198.12" width="0.1524" layer="91"/>
+<junction x="76.2" y="200.66"/>
+<wire x1="76.2" y1="200.66" x2="66.04" y2="200.66" width="0.1524" layer="91"/>
+<label x="78.74" y="200.66" size="1.778" layer="95"/>
+</segment>
+</net>

Commit message: Renumbered.
Parts:
- removed Q3: 60V/32A/35mΩ, SparkFun-DiscreteSemi:MOSFET-NCH-FQP30N06L
- added Q10: 60V/32A/35mΩ, SparkFun-DiscreteSemi:MOSFET-NCH-FQP30N06L
Connections:
- net DTCT0: now also Q6.G; no longer Q5.G
- net DTCT1: now also Q7.G; no longer Q6.G
- net DTCT2: now also Q8.G; no longer Q7.G
- net GND: now also Q10.S; no longer Q3.S
- net GPIO0: now also Q5.G; no longer Q4.G
- net LD00: now also Q4.D; no longer Q3.D
- net LD01: now also Q5.D; no longer Q4.D
- net LD02: now also Q6.D; no longer Q5.D
- net LD03: now also Q7.D; no longer Q6.D
- net LD04: now also Q8.D; no longer Q7.D
- net LD05: now also Q9.D; no longer Q8.D
- net LD06: now also Q10.D; no longer Q9.D
- net LED0: now also Q10.G; no longer Q9.G
- net LED1: now also Q9.G; no longer Q8.G
- net SCL: now also Q4.G; no longer Q3.G
Other:
- moved on the sheet: Q4, Q5, Q6, Q7, Q8, Q9
Changed lines of the file:
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@@
 <part name="JMP3" library="jump-0r-smd" library_urn="urn:adsk.eagle:library:251" deviceset="0R-JUMP" device="A" package3d_urn="urn:adsk.eagle:package:15385/1"/>
 <part name="SV2" library="con-ml" library_urn="urn:adsk.eagle:library:164" deviceset="ML34L" device="" package3d_urn="urn:adsk.eagle:package:8689/1"/>
-<part name="Q3" library="SparkFun-DiscreteSemi" library_urn="urn:adsk.eagle:library:514" deviceset="MOSFET-NCH" device="-FQP30N06L" package3d_urn="urn:adsk.eagle:package:38447/1" value="60V/32A/35mΩ"/>
 <part name="Q4" library="SparkFun-DiscreteSemi" library_urn="urn:adsk.eagle:library:514" deviceset="MOSFET-NCH" device="-FQP30N06L" package3d_urn="urn:adsk.eagle:package:38447/1" value="60V/32A/35mΩ"/>
 <part name="Q5" library="SparkFun-DiscreteSemi" library_urn="urn:adsk.eagle:library:514" deviceset="MOSFET-NCH" device="-FQP30N06L" package3d_urn="urn:adsk.eagle:package:38447/1" value="60V/32A/35mΩ"/>
@@
 <part name="Q8" library="SparkFun-DiscreteSemi" library_urn="urn:adsk.eagle:library:514" deviceset="MOSFET-NCH" device="-FQP30N06L" package3d_urn="urn:adsk.eagle:package:38447/1" value="60V/32A/35mΩ"/>
 <part name="Q9" library="SparkFun-DiscreteSemi" library_urn="urn:adsk.eagle:library:514" deviceset="MOSFET-NCH" device="-FQP30N06L" package3d_urn="urn:adsk.eagle:package:38447/1" value="60V/32A/35mΩ"/>
+<part name="Q10" library="SparkFun-DiscreteSemi" library_urn="urn:adsk.eagle:library:514" deviceset="MOSFET-NCH" device="-FQP30N06L" package3d_urn="urn:adsk.eagle:package:38447/1" value="60V/32A/35mΩ"/>
 <part name="D4" library="SparkFun-DiscreteSemi" library_urn="urn:adsk.eagle:library:514" deviceset="DIODE" device="-1N4148" package3d_urn="urn:adsk.eagle:package:38452/1" value="200mA/100V/1V"/>
 <part name="D5" library="SparkFun-DiscreteSemi" library_urn="urn:adsk.eagle:library:514" deviceset="DIODE" device="-1N4148" package3d_urn="urn:adsk.eagle:package:38452/1" value="200mA/100V/1V"/>
@@
 </instance>
 <instance part="D1" gate="G$1" x="93.98" y="205.74" smashed="yes" rot="R180">
+<attribute name="NAME" x="93.98" y="211.328" size="1.778" layer="95" font="vector" rot="R180"/>
 <attribute name="VALUE" x="96.52" y="207.772" size="1.778" layer="96" font="vector" rot="R180" align="top-left"/>
 </instance>
@@
 <attribute name="NAME" x="31.75" y="125.222" size="1.778" layer="95"/>
 </instance>
-<instance part="Q3" gate="NMOS" x="71.12" y="152.4" smashed="yes">
+<instance part="Q4" gate="NMOS" x="71.12" y="152.4" smashed="yes">
 <attribute name="NAME" x="76.2" y="152.4" size="1.778" layer="95" font="vector"/>
 <attribute name="VALUE" x="76.2" y="149.86" size="1.778" layer="96" font="vector"/>
 </instance>
-<instance part="Q4" gate="NMOS" x="104.14" y="152.4" smashed="yes">
+<instance part="Q5" gate="NMOS" x="104.14" y="152.4" smashed="yes">
 <attribute name="NAME" x="109.22" y="152.4" size="1.778" layer="95" font="vector"/>
 <attribute name="VALUE" x="109.22" y="149.86" size="1.778" layer="96" font="vector"/>
 </instance>
-<instance part="Q5" gate="NMOS" x="137.16" y="152.4" smashed="yes">
+<instance part="Q6" gate="NMOS" x="137.16" y="152.4" smashed="yes">
 <attribute name="NAME" x="142.24" y="152.4" size="1.778" layer="95" font="vector"/>
 <attribute name="VALUE" x="142.24" y="149.86" size="1.778" layer="96" font="vector"/>
 </instance>
-<instance part="Q6" gate="NMOS" x="170.18" y="152.4" smashed="yes">
+<instance part="Q7" gate="NMOS" x="170.18" y="152.4" smashed="yes">
 <attribute name="NAME" x="175.26" y="152.4" size="1.778" layer="95" font="vector"/>
 <attribute name="VALUE" x="175.26" y="149.86" size="1.778" layer="96" font="vector"/>
 </instance>
-<instance part="Q7" gate="NMOS" x="71.12" y="124.46" smashed="yes">
+<instance part="Q8" gate="NMOS" x="71.12" y="124.46" smashed="yes">
 <attribute name="NAME" x="76.2" y="124.46" size="1.778" layer="95" font="vector"/>
 <attribute name="VALUE" x="76.2" y="121.92" size="1.778" layer="96" font="vector"/>
 </instance>
-<instance part="Q8" gate="NMOS" x="104.14" y="124.46" smashed="yes">
+<instance part="Q9" gate="NMOS" x="104.14" y="124.46" smashed="yes">
 <attribute name="NAME" x="109.22" y="124.46" size="1.778" layer="95" font="vector"/>
 <attribute name="VALUE" x="109.22" y="121.92" size="1.778" layer="96" font="vector"/>
 </instance>
-<instance part="Q9" gate="NMOS" x="137.16" y="124.46" smashed="yes">
+<instance part="Q10" gate="NMOS" x="137.16" y="124.46" smashed="yes">
 <attribute name="NAME" x="142.24" y="124.46" size="1.778" layer="95" font="vector"/>
 <attribute name="VALUE" x="142.24" y="121.92" size="1.778" layer="96" font="vector"/>
@@
 </segment>
 <segment>
-<pinref part="Q3" gate="NMOS" pin="S"/>
+<pinref part="Q4" gate="NMOS" pin="S"/>
 <wire x1="73.66" y1="147.32" x2="73.66" y2="144.78" width="0.1524" layer="91"/>
 <pinref part="SUPPLY4" gate="GND" pin="GND"/>
 </segment>
 <segment>
-<pinref part="Q4" gate="NMOS" pin="S"/>
+<pinref part="Q5" gate="NMOS" pin="S"/>
 <wire x1="106.68" y1="147.32" x2="106.68" y2="144.78" width="0.1524" layer="91"/>
 <pinref part="SUPPLY7" gate="GND" pin="GND"/>
 </segment>
 <segment>
-<pinref part="Q5" gate="NMOS" pin="S"/>
+<pinref part="Q6" gate="NMOS" pin="S"/>
 <wire x1="139.7" y1="147.32" x2="139.7" y2="144.78" width="0.1524" layer="91"/>
 <pinref part="SUPPLY9" gate="GND" pin="GND"/>
 </segment>
 <segment>
-<pinref part="Q6" gate="NMOS" pin="S"/>
+<pinref part="Q7" gate="NMOS" pin="S"/>
 <wire x1="172.72" y1="147.32" x2="172.72" y2="144.78" width="0.1524" layer="91"/>
 <pinref part="SUPPLY11" gate="GND" pin="GND"/>
 </segment>
 <segment>
-<pinref part="Q7" gate="NMOS" pin="S"/>
+<pinref part="Q8" gate="NMOS" pin="S"/>
 <wire x1="73.66" y1="119.38" x2="73.66" y2="116.84" width="0.1524" layer="91"/>
 <pinref part="SUPPLY12" gate="GND" pin="GND"/>
 </segment>
 <segment>
-<pinref part="Q8" gate="NMOS" pin="S"/>
+<pinref part="Q9" gate="NMOS" pin="S"/>
 <wire x1="106.68" y1="119.38" x2="106.68" y2="116.84" width="0.1524" layer="91"/>
 <pinref part="SUPPLY14" gate="GND" pin="GND"/>
 </segment>
 <segment>
-<pinref part="Q9" gate="NMOS" pin="S"/>
+<pinref part="Q10" gate="NMOS" pin="S"/>
 <wire x1="139.7" y1="119.38" x2="139.7" y2="116.84" width="0.1524" layer="91"/>
 <pinref part="SUPPLY15" gate="GND" pin="GND"/>
@@
 </segment>
 <segment>
-<pinref part="Q5" gate="NMOS" pin="G"/>
+<pinref part="Q6" gate="NMOS" pin="G"/>
 <wire x1="132.08" y1="149.86" x2="129.54" y2="149.86" width="0.1524" layer="91"/>
 <label x="129.54" y="149.86" size="0.8128" layer="95" rot="R180" xref="yes"/>
@@
 </segment>
 <segment>
-<pinref part="Q6" gate="NMOS" pin="G"/>
+<pinref part="Q7" gate="NMOS" pin="G"/>
 <wire x1="165.1" y1="149.86" x2="162.56" y2="149.86" width="0.1524" layer="91"/>
 <label x="162.56" y="149.86" size="0.8128" layer="95" rot="R180" xref="yes"/>
@@
 </segment>
 <segment>
-<pinref part="Q7" gate="NMOS" pin="G"/>
+<pinref part="Q8" gate="NMOS" pin="G"/>
 <wire x1="66.04" y1="121.92" x2="63.5" y2="121.92" width="0.1524" layer="91"/>
 <label x="63.5" y="121.92" size="0.8128" layer="95" rot="R180" xref="yes"/>
@@
 </segment>
 <segment>
-<pinref part="Q9" gate="NMOS" pin="G"/>
+<pinref part="Q10" gate="NMOS" pin="G"/>
 <wire x1="132.08" y1="121.92" x2="129.54" y2="121.92" width="0.1524" layer="91"/>
 <label x="129.54" y="121.92" size="0.8128" layer="95" rot="R180" xref="yes"/>
@@
 </segment>
 <segment>
-<pinref part="Q8" gate="NMOS" pin="G"/>
+<pinref part="Q9" gate="NMOS" pin="G"/>
 <wire x1="99.06" y1="121.92" x2="96.52" y2="121.92" width="0.1524" layer="91"/>
 <label x="96.52" y="121.92" size="0.8128" layer="95" rot="R180" xref="yes"/>
@@
 </segment>
 <segment>
-<pinref part="Q4" gate="NMOS" pin="G"/>
+<pinref part="Q5" gate="NMOS" pin="G"/>
 <wire x1="99.06" y1="149.86" x2="96.52" y2="149.86" width="0.1524" layer="91"/>
 <label x="96.52" y="149.86" size="0.8128" layer="95" rot="R180" xref="yes"/>
@@
 </segment>
 <segment>
-<pinref part="Q3" gate="NMOS" pin="G"/>
+<pinref part="Q4" gate="NMOS" pin="G"/>
 <wire x1="66.04" y1="149.86" x2="63.5" y2="149.86" width="0.1524" layer="91"/>
 <label x="63.5" y="149.86" size="0.8128" layer="95" rot="R180" xref="yes"/>
@@
 </segment>
 <segment>
-<pinref part="Q9" gate="NMOS" pin="D"/>
+<pinref part="Q10" gate="NMOS" pin="D"/>
 <wire x1="139.7" y1="129.54" x2="139.7" y2="132.08" width="0.1524" layer="91"/>
 <label x="139.7" y="134.62" size="0.8128" layer="95" rot="R90" xref="yes"/>
@@
 </segment>
 <segment>
-<pinref part="Q8" gate="NMOS" pin="D"/>
+<pinref part="Q9" gate="NMOS" pin="D"/>
 <wire x1="106.68" y1="129.54" x2="106.68" y2="132.08" width="0.1524" layer="91"/>
 <label x="106.68" y="134.62" size="0.8128" layer="95" rot="R90" xref="yes"/>
@@
 </segment>
 <segment>
-<pinref part="Q7" gate="NMOS" pin="D"/>
+<pinref part="Q8" gate="NMOS" pin="D"/>
 <wire x1="73.66" y1="129.54" x2="73.66" y2="132.08" width="0.1524" layer="91"/>
 <label x="73.66" y="134.62" size="0.8128" layer="95" rot="R90" xref="yes"/>
@@
 </segment>
 <segment>
-<pinref part="Q6" gate="NMOS" pin="D"/>
+<pinref part="Q7" gate="NMOS" pin="D"/>
 <wire x1="172.72" y1="157.48" x2="172.72" y2="160.02" width="0.1524" layer="91"/>
 <label x="172.72" y="162.56" size="0.8128" layer="95" rot="R90" xref="yes"/>
@@
 </segment>
 <segment>
-<pinref part="Q5" gate="NMOS" pin="D"/>
+<pinref part="Q6" gate="NMOS" pin="D"/>
 <wire x1="139.7" y1="157.48" x2="139.7" y2="160.02" width="0.1524" layer="91"/>
 <label x="139.7" y="162.56" size="0.8128" layer="95" rot="R90" xref="yes"/>
@@
 </segment>
 <segment>
-<pinref part="Q4" gate="NMOS" pin="D"/>
+<pinref part="Q5" gate="NMOS" pin="D"/>
 <wire x1="106.68" y1="157.48" x2="106.68" y2="160.02" width="0.1524" layer="91"/>
 <label x="106.68" y="162.56" size="0.8128" layer="95" rot="R90" xref="yes"/>
@@
 </segment>
 <segment>
-<pinref part="Q3" gate="NMOS" pin="D"/>
+<pinref part="Q4" gate="NMOS" pin="D"/>
 <wire x1="73.66" y1="157.48" x2="73.66" y2="160.02" width="0.1524" layer="91"/>
 <label x="73.66" y="162.56" size="0.8128" layer="95" rot="R90" xref="yes"/>
