File: Peripherals/ServoGear/hardware/logicboard/srvg-001.brd (EAGLE design)
At the start: 18 x 23 mm, 7 parts

Commit message: Routed.
Parts:
- removed J21, J22, J23, J24: (no value), SparkFun-Connectors:JST-4-PTH-VERT
- added J41, J42, J43: (no value), pinhead:1X03
- moved U$1 13.5 mm to (9.00, 0.50), turned to 0 degrees
- moved LOGO1 9.85 mm to (3.00, 20.0), flipped to the top
Connections:
- net ANLG0: no longer J21.2
- net ANLG1: no longer J22.2
- net ANLG2: no longer J23.2
- net ANLG3: no longer J24.2
- net DTCT0: now also J41.3; no longer J21.1
- net DTCT1: now also J42.3; no longer J22.1
- net DTCT2: now also J43.3; no longer J23.1
- net DTCT3: no longer J24.1
- net GND: now also J41.1, J42.1, J43.1; no longer J21.4, J22.4, J23.4, J24.4
- net VCC: now also J41.2, J42.2, J43.2; no longer J21.3, J22.3, J23.3, J24.3
Routing:
- net DTCT3: track 13.3 -> 0.00 mm
- net ANLG0: track 8.36 -> 0.00 mm
- net ANLG1: track 8.35 -> 0.00 mm
- net ANLG3: track 8.34 -> 0.00 mm
- net ANLG2: track 8.33 -> 0.00 mm
- net DTCT2: track 13.9 -> 8.07 mm
- net VCC: track 42.2 -> 36.7 mm
- net DTCT1: track 13.4 -> 8.56 mm
- net DTCT0: track 13.2 -> 9.02 mm
- net GND: track 31.1 -> 35.1 mm
Other:
- board text added: "1"
- board text added: "2"
- board text added: "P"
- board text added: "ServoGear 0.0.1-X"
- board text removed: "A"
- board text removed: "D"
- board text removed: "GroveGear 0.0.1-X"
