File: Peripherals/ServoGear/hardware/logicboard/srvg-001.sch (EAGLE design)
At the start: 7 parts

Commit message: Routed.
Parts:
- removed J21, J22, J23, J24: (no value), SparkFun-Connectors:CONN_04JST-PTH-VERT
- added J41, J42, J43: (no value), pinhead:PINHD-1X3
Connections:
- net ANLG0: no longer J21.2
- net ANLG1: no longer J22.2
- net ANLG2: no longer J23.2
- net ANLG3: no longer J24.2
- net DTCT0: now also J41.3; no longer J21.1
- net DTCT1: now also J42.3; no longer J22.1
- net DTCT2: now also J43.3; no longer J23.1
- net DTCT3: no longer J24.1
- net GND: now also J41.1, J42.1, J43.1; no longer J21.4, J22.4, J23.4, J24.4
- net VCC: now also J41.2, J42.2, J43.2; no longer J21.3, J22.3, J23.3, J24.3
Other:
- note removed: "Pineapple -> Switch 1->1 2->4 4->8 8->2"
Changed lines of the file:
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@@
 <part name="SUPPLY3" library="supply2" library_urn="urn:adsk.eagle:library:372" deviceset="VCC" device=""/>
 <part name="U$1" library="pineapple" deviceset="PINEAPPLE450_SILK" device=""/>
-<part name="J21" library="SparkFun-Connectors" library_urn="urn:adsk.eagle:library:513" deviceset="CONN_04" device="JST-PTH-VERT" package3d_urn="urn:adsk.eagle:package:38102/1"/>
-<part name="J22" library="SparkFun-Connectors" library_urn="urn:adsk.eagle:library:513" deviceset="CONN_04" device="JST-PTH-VERT" package3d_urn="urn:adsk.eagle:package:38102/1"/>
-<part name="J23" library="SparkFun-Connectors" library_urn="urn:adsk.eagle:library:513" deviceset="CONN_04" device="JST-PTH-VERT" package3d_urn="urn:adsk.eagle:package:38102/1"/>
-<part name="J24" library="SparkFun-Connectors" library_urn="urn:adsk.eagle:library:513" deviceset="CONN_04" device="JST-PTH-VERT" package3d_urn="urn:adsk.eagle:package:38102/1"/>
+<part name="J41" library="pinhead" library_urn="urn:adsk.eagle:library:325" deviceset="PINHD-1X3" device="" package3d_urn="urn:adsk.eagle:package:22458/2"/>
+<part name="J42" library="pinhead" library_urn="urn:adsk.eagle:library:325" deviceset="PINHD-1X3" device="" package3d_urn="urn:adsk.eagle:package:22458/2"/>
+<part name="J43" library="pinhead" library_urn="urn:adsk.eagle:library:325" deviceset="PINHD-1X3" device="" package3d_urn="urn:adsk.eagle:package:22458/2"/>
 </parts>
 <sheets>
@@
 <plain>
 <text x="218.44" y="20.32" size="1.778" layer="95">Pineapple IIc 2.5.0-RC</text>
-<text x="55.88" y="152.4" size="1.778" layer="97">Pineapple -&gt; Switch
-1-&gt;1
-2-&gt;4
-4-&gt;8
-8-&gt;2</text>
 <text x="139.7" y="101.6" size="1.778" layer="97">GeekPort II
 1: GND
@@
 </instance>
 <instance part="U$1" gate="G$1" x="241.3" y="142.24" smashed="yes"/>
-<instance part="J21" gate="G$1" x="48.26" y="121.92" smashed="yes">
-<attribute name="VALUE" x="43.18" y="114.554" size="1.778" layer="96" font="vector"/>
-<attribute name="NAME" x="43.18" y="130.048" size="1.778" layer="95" font="vector"/>
+<instance part="J41" gate="A" x="48.26" y="114.3" smashed="yes" rot="R180">
+<attribute name="NAME" x="54.61" y="108.585" size="1.778" layer="95" rot="R180"/>
+<attribute name="VALUE" x="54.61" y="121.92" size="1.778" layer="96" rot="R180"/>
 </instance>
-<instance part="J22" gate="G$1" x="48.26" y="104.14" smashed="yes">
-<attribute name="VALUE" x="43.18" y="96.774" size="1.778" layer="96" font="vector"/>
-<attribute name="NAME" x="43.18" y="112.268" size="1.778" layer="95" font="vector"/>
+<instance part="J42" gate="A" x="48.26" y="101.6" smashed="yes" rot="R180">
+<attribute name="NAME" x="54.61" y="95.885" size="1.778" layer="95" rot="R180"/>
+<attribute name="VALUE" x="54.61" y="109.22" size="1.778" layer="96" rot="R180"/>
 </instance>
-<instance part="J23" gate="G$1" x="48.26" y="86.36" smashed="yes">
-<attribute name="VALUE" x="43.18" y="78.994" size="1.778" layer="96" font="vector"/>
-<attribute name="NAME" x="43.18" y="94.488" size="1.778" layer="95" font="vector"/>
-</instance>
-<instance part="J24" gate="G$1" x="48.26" y="68.58" smashed="yes">
-<attribute name="VALUE" x="43.18" y="61.214" size="1.778" layer="96" font="vector"/>
-<attribute name="NAME" x="43.18" y="76.708" size="1.778" layer="95" font="vector"/>
+<instance part="J43" gate="A" x="48.26" y="88.9" smashed="yes" rot="R180">
+<attribute name="NAME" x="54.61" y="83.185" size="1.778" layer="95" rot="R180"/>
+<attribute name="VALUE" x="54.61" y="96.52" size="1.778" layer="96" rot="R180"/>
 </instance>
 </instances>
@@
 </busses>
 <nets>
-<net name="GND" class="0">
+<net name="GND" class="1">
 <segment>
 <pinref part="SV1" gate="A" pin="1"/>
@@
 </segment>
 <segment>
-<pinref part="J21" gate="G$1" pin="4"/>
-<wire x1="53.34" y1="127" x2="58.42" y2="127" width="0.1524" layer="91"/>
-<label x="58.42" y="127" size="0.8128" layer="95" xref="yes"/>
+<pinref part="J41" gate="A" pin="1"/>
+<wire x1="50.8" y1="111.76" x2="58.42" y2="111.76" width="0.1524" layer="91"/>
+<label x="58.42" y="111.76" size="0.8128" layer="95" xref="yes"/>
 </segment>
 <segment>
-<pinref part="J22" gate="G$1" pin="4"/>
-<wire x1="53.34" y1="109.22" x2="58.42" y2="109.22" width="0.1524" layer="91"/>
-<label x="58.42" y="109.22" size="0.8128" layer="95" xref="yes"/>
+<pinref part="J42" gate="A" pin="1"/>
+<wire x1="50.8" y1="99.06" x2="58.42" y2="99.06" width="0.1524" layer="91"/>
+<label x="58.42" y="99.06" size="0.8128" layer="95" xref="yes"/>
 </segment>
 <segment>
-<pinref part="J23" gate="G$1" pin="4"/>
-<wire x1="53.34" y1="91.44" x2="58.42" y2="91.44" width="0.1524" layer="91"/>
-<label x="58.42" y="91.44" size="0.8128" layer="95" xref="yes"/>
-</segment>
-<segment>
-<pinref part="J24" gate="G$1" pin="4"/>
-<wire x1="53.34" y1="73.66" x2="58.42" y2="73.66" width="0.1524" layer="91"/>
-<label x="58.42" y="73.66" size="0.8128" layer="95" xref="yes"/>
+<pinref part="J43" gate="A" pin="1"/>
+<wire x1="50.8" y1="86.36" x2="58.42" y2="86.36" width="0.1524" layer="91"/>
+<label x="58.42" y="86.36" size="0.8128" layer="95" xref="yes"/>
 </segment>
 </net>
@@
 </segment>
 <segment>
-<pinref part="J21" gate="G$1" pin="1"/>
-<wire x1="53.34" y1="119.38" x2="58.42" y2="119.38" width="0.1524" layer="91"/>
-<label x="58.42" y="119.38" size="0.8128" layer="95" xref="yes"/>
+<pinref part="J41" gate="A" pin="3"/>
+<wire x1="50.8" y1="116.84" x2="58.42" y2="116.84" width="0.1524" layer="91"/>
+<label x="58.42" y="116.84" size="0.8128" layer="95" xref="yes"/>
 </segment>
 </net>
-<net name="VCC" class="0">
+<net name="VCC" class="2">
 <segment>
 <pinref part="SV1" gate="A" pin="4"/>
@@
 </segment>
 <segment>
-<pinref part="J21" gate="G$1" pin="3"/>
-<wire x1="53.34" y1="124.46" x2="58.42" y2="124.46" width="0.1524" layer="91"/>
-<label x="58.42" y="124.46" size="0.8128" layer="95" xref="yes"/>
+<pinref part="J41" gate="A" pin="2"/>
+<wire x1="50.8" y1="114.3" x2="58.42" y2="114.3" width="0.1524" layer="91"/>
+<label x="58.42" y="114.3" size="0.8128" layer="95" xref="yes"/>
 </segment>
 <segment>
-<pinref part="J22" gate="G$1" pin="3"/>
-<wire x1="53.34" y1="106.68" x2="58.42" y2="106.68" width="0.1524" layer="91"/>
-<label x="58.42" y="106.68" size="0.8128" layer="95" xref="yes"/>
+<pinref part="J42" gate="A" pin="2"/>
+<wire x1="50.8" y1="101.6" x2="58.42" y2="101.6" width="0.1524" layer="91"/>
+<label x="58.42" y="101.6" size="0.8128" layer="95" xref="yes"/>
 </segment>
 <segment>
-<pinref part="J23" gate="G$1" pin="3"/>
-<wire x1="53.34" y1="88.9" x2="58.42" y2="88.9" width="0.1524" layer="91"/>
+<pinref part="J43" gate="A" pin="2"/>
+<wire x1="50.8" y1="88.9" x2="58.42" y2="88.9" width="0.1524" layer="91"/>
 <label x="58.42" y="88.9" size="0.8128" layer="95" xref="yes"/>
-</segment>
-<segment>
-<pinref part="J24" gate="G$1" pin="3"/>
-<wire x1="53.34" y1="71.12" x2="58.42" y2="71.12" width="0.1524" layer="91"/>
-<label x="58.42" y="71.12" size="0.8128" layer="95" xref="yes"/>
 </segment>
 </net>
@@
 </segment>
 <segment>
-<pinref part="J22" gate="G$1" pin="1"/>
-<wire x1="53.34" y1="101.6" x2="58.42" y2="101.6" width="0.1524" layer="91"/>
-<label x="58.42" y="101.6" size="0.8128" layer="95" xref="yes"/>
+<pinref part="J42" gate="A" pin="3"/>
+<wire x1="50.8" y1="104.14" x2="58.42" y2="104.14" width="0.1524" layer="91"/>
+<label x="58.42" y="104.14" size="0.8128" layer="95" xref="yes"/>
 </segment>
 </net>
@@
 </segment>
 <segment>
-<pinref part="J23" gate="G$1" pin="1"/>
-<wire x1="53.34" y1="83.82" x2="58.42" y2="83.82" width="0.1524" layer="91"/>
-<label x="58.42" y="83.82" size="0.8128" layer="95" xref="yes"/>
+<pinref part="J43" gate="A" pin="3"/>
+<wire x1="50.8" y1="91.44" x2="58.42" y2="91.44" width="0.1524" layer="91"/>
+<label x="58.42" y="91.44" size="0.8128" layer="95" xref="yes"/>
 </segment>
 </net>
@@
 <label x="132.08" y="93.98" size="0.8128" layer="95" xref="yes"/>
 </segment>
-<segment>
-<pinref part="J24" gate="G$1" pin="1"/>
-<wire x1="53.34" y1="66.04" x2="58.42" y2="66.04" width="0.1524" layer="91"/>
-<label x="58.42" y="66.04" size="0.8128" layer="95" xref="yes"/>
-</segment>
 </net>
 <net name="ANLG0" class="0">
@@
 <wire x1="109.22" y1="106.68" x2="96.52" y2="106.68" width="0.1524" layer="91"/>
 <label x="96.52" y="106.68" size="0.8128" layer="95" rot="R180" xref="yes"/>
-</segment>
-<segment>
-<pinref part="J21" gate="G$1" pin="2"/>
-<wire x1="53.34" y1="121.92" x2="58.42" y2="121.92" width="0.1524" layer="91"/>
-<label x="58.42" y="121.92" size="0.8128" layer="95" xref="yes"/>
 </segment>
 </net>
@@
 <label x="96.52" y="101.6" size="0.8128" layer="95" rot="R180" xref="yes"/>
 </segment>
-<segment>
-<pinref part="J22" gate="G$1" pin="2"/>
-<wire x1="53.34" y1="104.14" x2="58.42" y2="104.14" width="0.1524" layer="91"/>
-<label x="58.42" y="104.14" size="0.8128" layer="95" xref="yes"/>
-</segment>
 </net>
 <net name="ANLG3" class="0">
@@
 <wire x1="109.22" y1="91.44" x2="96.52" y2="91.44" width="0.1524" layer="91"/>
 <label x="96.52" y="91.44" size="0.8128" layer="95" rot="R180" xref="yes"/>
-</segment>
-<segment>
-<pinref part="J24" gate="G$1" pin="2"/>
-<wire x1="53.34" y1="68.58" x2="58.42" y2="68.58" width="0.1524" layer="91"/>
-<label x="58.42" y="68.58" size="0.8128" layer="95" xref="yes"/>
 </segment>
 </net>
@@
 <label x="96.52" y="96.52" size="0.8128" layer="95" rot="R180" xref="yes"/>
 </segment>
-<segment>
-<pinref part="J23" gate="G$1" pin="2"/>
-<wire x1="53.34" y1="86.36" x2="58.42" y2="86.36" width="0.1524" layer="91"/>
-<label x="58.42" y="86.36" size="0.8128" layer="95" xref="yes"/>
-</segment>
 </net>
