File: Bellini/hardware/logicboard/bln-001.sch (EAGLE design)
At the start: 49 parts, among them IC1 74ACT06N, J1 MKR, J10 THS, J16 MNTR, J2 GPIO, J20 GPIO, J21 Grove, J22 Grove, J23 Grove, J24 Grove, J5 SPI, J6 LED, J7 DIN5, J8 DIN5, J9 DIN5, K1 G5V1, T1 2SC1815, X3 FAN

Commit message: Prototyping...
Parts:
- removed B0: 0, rcl:R-EU_M3216
- removed C11: 100n, rcl:C-EU025-024X044
- removed C12, C13: 1u, rcl:C-EU050-024X044
- removed D2, D3, D4: DIODE-1N4148, SparkFun-DiscreteSemi:DIODE-1N4148
- removed DISP1: AQM0802A-RN-GBW, AQM0802A-RN-GBW:AQM0802A-RN-GBW
- removed IC1: 74ACT06N, 74xx-eu:74ACT06N
- removed J1: MKR, SparkFun-Connectors:CONN_05JST
- removed J10: THS, SparkFun-Connectors:CONN_03JST-PTH-VERT
- removed J16: MNTR, SparkFun-Connectors:CONN_02-JST-2-PTH-NO_SILK
- removed J2: GPIO, SparkFun-Connectors:CONN_04JST-PTH
- removed J20: GPIO, SparkFun-Connectors:CONN_041.27MM
- removed J5: SPI, SparkFun-Connectors:CONN_061.27MM
- removed J6: LED, SparkFun-Connectors:CONN_03JST-PTH-VERT
- removed J7, J8, J9: DIN5, SparkFun-Connectors:DIN5
- removed JP8: Extended GPIO, SparkFun-Connectors:CONN_10LOCK
- removed K1: G5V1, relay:G5V1
- removed LED0: Green, led:LEDKA-3528ASYC
- removed LED1: Red, led:LEDKA-3528ASYC
- removed OK1: HCPL2630, optocoupler:HCPL2630
- removed R1, R4, R5: 1k, resistor:R-EU_0204/5
- removed R2: 10k, resistor:R-EU_0204/5
- removed RN2, RN3: 4.7k, resistor-net:RN04
- removed RN4: 220, resistor-dil:8R-N
- removed T1: 2SC1815, transistor:2SC1815
- removed X3: FAN, pinhead:PINHD-2X2
Connections:
- removed net BASE: R1.1, R2.2, T1.B
- removed net CAP1N: C12.2, DISP1.3
- removed net CAP1P: C12.1, DISP1.4
- removed net COLLECTOR: D2.A, K11.2, T1.C
- removed net COMMON: K12.P, K12.P@1, X3.2
- removed net FANDRIVE: B0.2, K12.S, X3.4
- removed net LCDVOUT: C13.2, DISP1.2
- removed net LED0A: J6.3, LED0.A, R4.1
- removed net LED1A: J6.1, LED1.A, R5.1
- removed net MIDIINSND: D3.C, OK1A.A1, RN4B.1
- removed net MIRTN: D3.A, J7.5, OK1A.C1
- removed net MISND: J7.4, RN4B.2
- removed net MNTRA: J16.2, RN4A.1
- removed net MNTRAA: D4.C, OK1B.A2, RN4A.2
- removed net MNTRK: D4.A, J16.1, OK1B.C2
- removed net MO2RTN: RN4H.2
- removed net MO2RTNRAW: IC1F.O, RN4H.1
- removed net MO2SND: RN4G.2
- removed net MORTN: J9.5, RN4D.2
- removed net MORTNRAW: IC1E.O, RN4D.1
- removed net MOSND: J9.4, RN4C.2
- removed net MTRTN: J8.5, RN4F.2
- removed net MTRTNRAW: IC1D.O, RN4F.1
- removed net MTSND: J8.4, RN4E.2
- removed net NMO2RTN: IC1C.O, IC1F.I, RN2.5
- removed net NMORTN: IC1B.O, IC1E.I, RN2.4
- removed net NMTRTN: IC1A.O, IC1D.I, RN2.3
- net DIGITAL7: no longer J1.4
- net GND: no longer C11.2, DISP1.6, J1.1, J10.1, J2.1, J5.6, J6.2, J8.2, J9.2, JP8.1, K12.O, LED0.C, LED1.C, OK1A.GND, R2.1, T1.E, X3.1
- net GPIO0: no longer J2.3, J20.3
- net GPIO1: no longer J2.4, J20.4
- net GPIO2: no longer JP8.3
- net GPIO3: no longer JP8.4
- net GPIO4: no longer JP8.5
- net GPIO5: no longer JP8.6
- net GPIO6: no longer JP8.7
- net GPIO7: no longer JP8.8
- net LED0: no longer R4.2
- net LED1: no longer R5.2
- net MISO: no longer J5.1
- net MNTR: no longer OK1B.VO2, RN3.5
- net MOSI: no longer J5.4
- net RLY: no longer R1.2
- net RST: no longer J5.5
- net RX: no longer IC1A.I, OK1A.VO1, RN3.4
- net SCK: no longer J5.3
- net SCL: no longer DISP1.8, J1.3
- net SDA: no longer DISP1.7, J1.2
- net THS: no longer J10.2, RN3.3
- net TX: no longer IC1B.I, IC1C.I
- net VCC: no longer B0.1, RN2.1, RN4C.1, RN4E.1, RN4G.1, X3.3
- net VDD: no longer C11.1, C13.1, D2.C, DISP1.5, DISP1.9, J1.5, J10.3, J2.2, J5.2, JP8.2, K11.1, OK1A.VCC, RN3.1

Commit message: Cleaning.
Parts:
- removed H1, H2: STAND-OFF, SparkFun-Hardware:STAND-OFF
- removed J23, J24: Grove, Connector:TWIG-4P-2.0
- removed JP2: RTC, SparkFun-Connectors:CONN_05PTH
- removed SV3: Testport II, pinhead:PINHD-2X7
- added JP01: (no value), pinhead:PINHD-2X5
Connections:
- net DIGITAL7: no longer SV3.11
- net DTCT0: no longer SV3.8
- net DTCT1: no longer SV3.10
- net DTCT2: no longer SV3.12
- net DTCT3: no longer SV3.14
- net GND: no longer J23.4, J24.4, JP2.2, SV3.5
- net GPIO0: no longer SV3.2
- net GPIO1: no longer SV3.4
- net RX: no longer SV3.3
- net SCL: no longer J23.1, J24.1, JP2.4, SV3.9
- net SDA: no longer J23.2, J24.2, JP2.5, SV3.7
- net THS: no longer SV3.6
- net TX: no longer SV3.1
- net VDD: no longer J23.3, J24.3, JP2.1, SV3.13

Commit message: Layout.
Parts:
- removed J22: Grove, Connector:TWIG-4P-2.0'90D'
- added JP02, JP03: (no value), adafruit:PINHD-1X8BIG
- added JP04, JP05: (no value), pinhead:PINHD-1X14
Connections:
- net GND: no longer J22.4
- net SCL: no longer J22.1
- net SDA: no longer J22.2
- net VDD: no longer J22.3
Changed lines of the file:
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@@
 <part name="S1" library="switch-omron" library_urn="urn:adsk.eagle:library:377" deviceset="31-XX" device="" package3d_urn="urn:adsk.eagle:package:27487/1" value="RST"/>
 <part name="J21" library="Connector" deviceset="TWIG-4P-2.0" device="'90D'" value="Grove"/>
-<part name="J22" library="Connector" deviceset="TWIG-4P-2.0" device="'90D'" value="Grove"/>
 <part name="NC11" library="wirepad" library_urn="urn:adsk.eagle:library:412" deviceset="PAD-N" device=""/>
 <part name="JP01" library="pinhead" library_urn="urn:adsk.eagle:library:325" deviceset="PINHD-2X5" device="" package3d_urn="urn:adsk.eagle:package:22470/2"/>
+<part name="JP02" library="adafruit" library_urn="urn:adsk.eagle:library:420" deviceset="PINHD-1X8" device="BIG" package3d_urn="urn:adsk.eagle:package:6240707/1"/>
+<part name="JP03" library="adafruit" library_urn="urn:adsk.eagle:library:420" deviceset="PINHD-1X8" device="BIG" package3d_urn="urn:adsk.eagle:package:6240707/1"/>
+<part name="JP04" library="pinhead" library_urn="urn:adsk.eagle:library:325" deviceset="PINHD-1X14" device="" package3d_urn="urn:adsk.eagle:package:22417/2"/>
+<part name="JP05" library="pinhead" library_urn="urn:adsk.eagle:library:325" deviceset="PINHD-1X14" device="" package3d_urn="urn:adsk.eagle:package:22417/2"/>
 </parts>
 <sheets>
@@
 <attribute name="VALUE" x="45.72" y="125.73" size="1.27" layer="96" rot="R270"/>
 </instance>
-<instance part="J22" gate="G$1" x="48.26" y="109.22" smashed="yes" rot="R180">
-<attribute name="NAME" x="49.53" y="104.14" size="1.27" layer="95" rot="R180"/>
-<attribute name="VALUE" x="45.72" y="113.03" size="1.27" layer="96" rot="R270"/>
-</instance>
 <instance part="NC11" gate="G$1" x="228.6" y="157.48" smashed="yes"/>
 <instance part="JP01" gate="A" x="274.32" y="96.52" smashed="yes">
 <attribute name="NAME" x="267.97" y="104.775" size="1.778" layer="95"/>
 <attribute name="VALUE" x="267.97" y="86.36" size="1.778" layer="96"/>
+</instance>
+<instance part="JP02" gate="G$1" x="152.4" y="104.14" smashed="yes">
+<attribute name="NAME" x="146.05" y="114.935" size="1.778" layer="95"/>
+<attribute name="VALUE" x="146.05" y="88.9" size="1.778" layer="96"/>
+</instance>
+<instance part="JP03" gate="G$1" x="190.5" y="99.06" smashed="yes">
+<attribute name="NAME" x="184.15" y="109.855" size="1.778" layer="95"/>
+<attribute name="VALUE" x="184.15" y="83.82" size="1.778" layer="96"/>
+</instance>
+<instance part="JP04" gate="A" x="45.72" y="200.66" smashed="yes">
+<attribute name="NAME" x="39.37" y="219.075" size="1.778" layer="95"/>
+<attribute name="VALUE" x="39.37" y="177.8" size="1.778" layer="96"/>
+</instance>
+<instance part="JP05" gate="A" x="78.74" y="195.58" smashed="yes">
+<attribute name="NAME" x="72.39" y="213.995" size="1.778" layer="95"/>
+<attribute name="VALUE" x="72.39" y="172.72" size="1.778" layer="96"/>
 </instance>
 </instances>
@@
 <wire x1="53.34" y1="127" x2="55.88" y2="127" width="0.1524" layer="91"/>
 <label x="96.52" y="127" size="0.8128" layer="95" xref="yes"/>
-<pinref part="J22" gate="G$1" pin="4"/>
 <wire x1="55.88" y1="127" x2="66.04" y2="127" width="0.1524" layer="91"/>
 <wire x1="66.04" y1="127" x2="76.2" y2="127" width="0.1524" layer="91"/>
@@
 <wire x1="53.34" y1="121.92" x2="60.96" y2="121.92" width="0.1524" layer="91"/>
 <label x="96.52" y="121.92" size="0.8128" layer="95" xref="yes"/>
-<pinref part="J22" gate="G$1" pin="2"/>
 <wire x1="60.96" y1="121.92" x2="71.12" y2="121.92" width="0.1524" layer="91"/>
 <wire x1="71.12" y1="121.92" x2="81.28" y2="121.92" width="0.1524" layer="91"/>
@@
 <wire x1="53.34" y1="124.46" x2="58.42" y2="124.46" width="0.1524" layer="91"/>
 <label x="96.52" y="124.46" size="0.8128" layer="95" xref="yes"/>
-<pinref part="J22" gate="G$1" pin="3"/>
 <wire x1="58.42" y1="124.46" x2="68.58" y2="124.46" width="0.1524" layer="91"/>
 <wire x1="68.58" y1="124.46" x2="78.74" y2="124.46" width="0.1524" layer="91"/>
@@
 <wire x1="53.34" y1="119.38" x2="63.5" y2="119.38" width="0.1524" layer="91"/>
 <label x="96.52" y="119.38" size="0.8128" layer="95" xref="yes"/>
-<pinref part="J22" gate="G$1" pin="1"/>
 <wire x1="63.5" y1="119.38" x2="73.66" y2="119.38" width="0.1524" layer="91"/>
 <wire x1="73.66" y1="119.38" x2="83.82" y2="119.38" width="0.1524" layer="91"/>

Commit message: Routed.
Parts:
- removed JP01: (no value), pinhead:PINHD-2X5
- removed JP02, JP03: (no value), adafruit:PINHD-1X8BIG
- removed JP04, JP05: (no value), pinhead:PINHD-1X14
- added DRIVERPIN1, DRIVERPIN2: (no value), pinhead:PINHD-1X14
- added LEDPIN1, LEDPIN2: (no value), adafruit:PINHD-1X8BIG
- added LEVELSHIFT1, LEVELSHIFT2: (no value), pinhead:PINHD-1X4
- added RTCPIN: (no value), pinhead:PINHD-2X5
- renumbered J21 to GROVE1
Connections:
- removed net DTCT0: MC2.GPIO_22
- removed net DTCT1: MC2.GPIO_23
- removed net DTCT2: MC2.GPIO_24
- removed net DTCT3: MC2.GPIO_25
- removed net GPIO0: MC2.GPIO20/SPI0_MOSI1
- removed net GPIO1: MC2.GPIO21/SPI0_SCLK1
- removed net GPIO2: MC2.GPIO_8/SPI0_CE1_N
- removed net GPIO3: MC2.GPIO16/SPI1_CS2
- removed net GPIO4: MC2.GPIO_17/SPI1_CS1
- removed net GPIO5: MC2.GPIO_18/PWM0/SPI1_CS0
- removed net GPIO6: MC2.GPIO19/SPI0_MISO1/PWM1
- removed net GPIO7: MC2.GPIO26
- removed net LED0: MC2.GPIO12/PWM0
- removed net LED1: MC2.GPIO13/PWM1
- removed net MISO: MC2.GPIO_9/SPI0_MISO
- removed net MNTR: MC2.GPIO6/GPCLK2
- removed net MOSI: MC2.GPIO_10/SPI0_MOSI
- removed net RLY: MC2.GPIO5//GPCLK1
- removed net SCK: MC2.GPIO_11/SPI0_SCLK
- removed net THS: MC2.GPIO_4/GPCLK0
- new net COL1: DRIVERPIN2.11, LEDPIN2.5
- new net COL2: DRIVERPIN2.10, LEDPIN1.3
- new net COL3: DRIVERPIN2.9, LEDPIN1.4
- new net COL4: DRIVERPIN2.8, LEDPIN2.3
- new net COL5: DRIVERPIN2.7, LEDPIN1.6
- new net COL6: DRIVERPIN2.6
- new net COL7: DRIVERPIN2.5, LEDPIN2.7
- new net COL8: DRIVERPIN2.4, LEDPIN2.8
- new net N$10: DRIVERPIN1.11
- new net N$11: DRIVERPIN1.12
- new net N$12: DRIVERPIN1.13
- new net N$13: DRIVERPIN1.14
- new net N$14: DRIVERPIN2.1
- new net N$15: DRIVERPIN2.2
- new net N$16: DRIVERPIN2.3
- new net N$5: LEVELSHIFT1.4
- new net N$9: DRIVERPIN1.10
- new net ROW1: DRIVERPIN1.2, LEDPIN2.1
- new net ROW2: DRIVERPIN1.3, LEDPIN2.6
- new net ROW3: DRIVERPIN1.4, LEDPIN1.8
- new net ROW4: DRIVERPIN1.5, LEDPIN2.4
- new net ROW5: DRIVERPIN1.6, LEDPIN1.1
- new net ROW6: DRIVERPIN1.7, LEDPIN1.7
- new net ROW7: DRIVERPIN1.8, LEDPIN1.2, LEDPIN2.2
- new net ROW8: DRIVERPIN1.9, LEDPIN1.5
- new net SCL5V: DRIVERPIN2.12, LEVELSHIFT2.3
- new net SDA5V: DRIVERPIN2.13, LEVELSHIFT2.2
- net DIGITAL7: now also RTCPIN.7
- net GND: now also DRIVERPIN1.1, LEVELSHIFT2.1, RTCPIN.6, RTCPIN.9; no longer MC2.GND5
- net RX: now also RTCPIN.10
- net SCL: now also LEVELSHIFT1.2, RTCPIN.5
- net SDA: now also LEVELSHIFT1.3, RTCPIN.3
- net TX: now also RTCPIN.8
- net VCC: now also DRIVERPIN2.14, LEVELSHIFT2.4, RTCPIN.2, RTCPIN.4
- net VDD: now also LEVELSHIFT1.1, RTCPIN.1

Commit message: Fixed errors.
Connections:
- net COL1 renamed A0
- net COL2 renamed A1
- net COL3 renamed A2
- net COL5 renamed A4
- net COL7 renamed A6
- net COL8 renamed A7
- net ROW1 renamed C0
- net ROW2 renamed C1
- net ROW3 renamed C2
- net ROW4 renamed C3
- net ROW5 renamed C4
- net ROW6 renamed C5
- net ROW8 renamed C7
- removed net COL4: DRIVERPIN2.8, LEDPIN2.3
- removed net COL6: DRIVERPIN2.6
- removed net ROW7: DRIVERPIN1.8, LEDPIN1.2, LEDPIN2.2
- new net A3: DRIVERPIN2.8, LEDPIN2.2
- new net A5: DRIVERPIN2.6, LEDPIN2.3
- new net C6: DRIVERPIN1.8, LEDPIN1.2
