File: Bellini/hardware/logicboard/bln-000.sch (EAGLE design)
At the start: 16 parts

Commit message: 000.
Parts:
- removed DRIVERPIN1, DRIVERPIN2: (no value), pinhead:PINHD-1X14
- removed LEDPIN1, LEDPIN2: (no value), adafruit:PINHD-1X8BIG
- removed LEVELSHIFT1, LEVELSHIFT2: (no value), pinhead:PINHD-1X4
- removed RTCPIN: (no value), pinhead:PINHD-2X5
- added H1, H2, H3, H4, H5, H6, H7, H8: STAND-OFF, SparkFun-Hardware:STAND-OFF
- added QWIIC1: QWIIC_RIGHT_ANGLE, SparkFun-Connectors:QWIIC_CONNECTORJS-1MM
Connections:
- removed net A0: DRIVERPIN2.11, LEDPIN2.5
- removed net A1: DRIVERPIN2.10, LEDPIN1.3
- removed net A2: DRIVERPIN2.9, LEDPIN1.4
- removed net A3: DRIVERPIN2.8, LEDPIN2.2
- removed net A4: DRIVERPIN2.7, LEDPIN1.6
- removed net A5: DRIVERPIN2.6, LEDPIN2.3
- removed net A6: DRIVERPIN2.5, LEDPIN2.7
- removed net A7: DRIVERPIN2.4, LEDPIN2.8
- removed net C0: DRIVERPIN1.2, LEDPIN2.1
- removed net C1: DRIVERPIN1.3, LEDPIN2.6
- removed net C2: DRIVERPIN1.4, LEDPIN1.8
- removed net C3: DRIVERPIN1.5, LEDPIN2.4
- removed net C4: DRIVERPIN1.6, LEDPIN1.1
- removed net C5: DRIVERPIN1.7, LEDPIN1.7
- removed net C6: DRIVERPIN1.8, LEDPIN1.2
- removed net C7: DRIVERPIN1.9, LEDPIN1.5
- removed net N$10: DRIVERPIN1.11
- removed net N$11: DRIVERPIN1.12
- removed net N$12: DRIVERPIN1.13
- removed net N$13: DRIVERPIN1.14
- removed net N$14: DRIVERPIN2.1
- removed net N$15: DRIVERPIN2.2
- removed net N$16: DRIVERPIN2.3
- removed net N$5: LEVELSHIFT1.4
- removed net N$9: DRIVERPIN1.10
- removed net SCL5V: DRIVERPIN2.12, LEVELSHIFT2.3
- removed net SDA5V: DRIVERPIN2.13, LEVELSHIFT2.2
- net DIGITAL7: no longer RTCPIN.7
- net GND: now also QWIIC1.1; no longer DRIVERPIN1.1, LEVELSHIFT2.1, RTCPIN.6, RTCPIN.9
- net RX: no longer RTCPIN.10
- net SCL: now also QWIIC1.4; no longer LEVELSHIFT1.2, RTCPIN.5
- net SDA: now also QWIIC1.3; no longer LEVELSHIFT1.3, RTCPIN.3
- net TX: no longer RTCPIN.8
- net VCC: no longer DRIVERPIN2.14, LEVELSHIFT2.4, RTCPIN.2, RTCPIN.4
- net VDD: now also QWIIC1.2; no longer LEVELSHIFT1.1, RTCPIN.1
