File: Bellini/hardware/logicboard/bln-001.brd (EAGLE design)
At the start: 100 x 80 mm, 16 parts

Commit message: 000.
Parts:
- moved LEVELSHIFT1 4.00 mm to (86.2, 64.0)
- moved LEVELSHIFT2 4.00 mm to (93.8, 64.0)
Routing:
- net GND: track 207.3 -> 0.00 mm
- net VDD: track 160.5 -> 0.00 mm, vias 1 -> 0
- net SDA: track 115.0 -> 0.00 mm
- net SCL: track 113.1 -> 0.00 mm
- net VCC: track 109.5 -> 0.00 mm, vias 1 -> 0
- net A4: track 73.1 -> 0.00 mm
- net A2: track 68.1 -> 0.00 mm
- net A1: track 63.7 -> 0.00 mm
- net TX: track 54.5 -> 0.00 mm
- net RST: track 54.3 -> 0.00 mm
- net RX: track 49.1 -> 0.00 mm
- net C4: track 47.6 -> 0.00 mm
- net A0: track 43.3 -> 0.00 mm
- net C5: track 39.6 -> 0.00 mm
- net C7: track 38.7 -> 0.00 mm
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- removed copper zone on layer 1, net GND
- removed copper zone on layer 16, net GND
