File: Bellini/hardware/logicboard/bln-002.brd (EAGLE design)
At the start: 100 x 80 mm, 16 parts

Commit message: Belini 2 (?).
Parts:
- removed LEDPIN1, LEDPIN2: (no value), adafruit:1X08-BIG
- added DZ1, DZ2, DZ3: LB10, led:LB10
Connections:
- net A0: no longer LEDPIN2.5
- net A1: no longer LEDPIN1.3
- net A2: no longer LEDPIN1.4
- net A3: no longer LEDPIN2.2
- net A4: no longer LEDPIN1.6
- net A5: no longer LEDPIN2.3
- net A6: no longer LEDPIN2.7
- net A7: no longer LEDPIN2.8
- net C0: no longer LEDPIN2.1
- net C1: no longer LEDPIN2.6
- net C2: no longer LEDPIN1.8
- net C3: no longer LEDPIN2.4
- net C4: no longer LEDPIN1.1
- net C5: no longer LEDPIN1.7
- net C6: no longer LEDPIN1.2
- net C7: no longer LEDPIN1.5
Changed lines of the file:
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@@
 <setting verticaltext="up"/>
 </settings>
-<grid distance="1" unitdist="mm" unit="mm" style="lines" multiple="2" display="yes" altdistance="50" altunitdist="mil" altunit="mil"/>
+<grid distance="2" unitdist="mm" unit="mm" style="lines" multiple="2" display="yes" altdistance="50" altunitdist="mil" altunit="mil"/>
 <layers>
 <layer number="1" name="Top" color="4" fill="1" visible="yes" active="yes"/>
@@
 <attribute name="VALUE" x="8.65" y="35.555" size="1.27" layer="27"/>
 </element>
-<element name="LEDPIN1" library="adafruit" library_urn="urn:adsk.eagle:library:420" package="1X08-BIG" package3d_urn="urn:adsk.eagle:package:6240707/1" value="" x="35.8" y="25" smashed="yes" rot="R90">
-<attribute name="NAME" x="33" y="25" size="1" layer="25" ratio="10" rot="R90" align="center"/>
-<attribute name="VALUE" x="38.975" y="14.84" size="1.27" layer="27" rot="R90"/>
-</element>
-<element name="LEDPIN2" library="adafruit" library_urn="urn:adsk.eagle:library:420" package="1X08-BIG" package3d_urn="urn:adsk.eagle:package:6240707/1" value="" x="64.2" y="25" smashed="yes" rot="R270">
-<attribute name="NAME" x="67" y="25" size="1" layer="25" ratio="10" rot="R90" align="center"/>
-<attribute name="VALUE" x="61.025" y="35.16" size="1.27" layer="27" rot="R270"/>
-</element>
 <element name="DRIVERPIN1" library="pinhead" library_urn="urn:adsk.eagle:library:325" package="1X14" package3d_urn="urn:adsk.eagle:package:22417/2" value="" x="72.36" y="25" smashed="yes" rot="R270">
 <attribute name="NAME" x="70" y="25" size="1" layer="25" ratio="10" rot="R90" align="center"/>
@@
 <attribute name="POPULARITY" value="91" x="93.81" y="64" size="1.778" layer="27" rot="R90" display="off"/>
 <attribute name="VALUE" x="96.985" y="58.92" size="1.27" layer="27" rot="R90"/>
+</element>
+<element name="DZ1" library="led" library_urn="urn:adsk.eagle:library:259" package="LB10" package3d_urn="urn:adsk.eagle:package:15791/1" value="LB10" x="18" y="40" smashed="yes">
+<attribute name="NAME" x="5.3" y="45.715" size="1.27" layer="25" ratio="10"/>
+<attribute name="POPULARITY" value="1" x="18" y="40" size="1.778" layer="27" display="off"/>
+<attribute name="VALUE" x="14.19" y="45.715" size="1.27" layer="27" ratio="10"/>
+</element>
+<element name="DZ2" library="led" library_urn="urn:adsk.eagle:library:259" package="LB10" package3d_urn="urn:adsk.eagle:package:15791/1" value="LB10" x="50" y="40" smashed="yes">
+<attribute name="NAME" x="37.3" y="45.715" size="1.27" layer="25" ratio="10"/>
+<attribute name="POPULARITY" value="1" x="50" y="40" size="1.778" layer="27" display="off"/>
+<attribute name="VALUE" x="46.19" y="45.715" size="1.27" layer="27" ratio="10"/>
+</element>
+<element name="DZ3" library="led" library_urn="urn:adsk.eagle:library:259" package="LB10" package3d_urn="urn:adsk.eagle:package:15791/1" value="LB10" x="79" y="40" smashed="yes">
+<attribute name="NAME" x="66.3" y="45.715" size="1.27" layer="25" ratio="10"/>
+<attribute name="POPULARITY" value="1" x="79" y="40" size="1.778" layer="27" display="off"/>
+<attribute name="VALUE" x="75.19" y="45.715" size="1.27" layer="27" ratio="10"/>
 </element>
 </elements>
@@
 <signal name="A3">
 <contactref element="DRIVERPIN2" pad="8"/>
-<contactref element="LEDPIN2" pad="2"/>
-<wire x1="64.2" y1="31.35" x2="90.14" y2="26.27" width="0" layer="19" extent="1-1"/>
 </signal>
 <signal name="N$9">
@@
 <signal name="C0">
 <contactref element="DRIVERPIN1" pad="2"/>
-<contactref element="LEDPIN2" pad="1"/>
-<wire x1="64.2" y1="33.89" x2="72.36" y2="38.97" width="0" layer="19" extent="1-1"/>
 </signal>
 <signal name="C1">
 <contactref element="DRIVERPIN1" pad="3"/>
-<contactref element="LEDPIN2" pad="6"/>
-<wire x1="64.2" y1="21.19" x2="72.36" y2="36.43" width="0" layer="19" extent="1-1"/>
 </signal>
 <signal name="C2">
 <contactref element="DRIVERPIN1" pad="4"/>
-<contactref element="LEDPIN1" pad="8"/>
-<wire x1="35.8" y1="33.89" x2="72.36" y2="33.89" width="0" layer="19" extent="1-1"/>
 </signal>
 <signal name="C3">
 <contactref element="DRIVERPIN1" pad="5"/>
-<contactref element="LEDPIN2" pad="4"/>
-<wire x1="64.2" y1="26.27" x2="72.36" y2="31.35" width="0" layer="19" extent="1-1"/>
 </signal>
 <signal name="C4">
 <contactref element="DRIVERPIN1" pad="6"/>
-<contactref element="LEDPIN1" pad="1"/>
-<wire x1="35.8" y1="16.11" x2="72.36" y2="28.81" width="0" layer="19" extent="1-1"/>
 </signal>
 <signal name="C5">
 <contactref element="DRIVERPIN1" pad="7"/>
-<contactref element="LEDPIN1" pad="7"/>
-<wire x1="35.8" y1="31.35" x2="72.36" y2="26.27" width="0" layer="19" extent="1-1"/>
 </signal>
 <signal name="C6">
 <contactref element="DRIVERPIN1" pad="8"/>
-<contactref element="LEDPIN1" pad="2"/>
-<wire x1="35.8" y1="18.65" x2="72.36" y2="23.73" width="0" layer="19" extent="1-1"/>
 </signal>
 <signal name="C7">
 <contactref element="DRIVERPIN1" pad="9"/>
-<contactref element="LEDPIN1" pad="5"/>
-<wire x1="35.8" y1="26.27" x2="72.36" y2="21.19" width="0" layer="19" extent="1-1"/>
 </signal>
 <signal name="A7">
 <contactref element="DRIVERPIN2" pad="4"/>
-<contactref element="LEDPIN2" pad="8"/>
-<wire x1="64.2" y1="16.11" x2="90.14" y2="16.11" width="0" layer="19" extent="1-1"/>
 </signal>
 <signal name="A6">
 <contactref element="DRIVERPIN2" pad="5"/>
-<contactref element="LEDPIN2" pad="7"/>
-<wire x1="64.2" y1="18.65" x2="90.14" y2="18.65" width="0" layer="19" extent="1-1"/>
 </signal>
 <signal name="A5">
 <contactref element="DRIVERPIN2" pad="6"/>
-<contactref element="LEDPIN2" pad="3"/>
-<wire x1="64.2" y1="28.81" x2="90.14" y2="21.19" width="0" layer="19" extent="1-1"/>
 </signal>
 <signal name="A4">
 <contactref element="DRIVERPIN2" pad="7"/>
-<contactref element="LEDPIN1" pad="6"/>
-<wire x1="35.8" y1="28.81" x2="90.14" y2="23.73" width="0" layer="19" extent="1-1"/>
 </signal>
 <signal name="A2">
 <contactref element="DRIVERPIN2" pad="9"/>
-<contactref element="LEDPIN1" pad="4"/>
-<wire x1="35.8" y1="23.73" x2="90.14" y2="28.81" width="0" layer="19" extent="1-1"/>
 </signal>
 <signal name="A1">
 <contactref element="DRIVERPIN2" pad="10"/>
-<contactref element="LEDPIN1" pad="3"/>
-<wire x1="35.8" y1="21.19" x2="90.14" y2="31.35" width="0" layer="19" extent="1-1"/>
 </signal>
 <signal name="A0">
 <contactref element="DRIVERPIN2" pad="11"/>
-<contactref element="LEDPIN2" pad="5"/>
-<wire x1="64.2" y1="23.73" x2="90.14" y2="33.89" width="0" layer="19" extent="1-1"/>
 </signal>
 </signals>
