File: Bellini/hardware/logicboard/bln-002.sch (EAGLE design)
At the start: 16 parts

Commit message: Belini 2 (?).
Parts:
- removed LEDPIN1, LEDPIN2: (no value), adafruit:PINHD-1X8BIG
- added DZ1, DZ2, DZ3: LB10, led:LB10
Connections:
- net A0: no longer LEDPIN2.5
- net A1: no longer LEDPIN1.3
- net A2: no longer LEDPIN1.4
- net A3: no longer LEDPIN2.2
- net A4: no longer LEDPIN1.6
- net A5: no longer LEDPIN2.3
- net A6: no longer LEDPIN2.7
- net A7: no longer LEDPIN2.8
- net C0: no longer LEDPIN2.1
- net C1: no longer LEDPIN2.6
- net C2: no longer LEDPIN1.8
- net C3: no longer LEDPIN2.4
- net C4: no longer LEDPIN1.1
- net C5: no longer LEDPIN1.7
- net C6: no longer LEDPIN1.2
- net C7: no longer LEDPIN1.5
